Commit message: updates in sync with test setup

File: rox_description/urdf/rox.urdf (robot description, URDF)
Before this commit: robot mpo_700, 12 links, 11 joints
Links:
- removed link mpo_700_caster_back_left_link
- removed link mpo_700_caster_back_right_link
- removed link mpo_700_caster_front_left_link
- removed link mpo_700_caster_front_right_link
- removed link mpo_700_wheel_back_left_link
- removed link mpo_700_wheel_back_right_link
- removed link mpo_700_wheel_front_left_link
- removed link mpo_700_wheel_front_right_link
- added link caster_back_left_link, mass 12.7; collision mesh filename=package://rox_description/meshes/argo_caster.dae scale=0.001 0.001 0.001; visual mesh filename=package://rox_description/meshes/argo_caster.dae scale=0.001 0.001 0.001
- added link caster_back_right_link, mass 12.7; collision mesh filename=package://rox_description/meshes/argo_caster.dae scale=0.001 0.001 0.001; visual mesh filename=package://rox_description/meshes/argo_caster.dae scale=0.001 0.001 0.001
- added link caster_front_left_link, mass 12.7; collision mesh filename=package://rox_description/meshes/argo_caster.dae scale=0.001 0.001 0.001; visual mesh filename=package://rox_description/meshes/argo_caster.dae scale=0.001 0.001 0.001
- added link caster_front_right_link, mass 12.7; collision mesh filename=package://rox_description/meshes/argo_caster.dae scale=0.001 0.001 0.001; visual mesh filename=package://rox_description/meshes/argo_caster.dae scale=0.001 0.001 0.001
- added link wheel_back_left_link, mass 1.2; collision sphere radius=0.09; visual mesh filename=package://rox_description/meshes/argo_wheel.dae scale=0.1 0.1 0.1
- added link wheel_back_right_link, mass 1.2; collision sphere radius=0.09; visual mesh filename=package://rox_description/meshes/argo_wheel.dae scale=0.1 0.1 0.1
- added link wheel_front_left_link, mass 1.2; collision sphere radius=0.09; visual mesh filename=package://rox_description/meshes/argo_wheel.dae scale=0.1 0.1 0.1
- added link wheel_front_right_link, mass 1.2; collision sphere radius=0.09; visual mesh filename=package://rox_description/meshes/argo_wheel.dae scale=0.1 0.1 0.1
Joints:
- removed joint mpo_700_caster_back_left_joint
- removed joint mpo_700_caster_back_right_joint
- removed joint mpo_700_caster_front_left_joint
- removed joint mpo_700_caster_front_right_joint
- removed joint mpo_700_wheel_back_left_joint
- removed joint mpo_700_wheel_back_right_joint
- removed joint mpo_700_wheel_front_left_joint
- removed joint mpo_700_wheel_front_right_joint
- added joint caster_back_left_joint: type revolute, parent base_footprint, child caster_back_left_link, origin xyz=-0.45 0.21 0.123 rpy=0 0 3.14, axis 0 0 1, limit lower=-1e+16 upper=1e+16 effort=1000.0 velocity=6.5
- added joint caster_back_right_joint: type revolute, parent base_footprint, child caster_back_right_link, origin xyz=-0.45 -0.21 0.123 rpy=0 0 0, axis 0 0 1, limit lower=-1e+16 upper=1e+16 effort=1000.0 velocity=6.5
- added joint caster_front_left_joint: type revolute, parent base_footprint, child caster_front_left_link, origin xyz=0.45 0.21 0.123 rpy=0 0 3.14, axis 0 0 1, limit lower=-1e+16 upper=1e+16 effort=1000.0 velocity=6.5
- added joint caster_front_right_joint: type revolute, parent base_footprint, child caster_front_right_link, origin xyz=0.45 -0.21 0.123 rpy=0 0 0, axis 0 0 1, limit lower=-1e+16 upper=1e+16 effort=1000.0 velocity=6.5
- added joint wheel_back_left_joint: type revolute, parent caster_back_left_link, child wheel_back_left_link, origin xyz=0.0 0.0 -0.07225 rpy=0 0 0, axis 0 -1 0, limit lower=-1e+16 upper=1e+16 effort=1000.0 velocity=20.5
- added joint wheel_back_right_joint: type revolute, parent caster_back_right_link, child wheel_back_right_link, origin xyz=0.0 0 -0.07225 rpy=0 0 3.14, axis 0 -1 0, limit lower=-1e+16 upper=1e+16 effort=1000.0 velocity=20.5
- added joint wheel_front_left_joint: type revolute, parent caster_front_left_link, child wheel_front_left_link, origin xyz=0.0 0.0 -0.07225 rpy=0 0 0, axis 0 -1 0, limit lower=-1e+16 upper=1e+16 effort=1000.0 velocity=20.5
- added joint wheel_front_right_joint: type revolute, parent caster_front_right_link, child wheel_front_right_link, origin xyz=0.0 0.0 -0.07225 rpy=0 0 3.14, axis 0 -1 0, limit lower=-1e+16 upper=1e+16 effort=1000.0 velocity=20.5
