Commit message: updating the xacross

File: rox_description/urdf/rox.urdf.xacro (robot description, xacro)
@@ -3,5 +3,5 @@
     <!-- Xacro Arguments-->
     <xacro:arg name="frame_type" default="short"/>
-    <xacro:arg name="joint_type" default="revolute"/>
+    <xacro:arg name="joint_type" default="fixed"/>
     <xacro:property name="frame" value="$(arg frame_type)"/>
     <xacro:property name="joint_typ" value="$(arg joint_type)"/>
@@ -10,4 +10,5 @@
     <xacro:include filename="$(find rox_description)/urdf/xacros/argo_caster.xacro" />
     <xacro:include filename="$(find rox_description)/urdf/xacros/argo_wheel.xacro" />
+    <xacro:include filename="$(find rox_description)/urdf/xacros/sick_nanoscan.xacro" />
     <!-- Assigning Xacro properties -->
     <xacro:if value="${frame == 'short'}">
@@ -67,5 +68,11 @@
         vis_rot="0 0 0" vis_pos="0 0 0"
         joint_type="${joint_typ}">
-        <origin xyz="${wheel_pos}" rpy="${wheel_rot}"/>
+        <origin rpy="3.14 0 0" xyz="0.60 0.25 0.10"/>
     </xacro:argo_wheel>
+    <xacro:sick_nanoscan name="lidar_1" parent="base_footprint">
+        <origin rpy="3.14 0 0" xyz="0.60 0.25 0.10"/>
+    </xacro:sick_nanoscan>
+    <xacro:sick_nanoscan name="lidar_2" parent="base_footprint">
+        <origin rpy="3.14 0 3.14" xyz="-0.60 -0.25 0.10"/>
+    </xacro:sick_nanoscan>
 </robot>

File: rox_description/urdf/xacros/argo_wheel.xacro (robot description, xacro)
@@ -1,5 +1,5 @@
 <?xml version="1.0"?>
 <robot xmlns:xacro="http://www.ros.org/wiki/xacro" name="rox">
-  <xacro:macro name="argo_caster" params="name parent *origin vis_rot vis_pos joint_type">
+  <xacro:macro name="argo_wheel" params="name parent *origin vis_rot vis_pos joint_type">
    <joint name="${name}_joint" type="${joint_type}">
     <xacro:insert_block name="origin" />
@@ -20,5 +20,5 @@
      <origin xyz="${vis_pos}" rpy="${vis_rot}" />
      <geometry>
-        <mesh filename="package://rox_description/meshes/argo_wheel.dae" scale="0.001 0.001 0.001"/>
+        <mesh filename="package://rox_description/meshes/argo_wheel.dae" scale="0.1 0.1 0.1"/>
      </geometry>
     </visual>
@@ -26,5 +26,5 @@
      <origin xyz="${vis_pos}" rpy="${vis_rot}" />
      <geometry>
-        <mesh filename="package://rox_description/meshes/argo_wheel.dae" scale="0.001 0.001 0.001"/>
+        <mesh filename="package://rox_description/meshes/argo_wheel.dae" scale="0.1 0.1 0.1"/>
      </geometry>
     </collision>

File: rox_description/urdf/xacros/frame.xacro (robot description, xacro)
@@ -21,5 +21,5 @@
         <origin xyz="${vis_pos}" rpy="${vis_rot}" />
         <geometry>
-            <mesh filename="package://rox_description/meshes/${type}_frame.dae" scale="0.001 0.001 0.001"/>
+            <mesh filename="package://rox_description/meshes/${type}_frame.dae" scale="0.1 0.1 0.1"/>
         </geometry>
       </visual>
@@ -27,5 +27,5 @@
         <origin xyz="${vis_pos}" rpy="${vis_rot}" />
         <geometry>
-            <mesh filename="package://rox_description/meshes/${type}_frame.dae" scale="0.001 0.001 0.001"/>
+            <mesh filename="package://rox_description/meshes/${type}_frame.dae" scale="0.1 0.1 0.1"/>
         </geometry>
       </collision>

Commit message: adding cabinet

File: rox_description/urdf/rox.urdf.xacro (robot description, xacro)
@@ -4,6 +4,8 @@
     <xacro:arg name="frame_type" default="short"/>
     <xacro:arg name="joint_type" default="fixed"/>
+    <xacro:arg name="arm_type" default=""/>
     <xacro:property name="frame" value="$(arg frame_type)"/>
     <xacro:property name="joint_typ" value="$(arg joint_type)"/>
+    <xacro:property name="arm" value="$(arg arm_type)"/>
     <!-- Include xacro files -->
     <xacro:include filename="$(find rox_description)/urdf/xacros/frame.xacro" />
@@ -17,4 +19,5 @@
         <xacro:property name="wheel_pos" value="0 0 0" />
         <xacro:property name="wheel_rot" value="0 0 0" />
+        <xacro:property name="cabinet_pos" value="0 0 0.33" />
     </xacro:if>
     <xacro:if value="${frame == 'long'}">
@@ -23,4 +26,5 @@
         <xacro:property name="wheel_pos" value="0 0 0" />
         <xacro:property name="wheel_rot" value="0 0 0" />
+        <xacro:property name="cabinet_pos" value="0.13 0 0.33" />
     </xacro:if>
     <link name="base_link" />
@@ -68,5 +72,5 @@
         vis_rot="0 0 0" vis_pos="0 0 0"
         joint_type="${joint_typ}">
-        <origin rpy="3.14 0 0" xyz="0.60 0.25 0.10"/>
+        <origin xyz="${wheel_pos}" rpy="${wheel_rot}"/>
     </xacro:argo_wheel>
     <xacro:sick_nanoscan name="lidar_1" parent="base_footprint">
@@ -76,3 +80,13 @@
         <origin rpy="3.14 0 3.14" xyz="-0.60 -0.25 0.10"/>
     </xacro:sick_nanoscan>
+    <xacro:unless value="${arm == ''}">
+        <xacro:include filename="$(find rox_description)/urdf/xacros/cabinet.xacro" />
+        <xacro:cabinet name="cabinet" parent="base_footprint">
+            <origin rpy="0 0 0" xyz="${cabinet_pos}"/>
+        </xacro:cabinet>
+        <!-- <xacro:include filename="$(find rox_description)/urdf/xacros/$(arg arm).xacro" />
+        <xacro:$(arg arm) name="arm" parent="base_footprint">
+            <origin rpy="0 0 0" xyz="0 0 0"/>
+        </xacro:$(arg arm)> -->
+    </xacro:unless>
 </robot>

Commit message: updating the laser scanner

File: rox_description/urdf/rox.urdf.xacro (robot description, xacro)
@@ -15,20 +15,11 @@
     <!-- Assigning Xacro properties -->
     <xacro:if value="${frame == 'short'}">
-        <xacro:property name="caster_pos" value="0 0 0" />
-        <xacro:property name="caster_rot" value="0 0 0" />
-        <xacro:property name="wheel_pos" value="0 0 0" />
-        <xacro:property name="wheel_rot" value="0 0 0" />
-        <xacro:property name="cabinet_pos" value="0 0 0.33" />
+        <xacro:property name="argo_ext" value="0.0" />
     </xacro:if>
     <xacro:if value="${frame == 'long'}">
-        <xacro:property name="caster_pos" value="0 0 0" />
-        <xacro:property name="caster_rot" value="0 0 0" />
-        <xacro:property name="wheel_pos" value="0 0 0" />
-        <xacro:property name="wheel_rot" value="0 0 0" />
-        <xacro:property name="cabinet_pos" value="0.13 0 0.33" />
+        <xacro:property name="argo_ext" value="0.13" />
     </xacro:if>
     <link name="base_link" />
     <xacro:rox_base name="base_footprint"  parent="base_link"
-        vis_rot="0 0 0" vis_pos="0 0 0"
         type="${frame}">
         <origin xyz="0 0 0" rpy="0 0 0" />
@@ -37,51 +28,47 @@
         vis_rot="0 0 0" vis_pos="0 0 0"
         joint_type="${joint_typ}">
-        <origin xyz="${caster_pos}" rpy="${caster_rot}"/>
+        <origin rpy="0 0 ${pi}" xyz="${0.234 + argo_ext} 0.238 0.123"/>
     </xacro:argo_caster>
     <xacro:argo_caster name="caster_front_right" parent="base_footprint"
-        vis_rot="0 0 0" vis_pos="0 0 0"
+        vis_rot="0 0 ${pi}" vis_pos="0 0 0"
         joint_type="${joint_typ}">
-        <origin xyz="${caster_pos}" rpy="${caster_rot}"/>
+        <origin rpy="0 0 0" xyz="${0.234 + argo_ext} -0.238 0.123"/>
     </xacro:argo_caster>
     <xacro:argo_caster name="caster_back_left" parent="base_footprint"
         vis_rot="0 0 0" vis_pos="0 0 0"
         joint_type="${joint_typ}">
-        <origin xyz="${caster_pos}" rpy="${caster_rot}"/>
+        <origin rpy="0 0 ${pi}" xyz="-${0.234 + argo_ext} 0.238 0.123"/>
     </xacro:argo_caster>
     <xacro:argo_caster name="caster_back_right" parent="base_footprint"
-        vis_rot="0 0 0" vis_pos="0 0 0"
+        vis_rot="0 0 ${pi}" vis_pos="0 0 0"
         joint_type="${joint_typ}">
-        <origin xyz="${caster_pos}" rpy="${caster_rot}"/>
+        <origin rpy="0 0 0" xyz="-${0.234 + argo_ext} -0.238 0.123"/>
     </xacro:argo_caster>
-    <xacro:argo_wheel name="wheel_front_left" parent="base_footprint"
-        vis_rot="0 0 0" vis_pos="0 0 0"
+    <xacro:argo_wheel name="wheel_front_left" parent="caster_front_left_link"
         joint_type="${joint_typ}">
-        <origin xyz="${wheel_pos}" rpy="${wheel_rot}"/>
+        <origin xyz="0.0 0.0 -0.07225" rpy="0 0 0" />
     </xacro:argo_wheel>
-    <xacro:argo_wheel name="wheel_front_right" parent="base_footprint"
-        vis_rot="0 0 0" vis_pos="0 0 0"
+    <xacro:argo_wheel name="wheel_front_right" parent="caster_front_right_link"
         joint_type="${joint_typ}">
-        <origin xyz="${wheel_pos}" rpy="${wheel_rot}"/>
+        <origin xyz="0.0 0.0 -0.07225" rpy="0 0 ${pi}" />
     </xacro:argo_wheel>
-    <xacro:argo_wheel name="wheel_back_left" parent="base_footprint"
-        vis_rot="0 0 0" vis_pos="0 0 0"
+    <xacro:argo_wheel name="wheel_back_left" parent="caster_back_left_link"
         joint_type="${joint_typ}">
-        <origin xyz="${wheel_pos}" rpy="${wheel_rot}"/>
+        <origin xyz="0.0 0.0 -0.07225" rpy="0 0 0" />
     </xacro:argo_wheel>
-    <xacro:argo_wheel name="wheel_back_right" parent="base_footprint"
-        vis_rot="0 0 0" vis_pos="0 0 0"
+    <xacro:argo_wheel name="wheel_back_right" parent="caster_back_right_link"
         joint_type="${joint_typ}">
-        <origin xyz="${wheel_pos}" rpy="${wheel_rot}"/>
+        <origin xyz="0.0 0.0 -0.07225" rpy="0 0 ${pi}" />
     </xacro:argo_wheel>
     <xacro:sick_nanoscan name="lidar_1" parent="base_footprint">
-        <origin rpy="3.14 0 0" xyz="0.60 0.25 0.10"/>
+        <origin rpy="${pi} 0 ${pi/4}" xyz="${0.2995 + argo_ext} 0.269 0.19"/>
     </xacro:sick_nanoscan>
     <xacro:sick_nanoscan name="lidar_2" parent="base_footprint">
-        <origin rpy="3.14 0 3.14" xyz="-0.60 -0.25 0.10"/>
+        <origin rpy="${pi} 0 -${pi - pi/4}" xyz="-${0.2995 + argo_ext} -0.269 0.19"/>
     </xacro:sick_nanoscan>
     <xacro:unless value="${arm == ''}">
         <xacro:include filename="$(find rox_description)/urdf/xacros/cabinet.xacro" />
         <xacro:cabinet name="cabinet" parent="base_footprint">
-            <origin rpy="0 0 0" xyz="${cabinet_pos}"/>
+            <origin rpy="0 0 0" xyz="${argo_ext} 0 0.33"/>
         </xacro:cabinet>
         <!-- <xacro:include filename="$(find rox_description)/urdf/xacros/$(arg arm).xacro" />

File: rox_description/urdf/xacros/argo_wheel.xacro (robot description, xacro)
@@ -1,5 +1,5 @@
 <?xml version="1.0"?>
 <robot xmlns:xacro="http://www.ros.org/wiki/xacro" name="rox">
-  <xacro:macro name="argo_wheel" params="name parent *origin vis_rot vis_pos joint_type">
+  <xacro:macro name="argo_wheel" params="name parent *origin joint_type">
    <joint name="${name}_joint" type="${joint_type}">
     <xacro:insert_block name="origin" />
@@ -14,15 +14,15 @@
     <!-- These are not accurate value -->
       <mass value="2" />
-      <origin xyz="0 0 0" rpy="0 0 0" />
+      <origin rpy="0 0 3.14" xyz="0 0.020 0" />
       <inertia ixx="0.00044332" ixy="0" ixz="0" iyy="0.00044332" iyz="0" izz="0.00072" />
     </inertial>
     <visual>
-     <origin xyz="${vis_pos}" rpy="${vis_rot}" />
-     <geometry>
+      <origin rpy="0 0 3.14" xyz="0 0.020 0" />
+      <geometry>
         <mesh filename="package://rox_description/meshes/argo_wheel.dae" scale="0.1 0.1 0.1"/>
-     </geometry>
+      </geometry>
     </visual>
     <collision>
-     <origin xyz="${vis_pos}" rpy="${vis_rot}" />
+     <origin rpy="0 0 3.14" xyz="0 0.020 0" />
      <geometry>
         <mesh filename="package://rox_description/meshes/argo_wheel.dae" scale="0.1 0.1 0.1"/>

File: rox_description/urdf/xacros/frame.xacro (robot description, xacro)
@@ -1,5 +1,5 @@
 <?xml version="1.0"?>
 <robot xmlns:xacro="http://www.ros.org/wiki/xacro" name="rox">
-  <xacro:macro name="rox_base" params="name parent type *origin vis_rot vis_pos">
+  <xacro:macro name="rox_base" params="name parent type *origin">
    <joint name="${name}_joint" type="fixed">
     <xacro:insert_block name="origin" />
@@ -19,5 +19,5 @@
       </inertial>
       <visual>
-        <origin xyz="${vis_pos}" rpy="${vis_rot}" />
+        <origin xyz="0 0 0" rpy="0 0 0" />
         <geometry>
             <mesh filename="package://rox_description/meshes/${type}_frame.dae" scale="0.1 0.1 0.1"/>
@@ -25,5 +25,5 @@
       </visual>
       <collision>
-        <origin xyz="${vis_pos}" rpy="${vis_rot}" />
+        <origin xyz="0 0 0" rpy="0 0 0"/>
         <geometry>
             <mesh filename="package://rox_description/meshes/${type}_frame.dae" scale="0.1 0.1 0.1"/>

File: rox_description/urdf/xacros/sick_nanoscan.xacro (robot description, xacro)
@@ -11,9 +11,9 @@
       <inertial>
       <mass value="0.001"/>
-      <origin rpy="-3.14 0 0" xyz="0 0 0.0"/>
+      <origin rpy="${pi} 0 ${pi/2}" xyz="0 0 0.0"/>
       <inertia ixx="0.0001" ixy="0" ixz="0" iyy="0.000001" iyz="0" izz="0.0001"/>
     </inertial>
     <visual>
-      <origin rpy="-3.14 0 0" xyz="0 0 -0.0"/>
+      <origin rpy="${pi} 0 ${pi/2}" xyz="0 0 -0.02"/>
       <geometry>
         <mesh filename="package://rox_description/meshes/nanoscan_3.dae" scale="0.1 0.1 0.1"/>
@@ -21,5 +21,5 @@
     </visual>
     <collision>
-      <origin rpy="-3.14 0 0" xyz="0 0 -0.0"/>
+      <origin rpy="${pi} 0 ${pi/2}" xyz="0 0 -0.02"/>
       <geometry>
         <mesh filename="package://rox_description/meshes/nanoscan_3.dae" scale="0.1 0.1 0.1"/>

Commit message: user can now select the rox_type

File: rox_description/urdf/rox.urdf.xacro (robot description, xacro)
@@ -3,21 +3,22 @@
     <!-- Xacro Arguments-->
     <xacro:arg name="frame_type" default="short"/>
+    <xacro:arg name="rox_type" default="argo"/>
     <xacro:arg name="joint_type" default="fixed"/>
     <xacro:arg name="arm_type" default=""/>
     <xacro:property name="frame" value="$(arg frame_type)"/>
+    <xacro:property name="rox_typ" default="$(arg rox_type)"/>
     <xacro:property name="joint_typ" value="$(arg joint_type)"/>
     <xacro:property name="arm" value="$(arg arm_type)"/>
     <!-- Include xacro files -->
     <xacro:include filename="$(find rox_description)/urdf/xacros/frame.xacro" />
-    <xacro:include filename="$(find rox_description)/urdf/xacros/argo_caster.xacro" />
-    <xacro:include filename="$(find rox_description)/urdf/xacros/argo_wheel.xacro" />
     <xacro:include filename="$(find rox_description)/urdf/xacros/sick_nanoscan.xacro" />
     <!-- Assigning Xacro properties -->
     <xacro:if value="${frame == 'short'}">
-        <xacro:property name="argo_ext" value="0.0" />
+        <xacro:property name="frame_len" value="0.0" />
     </xacro:if>
     <xacro:if value="${frame == 'long'}">
-        <xacro:property name="argo_ext" value="0.13" />
+        <xacro:property name="frame_len" value="0.13" />
     </xacro:if>
+    <!-- Building the robot from here -->
     <link name="base_link" />
     <xacro:rox_base name="base_footprint"  parent="base_link"
@@ -25,50 +26,32 @@
         <origin xyz="0 0 0" rpy="0 0 0" />
     </xacro:rox_base>
-    <xacro:argo_caster name="caster_front_left" parent="base_footprint"
-        vis_rot="0 0 0" vis_pos="0 0 0"
-        joint_type="${joint_typ}">
-        <origin rpy="0 0 ${pi}" xyz="${0.234 + argo_ext} 0.238 0.123"/>
-    </xacro:argo_caster>
-    <xacro:argo_caster name="caster_front_right" parent="base_footprint"
-        vis_rot="0 0 ${pi}" vis_pos="0 0 0"
-        joint_type="${joint_typ}">
-        <origin rpy="0 0 0" xyz="${0.234 + argo_ext} -0.238 0.123"/>
-    </xacro:argo_caster>
-    <xacro:argo_caster name="caster_back_left" parent="base_footprint"
-        vis_rot="0 0 0" vis_pos="0 0 0"
-        joint_type="${joint_typ}">
-        <origin rpy="0 0 ${pi}" xyz="-${0.234 + argo_ext} 0.238 0.123"/>
-    </xacro:argo_caster>
-    <xacro:argo_caster name="caster_back_right" parent="base_footprint"
-        vis_rot="0 0 ${pi}" vis_pos="0 0 0"
-        joint_type="${joint_typ}">
-        <origin rpy="0 0 0" xyz="-${0.234 + argo_ext} -0.238 0.123"/>
-    </xacro:argo_caster>
-    <xacro:argo_wheel name="wheel_front_left" parent="caster_front_left_link"
-        joint_type="${joint_typ}">
-        <origin xyz="0.0 0.0 -0.07225" rpy="0 0 0" />
-    </xacro:argo_wheel>
-    <xacro:argo_wheel name="wheel_front_right" parent="caster_front_right_link"
-        joint_type="${joint_typ}">
-        <origin xyz="0.0 0.0 -0.07225" rpy="0 0 ${pi}" />
-    </xacro:argo_wheel>
-    <xacro:argo_wheel name="wheel_back_left" parent="caster_back_left_link"
-        joint_type="${joint_typ}">
-        <origin xyz="0.0 0.0 -0.07225" rpy="0 0 0" />
-    </xacro:argo_wheel>
-    <xacro:argo_wheel name="wheel_back_right" parent="caster_back_right_link"
-        joint_type="${joint_typ}">
-        <origin xyz="0.0 0.0 -0.07225" rpy="0 0 ${pi}" />
-    </xacro:argo_wheel>
+    <!-- Argo drives -->
+    <xacro:if value="${rox_typ == 'argo'}">
+        <xacro:include filename="$(find rox_description)/urdf/xacros/argo_drive.xacro" />
+        <xacro:argo_drive parent="base_footprint"/>
+    </xacro:if>
+    <!-- Diff drive -->
+    <!-- Includes both Trike and Diff -->
+    <xacro:if value="${rox_typ == 'diff' or rox_typ == 'trike'}">
+        <xacro:include filename="$(find rox_description)/urdf/xacros/diff_drive.xacro" />
+        <xacro:trike_drive parent="base_footprint"/>
+    </xacro:if>
+    <!-- Meca drive -->
+    <xacro:if value="${rox_typ == 'meca'}">
+        <xacro:include filename="$(find rox_description)/urdf/xacros/meca_drive.xacro" />
+        <xacro:meca_drive parent="base_footprint"/>
+    </xacro:if>
+    <!-- Sensors -->
+    <!-- Laser scanners -->
     <xacro:sick_nanoscan name="lidar_1" parent="base_footprint">
-        <origin rpy="${pi} 0 ${pi/4}" xyz="${0.2995 + argo_ext} 0.269 0.19"/>
+        <origin rpy="${pi} 0 ${pi/4}" xyz="${0.2995 + frame_len} 0.269 0.19"/>
     </xacro:sick_nanoscan>
     <xacro:sick_nanoscan name="lidar_2" parent="base_footprint">
-        <origin rpy="${pi} 0 -${pi - pi/4}" xyz="-${0.2995 + argo_ext} -0.269 0.19"/>
+        <origin rpy="${pi} 0 -${pi - pi/4}" xyz="-${0.2995 + frame_len} -0.269 0.19"/>
     </xacro:sick_nanoscan>
     <xacro:unless value="${arm == ''}">
         <xacro:include filename="$(find rox_description)/urdf/xacros/cabinet.xacro" />
         <xacro:cabinet name="cabinet" parent="base_footprint">
-            <origin rpy="0 0 0" xyz="${argo_ext} 0 0.33"/>
+            <origin rpy="0 0 0" xyz="${frame_len} 0 0.33"/>
         </xacro:cabinet>
         <!-- <xacro:include filename="$(find rox_description)/urdf/xacros/$(arg arm).xacro" />

Commit message: adding modern gazebo support

File: rox_description/urdf/rox.urdf.xacro (robot description, xacro)
@@ -6,8 +6,10 @@
     <xacro:arg name="joint_type" default="fixed"/>
     <xacro:arg name="arm_type" default=""/>
+    <xacro:arg name="sim" default=""/>
     <xacro:property name="frame" value="$(arg frame_type)"/>
     <xacro:property name="rox_typ" default="$(arg rox_type)"/>
     <xacro:property name="joint_typ" value="$(arg joint_type)"/>
     <xacro:property name="arm" value="$(arg arm_type)"/>
+    <xacro:property name="gz" value="$(arg sim)"/>
     <!-- Include xacro files -->
     <xacro:include filename="$(find rox_description)/urdf/xacros/frame.xacro" />
@@ -60,3 +62,8 @@
         </xacro:$(arg arm)> -->
     </xacro:unless>
+    <!-- Check if simulation needs to be used -->
+    <xacro:if value="${gz == 'use_gz'}">
+        <xacro:include filename="$(find rox_description)/urdf/xacros/gazebo.xacro" />
+        <xacro:gazebo_plugins />
+    </xacro:if>
 </robot>
