Commit message: simulation update

File: rox_description/urdf/rox.urdf.xacro (robot description, xacro)
@@ -6,13 +6,23 @@
     <xacro:arg name="joint_type" default="fixed"/>
     <xacro:arg name="arm_type" default=""/>
-    <xacro:arg name="sim" default=""/>
+    <xacro:arg name="use_gz" default="false"/>
+    <xacro:arg name="use_imu" default="false"/>
+    <xacro:arg name="use_d435" default="false"/>
+    <!-- Xacro Properties -->
     <xacro:property name="frame" value="$(arg frame_type)"/>
     <xacro:property name="rox_typ" default="$(arg rox_type)"/>
     <xacro:property name="joint_typ" value="$(arg joint_type)"/>
     <xacro:property name="arm" value="$(arg arm_type)"/>
-    <xacro:property name="gz" value="$(arg sim)"/>
+    <xacro:property name="gz" value="$(arg use_gz)"/>
+    <xacro:property name="use_ur_arm" value="false"/>
+    <xacro:property name="imu" value="$(arg use_imu)"/>
+    <xacro:property name="d435" value="$(arg use_d435)"/>
     <!-- Include xacro files -->
     <xacro:include filename="$(find rox_description)/urdf/xacros/frame.xacro" />
     <xacro:include filename="$(find rox_description)/urdf/xacros/sick_nanoscan.xacro" />
+    <!-- checking if one of the UR arms is used -->
+    <xacro:if value="${arm == 'ur5' or arm == 'ur10' or arm == 'ur5e' or arm == 'ur10e'}">
+        <xacro:property name="use_ur_arm" value="true"/>
+    </xacro:if>
     <!-- Assigning Xacro properties -->
     <xacro:if value="${frame == 'short'}">
@@ -52,4 +62,28 @@
         <origin rpy="${pi} 0 -${pi - pi/4}" xyz="-${0.2995 + frame_len} -0.269 0.19"/>
     </xacro:sick_nanoscan>
+    <!-- IMU -->
+    <xacro:if value="${imu == True}">
+        <link name="imu_link">
+            <inertial>
+                <mass value="0.001" />
+                <origin xyz="0 0 0" rpy="0 0 0" />
+                <inertia ixx="0.0001" ixy="0" ixz="0" iyy="0.000001" iyz="0" izz="0.0001" />
+            </inertial>
+        </link>
+        <joint name="imu_joint" type="fixed">
+            <axis xyz="0 1 0"/>
+            <origin rpy="0 0 0" xyz="-0.052 0.208 0.266"/>
+            <parent link="base_link"/>
+            <child link="imu_link"/>
+        </joint>
+    </xacro:if>
+    <!-- Realsense D435 -->
+    <xacro:if value="${d435 == True}">
+        <xacro:include filename="$(find realsense2_description)/urdf/_d435.urdf.xacro"/>
+        <xacro:sensor_d435 parent="base_link">
+            <origin xyz="0.292 0.0 0.716" rpy="0 0 0"/>
+        </xacro:sensor_d435>
+    </xacro:if>
+    <!-- Lidar -->
     <xacro:unless value="${arm == ''}">
         <xacro:include filename="$(find rox_description)/urdf/xacros/cabinet.xacro" />
@@ -57,11 +91,34 @@
             <origin rpy="0 0 0" xyz="${frame_len} 0 0.33"/>
         </xacro:cabinet>
-        <!-- <xacro:include filename="$(find rox_description)/urdf/xacros/$(arg arm).xacro" />
-        <xacro:$(arg arm) name="arm" parent="base_footprint">
-            <origin rpy="0 0 0" xyz="0 0 0"/>
-        </xacro:$(arg arm)> -->
+        <xacro:if value="${use_ur_arm == True}">
+            <xacro:include filename="$(find ur_description)/urdf/ur_macro.xacro"/>
+            <xacro:arg name="tf_prefix" default="${arm}" />
+            <xacro:arg name="joint_limit_params" default="$(find ur_description)/config/$(arg arm_type)/joint_limits.yaml"/>
+            <xacro:arg name="kinematics_params" default="$(find ur_description)/config/$(arg arm_type)/default_kinematics.yaml"/>
+            <xacro:arg name="physical_params" default="$(find ur_description)/config/$(arg arm_type)/physical_parameters.yaml"/>
+            <xacro:arg name="visual_params" default="$(find ur_description)/config/$(arg arm_type)/visual_parameters.yaml"/>
+            <xacro:arg name="transmission_hw_interface" default=""/>
+            <xacro:arg name="safety_limits" default="false"/>
+            <xacro:arg name="safety_pos_margin" default="0.15"/>
+            <xacro:arg name="safety_k_position" default="20"/>
+            <xacro:arg name="force_abs_paths" default="false" />
+            <xacro:ur_robot name="${arm}"
+                parent="cabinet_link"
+                tf_prefix="$(arg tf_prefix)"
+                joint_limits_parameters_file="$(arg joint_limit_params)"
+                kinematics_parameters_file="$(arg kinematics_params)"
+                physical_parameters_file="$(arg physical_params)"
+                visual_parameters_file="$(arg visual_params)"
+                safety_limits="$(arg safety_limits)"
+                safety_pos_margin="$(arg safety_pos_margin)"
+                safety_k_position="$(arg safety_k_position)"
+                >
+                <!-- position robot in the world -->
+                <origin xyz="0.133 0.0 0.416" rpy="0.0 0.0 -1.5708" />
+            </xacro:ur_robot>
+        </xacro:if>
     </xacro:unless>
     <!-- Check if simulation needs to be used -->
-    <xacro:if value="${gz == 'use_gz'}">
+    <xacro:if value="${gz == True}">
         <xacro:include filename="$(find rox_description)/urdf/xacros/gazebo.xacro" />
         <xacro:gazebo_plugins />

File: rox_description/urdf/xacros/gazebo.xacro (robot description, xacro)
@@ -74,4 +74,13 @@
       </sensor>
     </gazebo>
+    <gazebo reference="imu_link">
+        <sensor name="imu_sensor" type="imu">
+            <ignition_frame_id>imu_link</ignition_frame_id>
+            <update_rate>50</update_rate>
+            <visualize>false</visualize>
+            <topic>imu</topic>
+            <always_on>true</always_on>
+        </sensor>
+    </gazebo>
     <gazebo>
       <plugin filename="ignition-gazebo-odometry-publisher-system"
@@ -80,6 +89,9 @@
           <odom_covariance_topic>odom</odom_covariance_topic>
           <tf_topic>tf</tf_topic>
-          <robot_base_frame>base_footprint</robot_base_frame>
+          <robot_base_frame>base_link</robot_base_frame>
           <odom_publish_frequency>100</odom_publish_frequency>
+      </plugin>
+      <plugin filename="ignition-gazebo-imu-system"
+          name="ignition::gazebo::systems::Imu">
       </plugin>
       <plugin filename="ignition-gazebo-velocity-control-system"

Commit message: adding Pilz PsenScanners to the description

File: rox_description/urdf/rox.urdf.xacro (robot description, xacro)
@@ -5,4 +5,5 @@
     <xacro:arg name="rox_type" default="argo"/>
     <xacro:arg name="joint_type" default="fixed"/>
+    <xacro:arg name="scanner" default="nanoscan"/>
     <xacro:arg name="arm_type" default=""/>
     <xacro:arg name="use_gz" default="false"/>
@@ -13,4 +14,5 @@
     <xacro:property name="rox_typ" default="$(arg rox_type)"/>
     <xacro:property name="joint_typ" value="$(arg joint_type)"/>
+    <xacro:property name="scanner_typ" value="$(arg scanner)"/>
     <xacro:property name="arm" value="$(arg arm_type)"/>
     <xacro:property name="gz" value="$(arg use_gz)"/>
@@ -20,5 +22,8 @@
     <!-- Include xacro files -->
     <xacro:include filename="$(find rox_description)/urdf/xacros/frame.xacro" />
+    <!-- Nanoscan -->
     <xacro:include filename="$(find rox_description)/urdf/xacros/sick_nanoscan.xacro" />
+    <!-- PSenScan -->
+    <xacro:include filename="$(find rox_description)/urdf/xacros/pilz_psenscan.xacro" />
     <!-- checking if one of the UR arms is used -->
     <xacro:if value="${arm == 'ur5' or arm == 'ur10' or arm == 'ur5e' or arm == 'ur10e'}">
@@ -56,10 +61,20 @@
     <!-- Sensors -->
     <!-- Laser scanners -->
-    <xacro:sick_nanoscan name="lidar_1" parent="base_footprint">
-        <origin rpy="${pi} 0 ${pi/4}" xyz="${0.2995 + frame_len} 0.269 0.19"/>
-    </xacro:sick_nanoscan>
-    <xacro:sick_nanoscan name="lidar_2" parent="base_footprint">
-        <origin rpy="${pi} 0 -${pi - pi/4}" xyz="-${0.2995 + frame_len} -0.269 0.19"/>
-    </xacro:sick_nanoscan>
+    <xacro:if value="${scanner_typ == 'nanoscan'}">
+        <xacro:sick_nanoscan name="lidar_1" parent="base_footprint">
+            <origin rpy="${pi} 0 ${pi/4}" xyz="${0.2995 + frame_len} 0.269 0.19"/>
+        </xacro:sick_nanoscan>
+        <xacro:sick_nanoscan name="lidar_2" parent="base_footprint">
+            <origin rpy="${pi} 0 -${pi - pi/4}" xyz="-${0.2995 + frame_len} -0.269 0.19"/>
+        </xacro:sick_nanoscan>
+    </xacro:if>
+    <xacro:if value="${scanner_typ == 'psenscan'}">
+        <xacro:pilz_psenscan name="lidar_1" parent="base_footprint">
+            <origin rpy="${pi} 0 ${pi/4}" xyz="${0.3016 + frame_len} 0.2719 0.191"/>
+        </xacro:pilz_psenscan>
+        <xacro:pilz_psenscan name="lidar_2" parent="base_footprint">
+            <origin rpy="${pi} 0 -${pi - pi/4}" xyz="-${0.3016 + frame_len} -0.2719 0.191"/>
+        </xacro:pilz_psenscan>
+    </xacro:if>
     <!-- IMU -->
     <xacro:if value="${imu == True}">

Commit message: Pilz scanners are added

File: rox_description/urdf/rox.urdf.xacro (robot description, xacro)
@@ -71,8 +71,8 @@
     <xacro:if value="${scanner_typ == 'psenscan'}">
         <xacro:pilz_psenscan name="lidar_1" parent="base_footprint">
-            <origin rpy="${pi} 0 ${pi/4}" xyz="${0.3016 + frame_len} 0.2719 0.191"/>
+            <origin rpy="0 0 ${pi/4}" xyz="${0.3016 + frame_len} 0.2719 0.191"/>
         </xacro:pilz_psenscan>
         <xacro:pilz_psenscan name="lidar_2" parent="base_footprint">
-            <origin rpy="${pi} 0 -${pi - pi/4}" xyz="-${0.3016 + frame_len} -0.2719 0.191"/>
+            <origin rpy="0 0 -${pi - pi/4}" xyz="-${0.3016 + frame_len} -0.2719 0.191"/>
         </xacro:pilz_psenscan>
     </xacro:if>

Commit message: support to the pilz scanner out of the box

File: rox_description/urdf/rox.urdf.xacro (robot description, xacro)
@@ -61,4 +61,5 @@
     <!-- Sensors -->
     <!-- Laser scanners -->
+    <!-- Nanoscans -->
     <xacro:if value="${scanner_typ == 'nanoscan'}">
         <xacro:sick_nanoscan name="lidar_1" parent="base_footprint">
@@ -69,4 +70,13 @@
         </xacro:sick_nanoscan>
     </xacro:if>
+    <xacro:if value="${scanner_typ == 'psenscan'}">
+        <xacro:pilz_psenscan name="lidar_1" parent="base_footprint">
+            <origin rpy="0 0 ${pi/4}" xyz="${0.3016 + frame_len} 0.2719 0.191"/>
+        </xacro:pilz_psenscan>
+        <xacro:pilz_psenscan name="lidar_2" parent="base_footprint">
+            <origin rpy="0 0 -${pi - pi/4}" xyz="-${0.3016 + frame_len} -0.2719 0.191"/>
+        </xacro:pilz_psenscan>
+    </xacro:if>
+    <!-- Pilz -->
     <xacro:if value="${scanner_typ == 'psenscan'}">
         <xacro:pilz_psenscan name="lidar_1" parent="base_footprint">
@@ -100,5 +110,5 @@
         </xacro:sensor_d435>
     </xacro:if>
-    <!-- Lidar -->
+    <!-- arm -->
     <xacro:unless value="${arm == ''}">
         <xacro:include filename="$(find rox_description)/urdf/xacros/cabinet.xacro" />

Commit message: fixes

File: rox_description/urdf/rox.urdf.xacro (robot description, xacro)
@@ -69,12 +69,4 @@
             <origin rpy="${pi} 0 -${pi - pi/4}" xyz="-${0.2995 + frame_len} -0.269 0.19"/>
         </xacro:sick_nanoscan>
-    </xacro:if>
-    <xacro:if value="${scanner_typ == 'psenscan'}">
-        <xacro:pilz_psenscan name="lidar_1" parent="base_footprint">
-            <origin rpy="0 0 ${pi/4}" xyz="${0.3016 + frame_len} 0.2719 0.191"/>
-        </xacro:pilz_psenscan>
-        <xacro:pilz_psenscan name="lidar_2" parent="base_footprint">
-            <origin rpy="0 0 -${pi - pi/4}" xyz="-${0.3016 + frame_len} -0.2719 0.191"/>
-        </xacro:pilz_psenscan>
     </xacro:if>
     <!-- Pilz -->

Commit message: param tuning, model updates and more

File: rox_description/urdf/rox.urdf.xacro (robot description, xacro)
@@ -46,5 +46,5 @@
     <xacro:if value="${rox_typ == 'argo'}">
         <xacro:include filename="$(find rox_description)/urdf/xacros/argo_drive.xacro" />
-        <xacro:argo_drive parent="base_footprint"/>
+        <xacro:argo_drive parent="base_link"/>
     </xacro:if>
     <!-- Diff drive -->
@@ -52,10 +52,11 @@
     <xacro:if value="${rox_typ == 'diff'}">
         <xacro:include filename="$(find rox_description)/urdf/xacros/diff_drive.xacro" />
-        <xacro:trike_drive parent="base_footprint"/>
+        <xacro:trike_drive parent="base_link"/>
     </xacro:if>
     <!-- Trike drive -->
     <xacro:if value="${rox_typ == 'trike'}">
         <xacro:include filename="$(find rox_description)/urdf/xacros/trike_drive.xacro" />
-        <xacro:trike_drive parent="base_footprint"/>
+        <xacro:trike_drive parent="base_link"/>
+        <xacro:property name="frame_len" value="-0.2435" />
     </xacro:if>
     <!-- Sensors -->
@@ -63,17 +64,17 @@
     <!-- Nanoscans -->
     <xacro:if value="${scanner_typ == 'nanoscan'}">
-        <xacro:sick_nanoscan name="lidar_1" parent="base_footprint">
+        <xacro:sick_nanoscan name="lidar_1" parent="base_link">
             <origin rpy="${pi} 0 ${pi/4}" xyz="${0.2995 + frame_len} 0.269 0.19"/>
         </xacro:sick_nanoscan>
-        <xacro:sick_nanoscan name="lidar_2" parent="base_footprint">
-            <origin rpy="${pi} 0 -${pi - pi/4}" xyz="-${0.2995 + frame_len} -0.269 0.19"/>
+        <xacro:sick_nanoscan name="lidar_2" parent="base_link">
+            <origin rpy="${pi} 0 -${pi - pi/4}" xyz="-${0.2995 - frame_len} -0.269 0.19"/>
         </xacro:sick_nanoscan>
     </xacro:if>
     <!-- Pilz -->
     <xacro:if value="${scanner_typ == 'psenscan'}">
-        <xacro:pilz_psenscan name="lidar_1" parent="base_footprint">
+        <xacro:pilz_psenscan name="lidar_1" parent="base_link">
             <origin rpy="0 0 ${pi/4}" xyz="${0.3016 + frame_len} 0.2719 0.191"/>
         </xacro:pilz_psenscan>
-        <xacro:pilz_psenscan name="lidar_2" parent="base_footprint">
+        <xacro:pilz_psenscan name="lidar_2" parent="base_link">
             <origin rpy="0 0 -${pi - pi/4}" xyz="-${0.3016 + frame_len} -0.2719 0.191"/>
         </xacro:pilz_psenscan>

File: rox_description/urdf/xacros/diff_caster.xacro (robot description, xacro)
@@ -2,5 +2,5 @@
 <robot xmlns:xacro="http://www.ros.org/wiki/xacro" name="rox">
   <xacro:macro name="diff_caster" params="name parent *origin vis_rot vis_pos joint_type">
-    <joint name="${name}_joint" type="${joint_type}">
+    <joint name="${name}_joint" type="fixed">
       <xacro:insert_block name="origin" />
       <axis xyz="1 0 0" />
@@ -10,8 +10,8 @@
     <link name="${name}_link" type="wheel">
       <inertial>
-      <!-- These are not accurate value -->
-        <mass value="0.025" />
+        <!-- These are not accurate value -->
+        <mass value="0.5" />
         <origin xyz="${vis_pos}" rpy="${vis_rot}" />
-        <inertia ixx="0.02" ixy="0" ixz="0" iyy="0.0" iyz="0" izz="0.02" />
+        <inertia ixx="0.02" ixy="0" ixz="0" iyy="0.02" iyz="0" izz="0.02" />
       </inertial>
       <visual>
@@ -24,8 +24,8 @@
         <origin xyz="${vis_pos}" rpy="${vis_rot}" />
         <geometry>
-          <mesh filename="package://rox_description/meshes/diff_caster.dae" scale="0.001 0.001 0.001"/>
+          <sphere radius="0.124" />
         </geometry>
       </collision>
-   </link>
+    </link>
   </xacro:macro>
 </robot>

File: rox_description/urdf/xacros/diff_wheel.xacro (robot description, xacro)
@@ -1,8 +1,9 @@
 <?xml version="1.0"?>
 <robot xmlns:xacro="http://www.ros.org/wiki/xacro" name="rox">
-  <xacro:macro name="diff_wheel" params="name parent *origin joint_type">
+  <xacro:macro name="diff_wheel" params="name parent vis_rot vis_pos *origin *axis joint_type">
     <joint name="${name}_joint" type="${joint_type}">
       <xacro:insert_block name="origin" />
-      <axis xyz="1 0 0" />
+      <xacro:insert_block name="axis" />
+      <limit effort="1000.0" lower="-1e+16" upper="1e+16" velocity="100"/>
       <parent link="${parent}" />
       <child link="${name}_link" />
@@ -11,10 +12,10 @@
       <inertial>
       <!-- These are not accurate value -->
-        <mass value="5" />
-        <origin xyz="0 0 0" rpy="0 0 0"/>
-        <inertia ixx="0.02" ixy="0" ixz="0" iyy="0.02" iyz="0" izz="0.02" />
+        <mass value="5.0" />
+        <origin xyz="0 0 0" rpy="0 0 0" />
+        <inertia ixx="0.02888" ixy="0" ixz="0" iyy="0.02888" iyz="0" izz="0.05625" />
       </inertial>
       <visual>
-        <origin rpy="0 0 ${pi/2}" xyz="0 0.0 0" />
+        <origin xyz="${vis_pos}" rpy="${vis_rot}" />
         <geometry>
         <mesh filename="package://rox_description/meshes/diff_wheel.dae" scale="0.001 0.001 0.001"/>
@@ -22,7 +23,7 @@
       </visual>
       <collision>
-        <origin rpy="0 0 0" xyz="0 0.0 0" />
+        <origin xyz="${vis_pos}" rpy="${vis_rot}" />
         <geometry>
-        <mesh filename="package://rox_description/meshes/diff_wheel.dae" scale="0.001 0.001 0.001"/>
+          <sphere radius="0.075" />
         </geometry>
       </collision>

File: rox_description/urdf/xacros/frame.xacro (robot description, xacro)
@@ -11,12 +11,12 @@
       <inertial>
       <!-- These are not accurate value -->
-        <mass value="80.1" />
-        <origin xyz="0 0 0.18" rpy="0.00 0.00 0.0"/>
-        <inertia ixx="3.947" ixy="0.000" ixz="0.000"
-                 iyy="6.249" iyz="0.000"
-                 izz="8.467" />
+        <mass value="8.0" />
+        <origin xyz="-0.243 0 0.18" rpy="0.0 0.0 0.0"/>
+        <inertia ixx="0.299" ixy="0.0" ixz="0.0"
+                 iyy="0.351" iyz="0.0"
+                 izz="0.360" />
       </inertial>
       <visual>
-        <origin xyz="0 0 0" rpy="0 0 0" />
+        <origin xyz="-0.243 0.0 0.0" rpy="0 0 0" />
         <geometry>
           <mesh filename="package://rox_description/meshes/${type}_frame.dae" scale="0.1 0.1 0.1"/>
@@ -24,5 +24,5 @@
       </visual>
       <collision>
-        <origin xyz="0.0 0.0 0.0" rpy="0 0 0"/>
+        <origin xyz="-0.243 0.0 0.0" rpy="0 0 0"/>
         <geometry>
           <mesh filename="package://rox_description/meshes/${type}_frame.dae" scale="0.1 0.1 0.1"/>

File: rox_description/urdf/xacros/gazebo.xacro (robot description, xacro)
@@ -95,10 +95,42 @@
           name="gz::sim::systems::Imu">
       </plugin>
-      <plugin filename="gz-sim-velocity-control-system"
-          name="gz::sim::systems::VelocityControl">
-          <topic>cmd_vel</topic>
-      </plugin>
+      <!-- <xacro:if value="${rox_typ == 'argo'}">
+        <plugin filename="gz-sim-velocity-control-system"
+            name="gz::sim::systems::VelocityControl">
+            <topic>cmd_vel</topic>
+        </plugin>
+      </xacro:if> -->
+      <!-- DiffDrive control for trike and diff -->
+      <xacro:if value="${rox_typ == 'diff' or rox_typ == 'trike'}">
+        <plugin filename="gz-sim-diff-drive-system"
+          name="gz::sim::systems::DiffDrive">
+          <left_joint>wheel_left_joint</left_joint>
+          <right_joint>wheel_right_joint</right_joint>
+          <wheel_separation>0.555</wheel_separation>
+          <wheel_radius>0.075</wheel_radius>
+          <max_linear_acceleration>1</max_linear_acceleration>
+          <min_linear_acceleration>-1</min_linear_acceleration>
+          <max_angular_acceleration>10.0</max_angular_acceleration>
+          <min_angular_acceleration>-10.0</min_angular_acceleration>
+          <max_linear_velocity>2.0</max_linear_velocity>
+          <min_linear_velocity>-2.0</min_linear_velocity>
+          <max_angular_velocity>10.0</max_angular_velocity>
+          <min_angular_velocity>-10.0</min_angular_velocity>
+          <topic>/cmd_vel</topic>
+          <odom_topic>/odom</odom_topic>
+          <tf_topic>/tf</tf_topic>
+          <odom_publish_frequency>50</odom_publish_frequency>
+        </plugin>
+        <plugin
+          filename="gz-sim-joint-state-publisher-system"
+          name="gz::sim::systems::JointStatePublisher">
+          <joint_name>wheel_left_joint</joint_name>
+          <joint_name>wheel_right_joint</joint_name>
+          <topic>joint_states</topic>
+          <update_rate>30</update_rate>
+        </plugin>
+      </xacro:if>
       <plugin filename="gz-sim-sensors-system"
-          name="gz::sim::systems::Sensors">
+        name="gz::sim::systems::Sensors">
       </plugin>
     </gazebo>

File: rox_description/urdf/xacros/trike_drive.xacro (robot description, xacro)
@@ -5,5 +5,5 @@
   <xacro:macro name="trike_drive" params="parent">
     <xacro:diff_caster name="caster_back" parent="${parent}"
-        vis_rot="-${pi/2} 0 -${pi/2}" vis_pos="0 0 0"
+        vis_rot="-${pi/2} 0 -${pi/2}" vis_pos="-0.2435 0 0"
         joint_type="${joint_typ}">
         <origin rpy="0 0 0" xyz="-${0.2785 - 0.045 + frame_len} 0.0 0.124"/>
@@ -11,10 +11,14 @@
     </xacro:diff_caster>
     <xacro:diff_wheel name="wheel_left" parent="${parent}"
+        vis_rot="0 0 0" vis_pos="0 0 0"
         joint_type="${joint_typ}">
-        <origin xyz="0.0 -0.297 0.075" rpy="0 0 0" />
+        <origin xyz="0.0 0.297 0.075" rpy="-${pi/2} 0 0" />
+        <axis xyz="0 0 1" />
     </xacro:diff_wheel>
     <xacro:diff_wheel name="wheel_right" parent="${parent}"
+        vis_rot="0 ${pi} 0" vis_pos="0 0 0"
         joint_type="${joint_typ}">
-        <origin xyz="0.0 0.297 0.075" rpy="0 0 ${pi}" />
+        <origin xyz="0.0 -0.297 0.075" rpy="-${pi/2} 0 0" />
+        <axis xyz="0 0 1" />
     </xacro:diff_wheel>
   </xacro:macro>
