Commit message: Trike support (#28)
* added trike support to rox-desc

* updating Trike description

* param tuning, model updates and more

* comment fixes

File: rox_description/urdf/rox.urdf.xacro (robot description, xacro)
@@ -46,16 +46,17 @@
     <xacro:if value="${rox_typ == 'argo'}">
         <xacro:include filename="$(find rox_description)/urdf/xacros/argo_drive.xacro" />
-        <xacro:argo_drive parent="base_footprint"/>
+        <xacro:argo_drive parent="base_link"/>
     </xacro:if>
     <!-- Diff drive -->
     <!-- Includes both Trike and Diff -->
-    <xacro:if value="${rox_typ == 'diff' or rox_typ == 'trike'}">
+    <xacro:if value="${rox_typ == 'diff'}">
         <xacro:include filename="$(find rox_description)/urdf/xacros/diff_drive.xacro" />
-        <xacro:trike_drive parent="base_footprint"/>
+        <xacro:trike_drive parent="base_link"/>
     </xacro:if>
-    <!-- Meca drive -->
-    <xacro:if value="${rox_typ == 'meca'}">
-        <xacro:include filename="$(find rox_description)/urdf/xacros/meca_drive.xacro" />
-        <xacro:meca_drive parent="base_footprint"/>
+    <!-- Trike drive -->
+    <xacro:if value="${rox_typ == 'trike'}">
+        <xacro:include filename="$(find rox_description)/urdf/xacros/trike_drive.xacro" />
+        <xacro:trike_drive parent="base_link"/>
+        <xacro:property name="frame_len" value="-0.2435" />
     </xacro:if>
     <!-- Sensors -->
@@ -63,17 +64,17 @@
     <!-- Nanoscans -->
     <xacro:if value="${scanner_typ == 'nanoscan'}">
-        <xacro:sick_nanoscan name="lidar_1" parent="base_footprint">
+        <xacro:sick_nanoscan name="lidar_1" parent="base_link">
             <origin rpy="${pi} 0 ${pi/4}" xyz="${0.2995 + frame_len} 0.269 0.19"/>
         </xacro:sick_nanoscan>
-        <xacro:sick_nanoscan name="lidar_2" parent="base_footprint">
-            <origin rpy="${pi} 0 -${pi - pi/4}" xyz="-${0.2995 + frame_len} -0.269 0.19"/>
+        <xacro:sick_nanoscan name="lidar_2" parent="base_link">
+            <origin rpy="${pi} 0 -${pi - pi/4}" xyz="-${0.2995 - frame_len} -0.269 0.19"/>
         </xacro:sick_nanoscan>
     </xacro:if>
     <!-- Pilz -->
     <xacro:if value="${scanner_typ == 'psenscan'}">
-        <xacro:pilz_psenscan name="lidar_1" parent="base_footprint">
+        <xacro:pilz_psenscan name="lidar_1" parent="base_link">
             <origin rpy="0 0 ${pi/4}" xyz="${0.3016 + frame_len} 0.2719 0.191"/>
         </xacro:pilz_psenscan>
-        <xacro:pilz_psenscan name="lidar_2" parent="base_footprint">
+        <xacro:pilz_psenscan name="lidar_2" parent="base_link">
             <origin rpy="0 0 -${pi - pi/4}" xyz="-${0.3016 + frame_len} -0.2719 0.191"/>
         </xacro:pilz_psenscan>

File: rox_description/urdf/xacros/gazebo.xacro (robot description, xacro)
@@ -95,10 +95,43 @@
           name="gz::sim::systems::Imu">
       </plugin>
-      <plugin filename="gz-sim-velocity-control-system"
-          name="gz::sim::systems::VelocityControl">
-          <topic>cmd_vel</topic>
-      </plugin>
+      <!-- For ArgoDrive platforms -->
+      <xacro:if value="${rox_typ == 'argo'}">
+        <plugin filename="gz-sim-velocity-control-system"
+            name="gz::sim::systems::VelocityControl">
+            <topic>cmd_vel</topic>
+        </plugin>
+      </xacro:if>
+      <!-- DiffDrive control for trike and diff -->
+      <xacro:if value="${rox_typ == 'diff' or rox_typ == 'trike'}">
+        <plugin filename="gz-sim-diff-drive-system"
+          name="gz::sim::systems::DiffDrive">
+          <left_joint>wheel_left_joint</left_joint>
+          <right_joint>wheel_right_joint</right_joint>
+          <wheel_separation>0.555</wheel_separation>
+          <wheel_radius>0.075</wheel_radius>
+          <max_linear_acceleration>1</max_linear_acceleration>
+          <min_linear_acceleration>-1</min_linear_acceleration>
+          <max_angular_acceleration>10.0</max_angular_acceleration>
+          <min_angular_acceleration>-10.0</min_angular_acceleration>
+          <max_linear_velocity>2.0</max_linear_velocity>
+          <min_linear_velocity>-2.0</min_linear_velocity>
+          <max_angular_velocity>10.0</max_angular_velocity>
+          <min_angular_velocity>-10.0</min_angular_velocity>
+          <topic>/cmd_vel</topic>
+          <odom_topic>/odom</odom_topic>
+          <tf_topic>/tf</tf_topic>
+          <odom_publish_frequency>50</odom_publish_frequency>
+        </plugin>
+        <plugin
+          filename="gz-sim-joint-state-publisher-system"
+          name="gz::sim::systems::JointStatePublisher">
+          <joint_name>wheel_left_joint</joint_name>
+          <joint_name>wheel_right_joint</joint_name>
+          <topic>joint_states</topic>
+          <update_rate>30</update_rate>
+        </plugin>
+      </xacro:if>
       <plugin filename="gz-sim-sensors-system"
-          name="gz::sim::systems::Sensors">
+        name="gz::sim::systems::Sensors">
       </plugin>
     </gazebo>

Commit message: diff drive fixes

File: rox_description/urdf/rox.urdf.xacro (robot description, xacro)
@@ -52,5 +52,5 @@
     <xacro:if value="${rox_typ == 'diff'}">
         <xacro:include filename="$(find rox_description)/urdf/xacros/diff_drive.xacro" />
-        <xacro:trike_drive parent="base_link"/>
+        <xacro:diff_drive parent="base_link"/>
     </xacro:if>
     <!-- Trike drive -->

File: rox_description/urdf/xacros/diff_drive.xacro (robot description, xacro)
@@ -2,24 +2,42 @@
 <robot xmlns:xacro="http://www.ros.org/wiki/xacro" name="rox">
   <xacro:include filename="$(find rox_description)/urdf/xacros/diff_caster.xacro" />
-  <xacro:include filename="$(find rox_description)/urdf/xacros/diff_fixed.xacro" />
+  <xacro:include filename="$(find rox_description)/urdf/xacros/diff_wheel.xacro" />
   <xacro:macro name="diff_drive" params="parent">
-    <xacro:diff_caster name="caster_wheel_front_left" parent="${parent}">
-        <origin rpy="0 0 ${pi}" xyz="${0.1885 + frame_len} -0.226 0.123"/>
+    <xacro:diff_caster name="caster_wheel_front_left" parent="${parent}"
+        vis_rot="-${pi/2} 0 -${pi/2}" vis_pos="0 0 0"
+        joint_type="fixed">
+        <origin rpy="0 0 0" xyz="${0.2785 + frame_len + 0.045} -0.226 0.124"/>
+        <!-- For the caster position 0.2785 is L3.2 and 0.045 is the Swivel lead -->
     </xacro:diff_caster>
-    <xacro:diff_caster name="caster_wheel_front_right" parent="${parent}">
-        <origin rpy="0 0 0" xyz="${0.1885 + frame_len} 0.226 0.04"/>
+    <xacro:diff_caster name="caster_wheel_front_right" parent="${parent}"
+        vis_rot="-${pi/2} 0 -${pi/2}" vis_pos="0 0 0"
+        joint_type="fixed">
+        <origin rpy="0 0 0" xyz="${0.2785 + frame_len + 0.045} 0.226 0.124"/>
+        <!-- For the caster position 0.2785 is L3.2 and 0.045 is the Swivel lead -->
     </xacro:diff_caster>
-    <xacro:diff_caster name="caster_wheel_back_left" parent="${parent}">
-        <origin rpy="0 0 ${pi}" xyz="-${0.2785 + frame_len} -0.226 0.04"/>
+    <xacro:diff_caster name="caster_wheel_back_left" parent="${parent}"
+        vis_rot="-${pi/2} 0 -${pi/2}" vis_pos="0 0 0"
+        joint_type="fixed">
+        <origin rpy="0 0 0" xyz="-${0.1885 + frame_len + 0.045} -0.226 0.124"/>
+        <!-- For the caster position 0.1885 is L3.2 and 0.045 is the Swivel lead -->
     </xacro:diff_caster>
-    <xacro:diff_caster name="caster_wheel_back_right" parent="${parent}">
-        <origin rpy="0 0 0" xyz="-${0.2785 + frame_len} 0.226 0.04"/>
+    <xacro:diff_caster name="caster_wheel_back_right" parent="${parent}"
+        vis_rot="-${pi/2} 0 -${pi/2}" vis_pos="0 0 0"
+        joint_type="fixed">
+        <origin rpy="0 0 0" xyz="-${0.1885 + frame_len + 0.045} 0.226 0.124"/>
+        <!-- For the caster position 0.1885 is L3.2 and 0.045 is the Swivel lead -->
     </xacro:diff_caster>
-    <xacro:diff_fixed name="drive_wheel_middle_left" parent="${parent}">
-        <origin xyz="0.0 -0.113 0.075" rpy="0 0 0" />
-    </xacro:diff_fixed>
-    <xacro:diff_fixed name="drive_wheel_middle_right" parent="${parent}">
-        <origin xyz="0.0 0.113 0.075" rpy="0 0 ${pi}" />
-    </xacro:diff_fixed>
+    <xacro:diff_wheel name="wheel_left" parent="${parent}"
+        vis_rot="0 0 0" vis_pos="0 0 0"
+        joint_type="${joint_typ}">
+        <origin xyz="0.0 0.297 0.075" rpy="-${pi/2} 0 0" />
+        <axis xyz="0 0 1" />
+    </xacro:diff_wheel>
+    <xacro:diff_wheel name="wheel_right" parent="${parent}"
+        vis_rot="0 ${pi} 0" vis_pos="0 0 0"
+        joint_type="${joint_typ}">
+        <origin xyz="0.0 -0.297 0.075" rpy="-${pi/2} 0 0" />
+        <axis xyz="0 0 1" />
+    </xacro:diff_wheel>
   </xacro:macro>
 </robot>

File: rox_description/urdf/xacros/frame.xacro (robot description, xacro)
@@ -12,5 +12,5 @@
       <!-- These are not accurate value -->
         <mass value="8.0" />
-        <origin xyz="-0.243 0 0.18" rpy="0.0 0.0 0.0"/>
+        <origin xyz="0.0 0 0.18" rpy="0.0 0.0 0.0"/>
         <inertia ixx="0.299" ixy="0.0" ixz="0.0"
                  iyy="0.351" iyz="0.0"
@@ -18,5 +18,5 @@
       </inertial>
       <visual>
-        <origin xyz="-0.243 0.0 0.0" rpy="0 0 0" />
+        <origin xyz="0.0 0.0 0.0" rpy="0 0 0" />
         <geometry>
           <mesh filename="package://rox_description/meshes/${type}_frame.dae" scale="0.1 0.1 0.1"/>
@@ -24,5 +24,5 @@
       </visual>
       <collision>
-        <origin xyz="-0.243 0.0 0.0" rpy="0 0 0"/>
+        <origin xyz="0.0 0.0 0.0" rpy="0 0 0"/>
         <geometry>
           <mesh filename="package://rox_description/meshes/${type}_frame.dae" scale="0.1 0.1 0.1"/>

Commit message: updating the changes for caroline

File: rox_description/urdf/rox.urdf.xacro (robot description, xacro)
@@ -65,8 +65,8 @@
     <xacro:if value="${scanner_typ == 'nanoscan'}">
         <xacro:sick_nanoscan name="lidar_1" parent="base_link">
-            <origin rpy="${pi} 0 ${pi/4}" xyz="${0.2995 + frame_len} 0.269 0.19"/>
+            <origin rpy="${pi} 0 ${pi/4}" xyz="${0.2995 + frame_len} 0.269 0.189"/>
         </xacro:sick_nanoscan>
         <xacro:sick_nanoscan name="lidar_2" parent="base_link">
-            <origin rpy="${pi} 0 -${pi - pi/4}" xyz="-${0.2995 - frame_len} -0.269 0.19"/>
+            <origin rpy="${pi} 0 -${pi - pi/4}" xyz="-${0.2995 - frame_len} -0.269 0.189"/>
         </xacro:sick_nanoscan>
     </xacro:if>

File: rox_description/urdf/xacros/diff_drive.xacro (robot description, xacro)
@@ -7,5 +7,5 @@
         vis_rot="-${pi/2} 0 -${pi/2}" vis_pos="0 0 0"
         joint_type="fixed">
-        <origin rpy="0 0 0" xyz="${0.2785 + frame_len + 0.045} -0.226 0.124"/>
+        <origin rpy="0 0 0" xyz="${0.2945 + frame_len + 0.045} -0.226 0.124"/>
         <!-- For the caster position 0.2785 is L3.2 and 0.045 is the Swivel lead -->
     </xacro:diff_caster>
@@ -13,5 +13,5 @@
         vis_rot="-${pi/2} 0 -${pi/2}" vis_pos="0 0 0"
         joint_type="fixed">
-        <origin rpy="0 0 0" xyz="${0.2785 + frame_len + 0.045} 0.226 0.124"/>
+        <origin rpy="0 0 0" xyz="${0.2945 + frame_len + 0.045} 0.226 0.124"/>
         <!-- For the caster position 0.2785 is L3.2 and 0.045 is the Swivel lead -->
     </xacro:diff_caster>
@@ -19,5 +19,5 @@
         vis_rot="-${pi/2} 0 -${pi/2}" vis_pos="0 0 0"
         joint_type="fixed">
-        <origin rpy="0 0 0" xyz="-${0.1885 + frame_len + 0.045} -0.226 0.124"/>
+        <origin rpy="0 0 0" xyz="-${0.2045 + frame_len + 0.045} -0.226 0.124"/>
         <!-- For the caster position 0.1885 is L3.2 and 0.045 is the Swivel lead -->
     </xacro:diff_caster>
@@ -25,5 +25,5 @@
         vis_rot="-${pi/2} 0 -${pi/2}" vis_pos="0 0 0"
         joint_type="fixed">
-        <origin rpy="0 0 0" xyz="-${0.1885 + frame_len + 0.045} 0.226 0.124"/>
+        <origin rpy="0 0 0" xyz="-${0.2045 + frame_len + 0.045} 0.226 0.124"/>
         <!-- For the caster position 0.1885 is L3.2 and 0.045 is the Swivel lead -->
     </xacro:diff_caster>
@@ -31,5 +31,5 @@
         vis_rot="0 0 0" vis_pos="0 0 0"
         joint_type="${joint_typ}">
-        <origin xyz="0.0 0.297 0.075" rpy="-${pi/2} 0 0" />
+        <origin xyz="0.0 0.317 0.075" rpy="-${pi/2} 0 0" />
         <axis xyz="0 0 1" />
     </xacro:diff_wheel>
@@ -37,5 +37,5 @@
         vis_rot="0 ${pi} 0" vis_pos="0 0 0"
         joint_type="${joint_typ}">
-        <origin xyz="0.0 -0.297 0.075" rpy="-${pi/2} 0 0" />
+        <origin xyz="0.0 -0.317 0.075" rpy="-${pi/2} 0 0" />
         <axis xyz="0 0 1" />
     </xacro:diff_wheel>

Commit message: support for the customized platform

File: rox_description/urdf/rox.urdf.xacro (robot description, xacro)
@@ -75,8 +75,8 @@
   <xacro:if value="${scanner == 'nanoscan'}">
     <xacro:sick_nanoscan name="lidar_1" parent="base_link">
-      <origin rpy="${pi} 0 ${pi/4}" xyz="${0.2995} 0.269 0.189"/>
+      <origin rpy="${pi} 0 ${pi/4}" xyz="${0.579} 0.399 0.288"/>
     </xacro:sick_nanoscan>
     <xacro:sick_nanoscan name="lidar_2" parent="base_link">
-      <origin rpy="${pi} 0 -${pi - pi/4}" xyz="-${0.2995} -0.269 0.189"/>
+      <origin rpy="${pi} 0 -${pi - pi/4}" xyz="-${0.579} -0.399 0.288"/>
     </xacro:sick_nanoscan>
   </xacro:if>
@@ -125,5 +125,5 @@
     <xacro:include filename="$(find rox_description)/urdf/xacros/cabinet.xacro" />
     <xacro:cabinet name="cabinet" parent="base_footprint">
-      <origin rpy="0 0 0" xyz="0 0 0.33"/>
+      <origin rpy="0 0 0" xyz="-0.301 0 0.412"/>
     </xacro:cabinet>
     <!-- Universal Robotics (UR) Arms-->

File: rox_description/urdf/xacros/argo_caster.xacro (robot description, xacro)
@@ -20,5 +20,5 @@
      <origin xyz="${vis_pos}" rpy="${vis_rot}" />
      <geometry>
-        <mesh filename="package://rox_description/meshes/argo_caster.dae" scale="0.001 0.001 0.001"/>
+        <mesh filename="package://rox_description/meshes/argo_caster.dae" scale="0.1 0.1 0.1"/>
      </geometry>
     </visual>
@@ -26,5 +26,5 @@
      <origin xyz="${vis_pos}" rpy="${vis_rot}" />
      <geometry>
-        <mesh filename="package://rox_description/meshes/argo_caster.dae" scale="0.001 0.001 0.001"/>
+        <mesh filename="package://rox_description/meshes/argo_caster.dae" scale="0.1 0.1 0.1"/>
      </geometry>
     </collision>

File: rox_description/urdf/xacros/argo_drive.xacro (robot description, xacro)
@@ -7,36 +7,36 @@
         vis_rot="0 0 0" vis_pos="0 0 0"
         joint_type="${joint_typ}">
-        <origin rpy="0 0 ${pi}" xyz="0.239 0.229 0.123"/>
+        <origin rpy="0 0 ${pi}" xyz="0.519 0.359 0.112"/>
     </xacro:argo_caster>
     <xacro:argo_caster name="caster_front_right" parent="${parent}"
         vis_rot="0 0 ${pi}" vis_pos="0 0 0"
         joint_type="${joint_typ}">
-        <origin rpy="0 0 0" xyz="0.239 -0.229 0.123"/>
+        <origin rpy="0 0 0" xyz="0.519 -0.359 0.112"/>
     </xacro:argo_caster>
     <xacro:argo_caster name="caster_back_left" parent="${parent}"
         vis_rot="0 0 0" vis_pos="0 0 0"
         joint_type="${joint_typ}">
-        <origin rpy="0 0 ${pi}" xyz="-0.239 0.229 0.123"/>
+        <origin rpy="0 0 ${pi}" xyz="-0.519 0.359 0.112"/>
     </xacro:argo_caster>
     <xacro:argo_caster name="caster_back_right" parent="${parent}"
         vis_rot="0 0 ${pi}" vis_pos="0 0 0"
         joint_type="${joint_typ}">
-        <origin rpy="0 0 0" xyz="-0.239 -0.229 0.123"/>
+        <origin rpy="0 0 0" xyz="-0.519 -0.359 0.112"/>
     </xacro:argo_caster>
     <xacro:argo_wheel name="wheel_front_left" parent="caster_front_left_link"
         joint_type="${joint_typ}">
-        <origin xyz="0.0 0.0 -0.07225" rpy="0 0 0" />
+        <origin xyz="0.0 0.0 -0.0" rpy="0 0 0" />
     </xacro:argo_wheel>
     <xacro:argo_wheel name="wheel_front_right" parent="caster_front_right_link"
         joint_type="${joint_typ}">
-        <origin xyz="0.0 0.0 -0.07225" rpy="0 0 ${pi}" />
+        <origin xyz="0.0 0.0 -0.0" rpy="0 0 ${pi}" />
     </xacro:argo_wheel>
     <xacro:argo_wheel name="wheel_back_left" parent="caster_back_left_link"
         joint_type="${joint_typ}">
-        <origin xyz="0.0 0.0 -0.07225" rpy="0 0 0" />
+        <origin xyz="0.0 0.0 -0.0" rpy="0 0 0" />
     </xacro:argo_wheel>
     <xacro:argo_wheel name="wheel_back_right" parent="caster_back_right_link"
         joint_type="${joint_typ}">
-        <origin xyz="0.0 0.0 -0.07225" rpy="0 0 ${pi}" />
+        <origin xyz="0.0 0.0 -0.0" rpy="0 0 ${pi}" />
     </xacro:argo_wheel>
   </xacro:macro>

File: rox_description/urdf/xacros/argo_wheel.xacro (robot description, xacro)
@@ -26,5 +26,5 @@
      <origin rpy="0 0 0" xyz="0 0.0 0" />
       <geometry>
-        <sphere radius="0.05" />
+        <sphere radius="0.112" />
       </geometry>
     </collision>

File: rox_description/urdf/xacros/frame.xacro (robot description, xacro)
@@ -12,5 +12,5 @@
       <!-- These are not accurate value -->
         <mass value="140.0" />
-        <origin xyz="0.0 0 0.18" rpy="0.0 0.0 0.0"/>
+        <origin xyz="0.0 0 0.0" rpy="0.0 0.0 0.0"/>
         <inertia ixx="7.8" ixy="0.0" ixz="0" iyy="7.8" iyz="0.0" izz="7.8"/>
       </inertial>

File: rox_description/urdf/xacros/ur_arm.urdf.xacro (robot description, xacro)
@@ -50,5 +50,5 @@
     >
     <!-- position of arm in the world -->
-    <origin xyz="0.218 0.0 ${arm_height}" rpy="0.0 0.0 3.1415926535897931" />
+    <origin xyz="-0.174 0.0 ${arm_height}" rpy="0.0 0.0 3.1415926535897931" />
   </xacro:ur_robot>
   <!-- this condition is to ensure that ros2_control doesn't interfere with gz_ros2_control during simulation  -->
