Commit message: support for simulation is added

File: rox_description/urdf/rox.urdf.xacro (robot description, xacro)
@@ -7,5 +7,5 @@
 <!-- This is the main URDF file for rox robot -->
   <!-- Xacro Arguments-->
-  <xacro:arg name="use_gz" default="false"/>
+  <xacro:arg name="use_gazebo" default="false"/>
   <xacro:arg name="use_imu" default="false"/>
   <xacro:arg name="use_d435" default="false"/>
@@ -25,5 +25,5 @@
   <xacro:arg name="include_gripper_ros2_control" default="false"/>
   <!-- Xacro Properties -->
-  <xacro:property name="gz" value="$(arg use_gz)"/>
+  <xacro:property name="gazebo" value="$(arg use_gazebo)"/>
   <xacro:property name="imu" value="$(arg use_imu)"/>
   <xacro:property name="d435" value="$(arg use_d435)"/>
@@ -37,4 +37,5 @@
   <!-- Include xacro files -->
   <xacro:include filename="$(find rox_description)/urdf/xacros/frame.xacro" />
+  <xacro:include filename="$(find rox_description)/urdf/xacros/gazebo.xacro" />
   <!-- Nanoscan -->
   <xacro:include filename="$(find rox_description)/urdf/xacros/sick_nanoscan.xacro" />
@@ -75,8 +76,8 @@
   <xacro:if value="${scanner == 'nanoscan'}">
     <xacro:sick_nanoscan name="lidar_1" parent="base_link">
-      <origin rpy="${pi} 0 ${pi/4}" xyz="${0.2995} 0.269 0.189"/>
+      <origin rpy="${pi} 0 ${pi/4}" xyz="${0.579} 0.399 0.288"/>
     </xacro:sick_nanoscan>
     <xacro:sick_nanoscan name="lidar_2" parent="base_link">
-      <origin rpy="${pi} 0 -${pi - pi/4}" xyz="-${0.2995} -0.269 0.189"/>
+      <origin rpy="${pi} 0 -${pi - pi/4}" xyz="-${0.579} -0.399 0.288"/>
     </xacro:sick_nanoscan>
   </xacro:if>
@@ -125,5 +126,5 @@
     <xacro:include filename="$(find rox_description)/urdf/xacros/cabinet.xacro" />
     <xacro:cabinet name="cabinet" parent="base_footprint">
-      <origin rpy="0 0 0" xyz="0 0 0.33"/>
+      <origin rpy="0 0 0" xyz="-0.301 0 0.412"/>
     </xacro:cabinet>
     <!-- Universal Robotics (UR) Arms-->
@@ -161,5 +162,5 @@
           use_mock_hardware="${use_mock}"
           mock_sensor_commands="${use_mock}"
-          sim_gazebo="${gz}"
+          sim_gazebo="${gazebo}"
           include_ros2_control="$(arg include_gripper_ros2_control)"
           >
@@ -178,7 +179,3 @@
   </xacro:unless>
   <!-- Check if simulation needs to be used -->
-  <xacro:if value="${gz == True}">
-    <xacro:include filename="$(find rox_description)/urdf/xacros/gazebo.xacro" />
-    <xacro:gazebo_plugins />
-  </xacro:if>
 </robot>

File: rox_description/urdf/xacros/gazebo.xacro (robot description, xacro)
@@ -1,196 +1,125 @@
 <?xml version="1.0"?>
-<robot xmlns:xacro="http://www.ros.org/wiki/xacro" name="rox">
-  <xacro:macro name="gazebo_plugins">
-    <gazebo reference="lidar_1_link">
-      <sensor name="lidar_1_sensor" type="gpu_lidar">
-        <always_on>true</always_on>
-        <pose>0 0 0 0 0 0</pose>
-        <visualize>false</visualize>
-        <update_rate>10</update_rate>
-        <topic>scan</topic>
-        <!-- Set output to sensor_msgs/LaserScan to get same output type as gazebo_ros_laser -->
-        <output_type>sensor_msgs/LaserScan</output_type>
-        <gz_frame_id>lidar_1_link</gz_frame_id>
-        <lidar>
-          <scan>
-            <horizontal>
-              <samples>720</samples>
-              <resolution>1</resolution>
-              <min_angle>-1.48</min_angle>
-              <max_angle>1.48</max_angle>
-            </horizontal>
-          </scan>
-          <range>
-            <min>0.10</min>
-            <max>30.0</max>
-            <resolution>0.05</resolution>
-          </range>
-          <noise>
-            <type>gaussian</type>
-            <!-- Noise parameters based on published spec for Hokuyo laser
-                    achieving "+-30mm" accuracy at range < 10m.  A mean of 0.0m and
-                    stddev of 0.01m will put 99.7% of samples within 0.03m of the true
-                    reading. -->
-            <mean>0.0</mean>
-            <stddev>0.01</stddev>
-          </noise>
-        </lidar>
-      </sensor>
-    </gazebo>
-    <gazebo reference="lidar_2_link">
-      <sensor name="lidar_2_sensor" type="gpu_lidar">
-        <always_on>true</always_on>
-        <pose>0 0 0 0 0 0</pose>
-        <visualize>false</visualize>
-        <update_rate>10</update_rate>
-        <topic>scan2</topic>
-        <!-- Set output to sensor_msgs/LaserScan to get same output type as gazebo_ros_laser -->
-        <output_type>sensor_msgs/LaserScan</output_type>
-        <gz_frame_id>lidar_2_link</gz_frame_id>
-        <lidar>
-          <scan>
-            <horizontal>
-              <samples>720</samples>
-              <resolution>1</resolution>
-              <min_angle>-1.48</min_angle>
-              <max_angle>1.48</max_angle>
-            </horizontal>
-          </scan>
-          <range>
-            <min>0.10</min>
-            <max>30.0</max>
-            <resolution>0.05</resolution>
-          </range>
-          <noise>
-            <type>gaussian</type>
-            <!-- Noise parameters based on published spec for Hokuyo laser
-                    achieving "+-30mm" accuracy at range < 10m.  A mean of 0.0m and
-                    stddev of 0.01m will put 99.7% of samples within 0.03m of the true
-                    reading. -->
-            <mean>0.0</mean>
-            <stddev>0.01</stddev>
-          </noise>
-        </lidar>
-      </sensor>
-    </gazebo>
-    <gazebo reference="imu_link">
-        <sensor name="imu_sensor" type="imu">
-            <gz_frame_id>imu_link</gz_frame_id>
-            <update_rate>50</update_rate>
-            <visualize>false</visualize>
-            <topic>imu</topic>
-            <always_on>true</always_on>
+<robot name="rox" xmlns:xacro="http://www.ros.org/wiki/xacro">
+  <gazebo reference="lidar_1_link">
+      <sensor type="ray" name="lidar_1_sensor">
+          <pose>0 0 0 0 0 0</pose>
+          <visualize>false</visualize>
+          <update_rate>40</update_rate>
+          <ray>
+            <scan>
+              <horizontal>
+                <samples>720</samples>
+                <resolution>1</resolution>
+                <min_angle>-1.48</min_angle>
+                <max_angle>1.48</max_angle>
+              </horizontal>
+            </scan>
+            <range>
+              <min>0.10</min>
+              <max>30.0</max>
+              <resolution>0.05</resolution>
+            </range>
+            <noise>
+              <type>gaussian</type>
+              <!-- Noise parameters based on published spec for Hokuyo laser
+                   achieving "+-30mm" accuracy at range < 10m.  A mean of 0.0m and
+                   stddev of 0.01m will put 99.7% of samples within 0.03m of the true
+                   reading. -->
+              <mean>0.0</mean>
+              <stddev>0.01</stddev>
+            </noise>
+          </ray>
+          <plugin name="lidar_1" filename="libgazebo_ros_laser.so">
+            <topicName>lidar_1/scan_filtered</topicName>
+            <frameName>lidar_1_link</frameName>
+          </plugin>
         </sensor>
-    </gazebo>
-    <gazebo>
-      <plugin filename="gz-sim-odometry-publisher-system"
-          name="gz::sim::systems::OdometryPublisher">
-          <odom_frame>odom</odom_frame>
-          <odom_covariance_topic>odom</odom_covariance_topic>
-          <tf_topic>tf</tf_topic>
-          <robot_base_frame>base_link</robot_base_frame>
-          <odom_publish_frequency>100</odom_publish_frequency>
+  </gazebo>
+  <gazebo reference="lidar_2_link">
+      <sensor type="ray" name="lidar_2_sensor">
+          <pose>0 0 0 0 0 0</pose>
+          <visualize>false</visualize>
+          <update_rate>40</update_rate>
+          <ray>
+            <scan>
+              <horizontal>
+                <samples>720</samples>
+                <resolution>1</resolution>
+                <min_angle>-1.48</min_angle>
+                <max_angle>1.48</max_angle>
+              </horizontal>
+            </scan>
+            <range>
+              <min>0.10</min>
+              <max>30.0</max>
+              <resolution>0.05</resolution>
+            </range>
+            <noise>
+              <type>gaussian</type>
+              <!-- Noise parameters based on published spec for Hokuyo laser
+                   achieving "+-30mm" accuracy at range < 10m.  A mean of 0.0m and
+                   stddev of 0.01m will put 99.7% of samples within 0.03m of the true
+                   reading. -->
+              <mean>0.0</mean>
+              <stddev>0.01</stddev>
+            </noise>
+          </ray>
+          <plugin name="lidar_2" filename="libgazebo_ros_laser.so">
+            <topicName>lidar_2/scan_filtered</topicName>
+            <frameName>lidar_2_link</frameName>
+          </plugin>
+        </sensor>
+  </gazebo>
+  <!-- Robot controller -->
+ <gazebo>
+    <plugin name="rox_controller" filename="libgazebo_ros_planar_move.so">
+      <commandTopic>cmd_vel</commandTopic>
+      <odometryTopic>odom</odometryTopic>
+      <odometryFrame>odom</odometryFrame>
+      <odometryRate>100.0</odometryRate>
+      <robotBaseFrame>base_link</robotBaseFrame>
+    </plugin>
+  </gazebo>
+  <!-- camera -->
+  <!-->
+  <gazebo reference="camera_link">
+    <sensor type="camera" name="camera1">
+      <update_rate>30.0</update_rate>
+      <camera name="head">
+        <horizontal_fov>1.3962634</horizontal_fov>
+  <image>
+    <width>800</width>
+    <height>800</height>
+    <format>R8G8B8</format>
+  </image>
+        <clip>
+          <near>0.02</near>
+          <far>300</far>
+        </clip>
+        <noise>
+          <type>gaussian</type>
+           Noise is sampled independently per pixel on each frame.
+               That pixel's noise value is added to each of its color
+               channels, which at that point lie in the range [0,1].
+          <mean>0.0</mean>
+          <stddev>0.007</stddev>
+        </noise>
+      </camera>
+      <plugin name="camera_controller" filename="libgazebo_ros_camera.so">
+        <alwaysOn>true</alwaysOn>
+        <updateRate>0.0</updateRate>
+        <cameraName>robot/camera1</cameraName>
+        <imageTopicName>image_raw</imageTopicName>
+        <cameraInfoTopicName>camera_info</cameraInfoTopicName>
+        <frameName>camera_link</frameName>
+        <hackBaseline>0.07</hackBaseline>
+        <distortionK1>0.0</distortionK1>
+        <distortionK2>0.0</distortionK2>
+        <distortionK3>0.0</distortionK3>
+        <distortionT1>0.0</distortionT1>
+        <distortionT2>0.0</distortionT2>
       </plugin>
-      <plugin filename="gz-sim-imu-system"
-          name="gz::sim::systems::Imu">
-      </plugin>
-      <!-- For ArgoDrive platforms -->
-      <xacro:if value="${rox_typ == 'argo' or rox_typ == 'argo-trio'}">
-        <plugin filename="gz-sim-velocity-control-system"
-            name="gz::sim::systems::VelocityControl">
-            <topic>cmd_vel</topic>
-        </plugin>
-      </xacro:if>
-      <!-- DiffDrive control for trike and diff -->
-      <xacro:if value="${rox_typ == 'diff' or rox_typ == 'trike'}">
-        <plugin filename="gz-sim-diff-drive-system"
-          name="gz::sim::systems::DiffDrive">
-          <left_joint>wheel_left_joint</left_joint>
-          <right_joint>wheel_right_joint</right_joint>
-          <wheel_separation>${wheel_separation}</wheel_separation>
-          <wheel_radius>0.075</wheel_radius>
-          <max_linear_acceleration>1</max_linear_acceleration>
-          <min_linear_acceleration>-1</min_linear_acceleration>
-          <max_angular_acceleration>10.0</max_angular_acceleration>
-          <min_angular_acceleration>-10.0</min_angular_acceleration>
-          <max_linear_velocity>2.0</max_linear_velocity>
-          <min_linear_velocity>-2.0</min_linear_velocity>
-          <max_angular_velocity>10.0</max_angular_velocity>
-          <min_angular_velocity>-10.0</min_angular_velocity>
-          <topic>/cmd_vel</topic>
-          <odom_topic>/odom</odom_topic>
-          <tf_topic>/tf</tf_topic>
-          <odom_publish_frequency>50</odom_publish_frequency>
-        </plugin>
-        <plugin
-          filename="gz-sim-joint-state-publisher-system"
-          name="gz::sim::systems::JointStatePublisher">
-          <joint_name>wheel_left_joint</joint_name>
-          <joint_name>wheel_right_joint</joint_name>
-          <topic>joint_states</topic>
-          <update_rate>30</update_rate>
-        </plugin>
-      </xacro:if>
-      <plugin filename="gz-sim-sensors-system"
-        name="gz::sim::systems::Sensors">
-      </plugin>
-    </gazebo>
-    <!-- Gazebo macro for Argo Wheels -->
-    <xacro:macro name="rox_argo_wheel_gazebo_macro" params="name">
-      <gazebo reference="${name}_link">
-        <mu1>0.001</mu1>
-        <mu2>0.001</mu2>
-        <kp>100000.0</kp>
-        <kd>1.0</kd>
-        <minDepth>0.000</minDepth>
-        <fdir1>1 0 0</fdir1>
-      </gazebo>
-    </xacro:macro>
-    <!-- Gazebo macro for Differential Castor Wheels -->
-    <xacro:macro name="rox_caster_wheel_gazebo_macro" params="name">
-      <gazebo reference="${name}_link">
-        <mu1>0.001</mu1>
-        <mu2>0.001</mu2>
-      </gazebo>
-    </xacro:macro>
-    <!-- Gazebo macro for Differential Wheels -->
-    <xacro:macro name="rox_diff_wheel_gazebo_macro" params="name">
-      <gazebo reference="${name}_link">
-        <mu1>1.0</mu1>
-        <mu2>1.0</mu2>
-        <kp>1000000.0</kp>
-        <kd>1.0</kd>
-        <minDepth>0.000</minDepth>
-        <fdir1>1 0 0</fdir1>
-      </gazebo>
-    </xacro:macro>
-    <!--Argo Drive-->
-    <xacro:if value="${rox_typ == 'argo'}">
-      <xacro:rox_argo_wheel_gazebo_macro name="wheel_front_left"/>
-      <xacro:rox_argo_wheel_gazebo_macro name="wheel_front_right"/>
-      <xacro:rox_argo_wheel_gazebo_macro name="wheel_back_left"/>
-      <xacro:rox_argo_wheel_gazebo_macro name="wheel_back_right"/>
-    </xacro:if>
-    <!--Argo Trio Drive-->
-    <xacro:if value="${rox_typ == 'argo-trio'}">
-      <xacro:rox_argo_wheel_gazebo_macro name="wheel_front_left"/>
-      <xacro:rox_argo_wheel_gazebo_macro name="wheel_front_right"/>
-      <xacro:rox_argo_wheel_gazebo_macro name="wheel_back"/>
-    </xacro:if>
-    <!--Diff Drive-->
-    <xacro:if value="${rox_typ == 'diff'}">
-      <xacro:rox_diff_wheel_gazebo_macro name="wheel_left"/>
-      <xacro:rox_diff_wheel_gazebo_macro name="wheel_right"/>
-      <xacro:rox_caster_wheel_gazebo_macro name="caster_wheel_front_left"/>
-      <xacro:rox_caster_wheel_gazebo_macro name="caster_wheel_front_right"/>
-      <xacro:rox_caster_wheel_gazebo_macro name="caster_wheel_back_left"/>
-      <xacro:rox_caster_wheel_gazebo_macro name="caster_wheel_back_right"/>
-    </xacro:if>
-    <!--Trike Drive-->
-    <xacro:if value="${rox_typ == 'trike'}">
-      <xacro:rox_diff_wheel_gazebo_macro name="wheel_left"/>
-      <xacro:rox_diff_wheel_gazebo_macro name="wheel_right"/>
-      <xacro:rox_caster_wheel_gazebo_macro name="caster_back"/>
-    </xacro:if>
-  </xacro:macro>
+    </sensor>
+  </gazebo>
+  <-->
 </robot>

Commit message: added d435 camera support for simulation

File: rox_description/urdf/rox.urdf.xacro (robot description, xacro)
@@ -116,6 +116,7 @@
   <xacro:if value="${d435 == True}">
     <xacro:include filename="$(find realsense2_description)/urdf/_d435.urdf.xacro"/>
-    <xacro:sensor_d435 parent="base_link">
-      <origin xyz="0.292 0.0 0.716" rpy="0 0 0"/>
+    <!-- use_nominal_extrinsics is True for simulation-->
+    <xacro:sensor_d435 parent="base_link" name="d435_camera" use_nominal_extrinsics="true">
+      <origin xyz="0.375 0.0 0.210" rpy="0 ${pi/6} 0"/>
     </xacro:sensor_d435>
   </xacro:if>

File: rox_description/urdf/xacros/gazebo.xacro (robot description, xacro)
@@ -82,4 +82,41 @@
             <always_on>true</always_on>
         </sensor>
+    </gazebo>
+    <gazebo reference="d435_camera_link">
+      <sensor name="camera" type="rgbd_camera">
+        <topic>camera</topic>
+        <gz_frame_id>d435_camera_link</gz_frame_id>
+        <update_rate>30.0</update_rate>
+        <always_on>true</always_on>
+        <visualize>true</visualize>
+        <camera>
+          <optical_frame_id>d435_camera_depth_optical_frame</optical_frame_id>
+          <!-- at 640×480 HFOV is 74 degrees -->
+          <horizontal_fov>1.29154</horizontal_fov>
+          <image>
+            <!--VGA format-->
+            <width>640</width>
+            <height>480</height>
+            <format>R8G8B8</format>
+          </image>
+          <clip>
+            <near>0.05</near>
+            <far>100</far>
+          </clip>
+          <!--d435 min depth range is 0.175m at 640×480
+           maximum range is ~10 m-->
+          <depth_camera>
+            <clip>
+              <near>0.175</near>
+              <far>10</far>
+            </clip>
+          </depth_camera>
+          <noise>
+            <type>gaussian</type>
+            <mean>0</mean>
+            <stddev>0.007</stddev>
+          </noise>
+        </camera>
+      </sensor>
     </gazebo>
     <gazebo>

Commit message: update d435 position

File: rox_description/urdf/rox.urdf.xacro (robot description, xacro)
@@ -118,5 +118,5 @@
     <!-- use_nominal_extrinsics is True for simulation-->
     <xacro:sensor_d435 parent="base_link" name="d435_camera" use_nominal_extrinsics="true">
-      <origin xyz="0.375 0.0 0.210" rpy="0 ${pi/6} 0"/>
+      <origin xyz="0.375 0.0 0.220" rpy="0 0 0"/>
     </xacro:sensor_d435>
   </xacro:if>

Commit message: Added d435 support

File: rox_description/urdf/rox.urdf.xacro (robot description, xacro)
@@ -116,6 +116,7 @@
   <xacro:if value="${d435 == True}">
     <xacro:include filename="$(find realsense2_description)/urdf/_d435.urdf.xacro"/>
-    <xacro:sensor_d435 parent="base_link">
-      <origin xyz="0.292 0.0 0.716" rpy="0 0 0"/>
+    <!-- use_nominal_extrinsics is True for simulation-->
+    <xacro:sensor_d435 parent="base_link" name="d435_camera" use_nominal_extrinsics="true">
+      <origin xyz="0.375 0.0 0.220" rpy="0 0 0"/>
     </xacro:sensor_d435>
   </xacro:if>

File: rox_description/urdf/xacros/gazebo.xacro (robot description, xacro)
@@ -82,4 +82,41 @@
             <always_on>true</always_on>
         </sensor>
+    </gazebo>
+    <gazebo reference="d435_camera_link">
+      <sensor name="camera" type="rgbd_camera">
+        <topic>camera</topic>
+        <gz_frame_id>d435_camera_link</gz_frame_id>
+        <update_rate>30.0</update_rate>
+        <always_on>true</always_on>
+        <visualize>true</visualize>
+        <camera>
+          <optical_frame_id>d435_camera_link</optical_frame_id>
+          <!-- at 640×480 HFOV is 74 degrees -->
+          <horizontal_fov>1.29154</horizontal_fov>
+          <image>
+            <!--VGA format-->
+            <width>640</width>
+            <height>480</height>
+            <format>R8G8B8</format>
+          </image>
+          <clip>
+            <near>0.05</near>
+            <far>100</far>
+          </clip>
+          <!--d435 min depth range is 0.175m at 640×480
+           maximum range is ~10 m-->
+          <depth_camera>
+            <clip>
+              <near>0.175</near>
+              <far>10</far>
+            </clip>
+          </depth_camera>
+          <noise>
+            <type>gaussian</type>
+            <mean>0</mean>
+            <stddev>0.007</stddev>
+          </noise>
+        </camera>
+      </sensor>
     </gazebo>
     <gazebo>

Commit message: adding battery simulation (not yet modelled to our battery types)
Signed-off-by: Adarsh Karan Kesavadas Prasanth <adarshkaran01@gmail.com>

File: rox_description/urdf/rox.urdf.xacro (robot description, xacro)
@@ -10,4 +10,5 @@
   <xacro:arg name="use_imu" default="false"/>
   <xacro:arg name="use_d435" default="false"/>
+  <xacro:arg name="use_battery" default="false"/>
   <xacro:arg name="scanner_type" default="nanoscan"/>
   <xacro:arg name="rox_type" default="argo"/>
@@ -28,4 +29,5 @@
   <xacro:property name="imu" value="$(arg use_imu)"/>
   <xacro:property name="d435" value="$(arg use_d435)"/>
+  <xacro:property name="battery" value="$(arg use_battery)"/>
   <xacro:property name="scanner" value="$(arg scanner_type)"/>
   <xacro:property name="rox_typ" value="$(arg rox_type)"/>

File: rox_description/urdf/xacros/gazebo.xacro (robot description, xacro)
@@ -124,4 +124,35 @@
           name="gz::sim::systems::Imu">
       </plugin>
+      <!-- Battery plugin for all rox platforms -->
+      <xacro:if value="${battery == True}">
+        <plugin filename="gz-sim-linearbatteryplugin-system"
+          name="gz::sim::systems::LinearBatteryPlugin">
+          <!--Li-ion battery spec from LIR18650 datasheet-->
+          <battery_name>linear_battery</battery_name>
+          <voltage>4.2</voltage>
+          <open_circuit_voltage_constant_coef>4.2</open_circuit_voltage_constant_coef>
+          <open_circuit_voltage_linear_coef>-2.0</open_circuit_voltage_linear_coef>
+          <!--Total charge that the battery can hold (Ah)- based on soc overcharging limit-->
+          <initial_charge>0.9</initial_charge>
+          <capacity>1.0 </capacity> <!-- was 50 Ah -->
+          <!-- Internal resistance of the battery (Ohm)-->
+          <resistance>0.05</resistance>
+          <!-- Coefficient for smoothing current-->
+          <smooth_current_tau>2.0</smooth_current_tau>
+          <!-- charging I = c / t, discharging I = P / V,
+          charging I should be > discharging I -->
+          <enable_recharge>true</enable_recharge>
+          <recharge_by_topic>true</recharge_by_topic>
+          <!-- Charging time = capacity/()-->
+          <charging_time>3.0</charging_time>
+          <!-- <soc_threshold>0.51</soc_threshold> not in plugin, deprecated-->
+          <!-- Consumer-specific -->
+          <power_load>2.1</power_load>
+          <!-- <start_draining>true</start_draining> -->
+          <power_draining_topic>/start_power_draining</power_draining_topic>
+          <stop_power_draining_topic>/stop_power_draining</stop_power_draining_topic>
+          <!-- battery_runtime (hours) = <capacity> * <voltage> / <power_load> -->
+        </plugin>
+      </xacro:if>
       <!-- For ArgoDrive platforms -->
       <xacro:if value="${rox_typ == 'argo' or rox_typ == 'argo-trio'}">
