Commit message: added battery type arg, added sample models for agm and lfp battery types
Signed-off-by: Adarsh Karan Kesavadas Prasanth <adarshkaran01@gmail.com>

File: rox_description/urdf/rox.urdf.xacro (robot description, xacro)
@@ -11,4 +11,5 @@
   <xacro:arg name="use_d435" default="false"/>
   <xacro:arg name="use_battery" default="false"/>
+  <xacro:arg name="battery_type" default="lfp"/>
   <xacro:arg name="scanner_type" default="nanoscan"/>
   <xacro:arg name="rox_type" default="argo"/>
@@ -30,4 +31,5 @@
   <xacro:property name="d435" value="$(arg use_d435)"/>
   <xacro:property name="battery" value="$(arg use_battery)"/>
+  <xacro:property name="battery_typ" value="$(arg battery_type)"/>
   <xacro:property name="scanner" value="$(arg scanner_type)"/>
   <xacro:property name="rox_typ" value="$(arg rox_type)"/>

File: rox_description/urdf/xacros/gazebo.xacro (robot description, xacro)
@@ -1,4 +1,6 @@
 <?xml version="1.0"?>
 <robot xmlns:xacro="http://www.ros.org/wiki/xacro" name="rox">
+  <!-- Include battery configuration macro -->
+  <xacro:include filename="$(find rox_description)/urdf/xacros/gazebo_battery.xacro" />
   <xacro:macro name="gazebo_plugins">
     <gazebo reference="lidar_1_link">
@@ -126,32 +128,5 @@
       <!-- Battery plugin for all rox platforms -->
       <xacro:if value="${battery == True}">
-        <plugin filename="gz-sim-linearbatteryplugin-system"
-          name="gz::sim::systems::LinearBatteryPlugin">
-          <!--Li-ion battery spec from LIR18650 datasheet-->
-          <battery_name>linear_battery</battery_name>
-          <voltage>4.2</voltage>
-          <open_circuit_voltage_constant_coef>4.2</open_circuit_voltage_constant_coef>
-          <open_circuit_voltage_linear_coef>-2.0</open_circuit_voltage_linear_coef>
-          <!--Total charge that the battery can hold (Ah)- based on soc overcharging limit-->
-          <initial_charge>0.9</initial_charge>
-          <capacity>1.0 </capacity> <!-- was 50 Ah -->
-          <!-- Internal resistance of the battery (Ohm)-->
-          <resistance>0.05</resistance>
-          <!-- Coefficient for smoothing current-->
-          <smooth_current_tau>2.0</smooth_current_tau>
-          <!-- charging I = c / t, discharging I = P / V,
-          charging I should be > discharging I -->
-          <enable_recharge>true</enable_recharge>
-          <recharge_by_topic>true</recharge_by_topic>
-          <!-- Charging time = capacity/()-->
-          <charging_time>3.0</charging_time>
-          <!-- <soc_threshold>0.51</soc_threshold> not in plugin, deprecated-->
-          <!-- Consumer-specific -->
-          <power_load>2.1</power_load>
-          <!-- <start_draining>true</start_draining> -->
-          <power_draining_topic>/start_power_draining</power_draining_topic>
-          <stop_power_draining_topic>/stop_power_draining</stop_power_draining_topic>
-          <!-- battery_runtime (hours) = <capacity> * <voltage> / <power_load> -->
-        </plugin>
+        <xacro:battery_plugin battery_type="${battery_typ}"/>
       </xacro:if>
       <!-- For ArgoDrive platforms -->

Commit message: fixing the heights of the laserscanner and the cabinet

File: rox_description/urdf/rox.urdf.xacro (robot description, xacro)
@@ -75,8 +75,8 @@
   <xacro:if value="${scanner == 'nanoscan'}">
     <xacro:sick_nanoscan name="lidar_1" parent="base_link">
-      <origin rpy="${pi} 0 ${pi/4}" xyz="${0.579} 0.399 0.288"/>
+      <origin rpy="${pi} 0 ${pi/4}" xyz="${0.579} 0.399 0.2855"/>
     </xacro:sick_nanoscan>
     <xacro:sick_nanoscan name="lidar_2" parent="base_link">
-      <origin rpy="${pi} 0 -${pi - pi/4}" xyz="-${0.579} -0.399 0.288"/>
+      <origin rpy="${pi} 0 -${pi - pi/4}" xyz="-${0.579} -0.399 0.2855"/>
     </xacro:sick_nanoscan>
   </xacro:if>
@@ -125,5 +125,5 @@
     <xacro:include filename="$(find rox_description)/urdf/xacros/cabinet.xacro" />
     <xacro:cabinet name="cabinet" parent="base_footprint">
-      <origin rpy="0 0 0" xyz="-0.301 0 0.412"/>
+      <origin rpy="0 0 0" xyz="-0.301 0 0.4095"/>
     </xacro:cabinet>
     <!-- Universal Robotics (UR) Arms-->

Commit message: fixing the heights of the laserscanner and the cabinet

File: rox_description/urdf/rox.urdf.xacro (robot description, xacro)
@@ -76,8 +76,8 @@
   <xacro:if value="${scanner == 'nanoscan'}">
     <xacro:sick_nanoscan name="lidar_1" parent="base_link">
-      <origin rpy="${pi} 0 ${pi/4}" xyz="${0.579} 0.399 0.288"/>
+      <origin rpy="${pi} 0 ${pi/4}" xyz="${0.579} 0.399 0.2855"/>
     </xacro:sick_nanoscan>
     <xacro:sick_nanoscan name="lidar_2" parent="base_link">
-      <origin rpy="${pi} 0 -${pi - pi/4}" xyz="-${0.579} -0.399 0.288"/>
+      <origin rpy="${pi} 0 -${pi - pi/4}" xyz="-${0.579} -0.399 0.2855"/>
     </xacro:sick_nanoscan>
   </xacro:if>
@@ -126,5 +126,5 @@
     <xacro:include filename="$(find rox_description)/urdf/xacros/cabinet.xacro" />
     <xacro:cabinet name="cabinet" parent="base_footprint">
-      <origin rpy="0 0 0" xyz="-0.301 0 0.412"/>
+      <origin rpy="0 0 0" xyz="-0.301 0 0.4095"/>
     </xacro:cabinet>
     <!-- Universal Robotics (UR) Arms-->

Commit message: added LFP battery model, removed agm option
Signed-off-by: Adarsh Karan Kesavadas Prasanth <adarshkaran01@gmail.com>

File: rox_description/urdf/rox.urdf.xacro (robot description, xacro)
@@ -11,5 +11,4 @@
   <xacro:arg name="use_d435" default="false"/>
   <xacro:arg name="use_battery" default="false"/>
-  <xacro:arg name="battery_type" default="lfp"/>
   <xacro:arg name="scanner_type" default="nanoscan"/>
   <xacro:arg name="rox_type" default="argo"/>
@@ -31,5 +30,4 @@
   <xacro:property name="d435" value="$(arg use_d435)"/>
   <xacro:property name="battery" value="$(arg use_battery)"/>
-  <xacro:property name="battery_typ" value="$(arg battery_type)"/>
   <xacro:property name="scanner" value="$(arg scanner_type)"/>
   <xacro:property name="rox_typ" value="$(arg rox_type)"/>

File: rox_description/urdf/xacros/gazebo.xacro (robot description, xacro)
@@ -128,5 +128,5 @@
       <!-- Battery plugin for all rox platforms -->
       <xacro:if value="${battery == True}">
-        <xacro:battery_plugin battery_type="${battery_typ}"/>
+        <xacro:battery_plugin/>
       </xacro:if>
       <!-- For ArgoDrive platforms -->

File: rox_description/urdf/xacros/gazebo_battery.xacro (robot description, xacro)
@@ -1,62 +1,30 @@
 <?xml version="1.0"?>
 <robot xmlns:xacro="http://www.ros.org/wiki/xacro" name="rox">
-  <!-- Battery configuration macro for different battery types -->
-  <xacro:macro name="battery_plugin" params="battery_type">
-    <!-- LFP (Lithium Iron Phosphate) Battery Configuration -->
-    <xacro:if value="${battery_type == 'lfp'}">
-      <plugin filename="gz-sim-linearbatteryplugin-system"
-        name="gz::sim::systems::LinearBatteryPlugin">
-        <battery_name>linear_battery</battery_name>
-        <voltage>48.0</voltage>
-        <open_circuit_voltage_constant_coef>48.0</open_circuit_voltage_constant_coef>
-        <!-- <open_circuit_voltage_linear_coef>-2.8</open_circuit_voltage_linear_coef> --> <!-- Missing -->
-        <!--Total charge that the battery can hold (Ah)- based on soc overcharging limit-->
-        <initial_charge>${0.9 * 21.0}</initial_charge> <!-- since the plugin internally clamps the SoC to 90% on full charge-->
-        <capacity>21.0</capacity>
-        <!-- Internal resistance of the battery (Ohm)-->
-        <resistance>0.03</resistance> <!-- Missing -->
-        <!-- Coefficient for smoothing current-->
-        <smooth_current_tau>2.0</smooth_current_tau> <!-- Missing -->
-        <!-- charging I = c / t, discharging I = P / V,
-        charging I should be > discharging I -->
-        <enable_recharge>true</enable_recharge>
-        <recharge_by_topic>true</recharge_by_topic>
-        <!-- Charging time = capacity/()-->
-        <charging_time>3.0</charging_time> <!-- Missing -->
-        <!-- Robot power draw (W) -->
-        <power_load>100.0</power_load> <!-- Missing -->
-        <power_draining_topic>/start_power_draining</power_draining_topic>
-        <stop_power_draining_topic>/stop_power_draining</stop_power_draining_topic>
-        <!-- battery_runtime (hours) = <capacity> * <voltage> / <power_load> -->
-      </plugin>
-    </xacro:if>
-    <!-- AGM (Absorbent Glass Mat) Battery Configuration -->
-    <xacro:if value="${battery_type == 'agm'}">
-      <plugin filename="gz-sim-linearbatteryplugin-system"
-        name="gz::sim::systems::LinearBatteryPlugin">
-        <battery_name>linear_battery</battery_name>
-        <voltage>48.0</voltage>
-        <open_circuit_voltage_constant_coef>48.0</open_circuit_voltage_constant_coef>
-        <open_circuit_voltage_linear_coef>-2.2</open_circuit_voltage_linear_coef>
-        <!--Total charge that the battery can hold (Ah)- based on soc overcharging limit-->
-        <initial_charge>${0.9 * 26.0}</initial_charge> <!-- since the plugin internally clamps the SoC to 90% on full charge-->
-        <capacity>26.0</capacity>
-        <!-- Internal resistance of the battery (Ohm)-->
-        <resistance>0.08</resistance> <!-- Missing -->
-        <!-- Coefficient for smoothing current-->
-        <smooth_current_tau>2.0</smooth_current_tau> <!-- Missing -->
-        <!-- charging I = c / t, discharging I = P / V,
-        charging I should be > discharging I -->
-        <enable_recharge>true</enable_recharge>
-        <recharge_by_topic>true</recharge_by_topic>
-        <!-- Charging time = capacity/()-->
-        <charging_time>2.0</charging_time> <!-- Missing -->
-        <!-- Consumer-specific -->
-        <power_load>100.0</power_load> <!-- Missing -->
-        <power_draining_topic>/start_power_draining</power_draining_topic>
-        <stop_power_draining_topic>/stop_power_draining</stop_power_draining_topic>
-        <!-- battery_runtime (hours) = <capacity> * <voltage> / <power_load> -->
-      </plugin>
-    </xacro:if>
+  <!-- Battery configuration macro - LFP (Lithium Iron Phosphate) -->
+  <xacro:macro name="battery_plugin">
+    <plugin filename="gz-sim-linearbatteryplugin-system"
+      name="gz::sim::systems::LinearBatteryPlugin">
+      <battery_name>linear_battery</battery_name>
+      <voltage>54.0</voltage>
+      <open_circuit_voltage_constant_coef>54.0</open_circuit_voltage_constant_coef>
+      <!-- Initial charge set to 100% of capacity -->
+      <initial_charge>26.0</initial_charge>
+      <capacity>26.0</capacity>
+      <!-- Internal resistance of the battery (Ohm) -->
+      <resistance>0.01</resistance>
+      <!-- Coefficient for smoothing current -->
+      <smooth_current_tau>2.0</smooth_current_tau>
+      <!-- charging I = c / t, discharging I = P / V,
+      charging I should be > discharging I -->
+      <enable_recharge>true</enable_recharge>
+      <recharge_by_topic>true</recharge_by_topic>
+      <!-- Charging time: 30 minutes = 0.5 hours -->
+      <charging_time>0.5</charging_time>
+      <!-- Robot power draw (Wh) -->
+      <power_load>260.0</power_load>
+      <power_draining_topic>/start_power_draining</power_draining_topic>
+      <stop_power_draining_topic>/stop_power_draining</stop_power_draining_topic>
+      <!-- battery_runtime (hours) = <capacity> * <voltage> / <power_load> -->
+    </plugin>
   </xacro:macro>
 </robot>

Commit message: URDF flip fix

File: rox_description/urdf/rox.urdf.xacro (robot description, xacro)
@@ -126,5 +126,5 @@
     <xacro:include filename="$(find rox_description)/urdf/xacros/cabinet.xacro" />
     <xacro:cabinet name="cabinet" parent="base_footprint">
-      <origin rpy="0 0 0" xyz="-0.301 0 0.4095"/>
+      <origin rpy="0 0 0" xyz="0.301 0 0.4095"/>
     </xacro:cabinet>
     <!-- Universal Robotics (UR) Arms-->

Commit message: URDF flip fix

File: rox_description/urdf/rox.urdf.xacro (robot description, xacro)
@@ -125,5 +125,5 @@
     <xacro:include filename="$(find rox_description)/urdf/xacros/cabinet.xacro" />
     <xacro:cabinet name="cabinet" parent="base_footprint">
-      <origin rpy="0 0 0" xyz="-0.301 0 0.4095"/>
+      <origin rpy="0 0 0" xyz="0.301 0 0.4095"/>
     </xacro:cabinet>
     <!-- Universal Robotics (UR) Arms-->

File: rox_description/urdf/xacros/ur_arm.urdf.xacro (robot description, xacro)
@@ -50,5 +50,5 @@
     >
     <!-- position of arm in the world -->
-    <origin xyz="-0.174 0.0 ${arm_height}" rpy="0.0 0.0 3.1415926535897931" />
+    <origin xyz="0.174 0.0 ${arm_height}" rpy="0.0 0.0 3.1415926535897931" />
   </xacro:ur_robot>
   <!-- this condition is to ensure that ros2_control doesn't interfere with gz_ros2_control during simulation  -->

Commit message: Issue with ros2control for franka

File: rox_description/urdf/rox.urdf.xacro (robot description, xacro)
@@ -145,4 +145,16 @@
       <xacro:include filename="$(find rox_description)/urdf/xacros/elite_arm.urdf.xacro"/>
     </xacro:if>
+    <!-- Franka Robotics Arms-->
+    <xacro:if value="${arm == 'fr3'}">
+      <!-- Different height for AC arm-->
+      <xacro:if value="${ur_dc == False}">
+        <xacro:property name="arm_height" value="0.376" />
+      </xacro:if>
+      <xacro:if value="${ur_dc == True}">
+        <xacro:property name="arm_height" value="0.276" />
+      </xacro:if>
+      <!-- Include the franka arm -->
+      <xacro:include filename="$(find rox_description)/urdf/xacros/franka_arm.urdf.xacro"/>
+    </xacro:if>
     <!-- add gripper-->
     <xacro:unless value="${gripper == ''}">

Commit message: Fixed review changes + added args for franka ros2control + updates for dc control

File: rox_description/urdf/rox.urdf.xacro (robot description, xacro)
@@ -18,4 +18,5 @@
   <xacro:arg name="gripper_type" default=""/>
   <xacro:arg name="use_ur_dc" default="false"/>
+  <xacro:arg name="use_dc_control_box" default="false"/>
   <xacro:arg name="force_abs_paths" default="false"/>
   <xacro:arg name="simulation_controllers" default=""/>
@@ -33,4 +34,5 @@
   <xacro:property name="arm" value="$(arg arm_type)"/>
   <xacro:property name="ur_dc" value="$(arg use_ur_dc)"/>
+  <xacro:property name="dc_control_box" value="$(arg use_dc_control_box)"/>
   <xacro:property name="gripper" value="$(arg gripper_type)"/>
   <xacro:property name="use_mock" value="$(arg use_mock_hardware)"/>
@@ -148,8 +150,8 @@
     <xacro:if value="${arm == 'fr3'}">
       <!-- Different height for AC arm-->
-      <xacro:if value="${ur_dc == False}">
+      <xacro:if value="${dc_control_box == False}">
         <xacro:property name="arm_height" value="0.376" />
       </xacro:if>
-      <xacro:if value="${ur_dc == True}">
+      <xacro:if value="${dc_control_box == True}">
         <xacro:property name="arm_height" value="0.276" />
       </xacro:if>

File: rox_description/urdf/xacros/franka_arm.urdf.xacro (robot description, xacro)
@@ -21,5 +21,5 @@
     <xacro:arg name="initial_positions_file"
                default="$(find rox_bringup)/configs/franka/initial_joint_positions.yaml"/>
-    <xacro:property name="ur_initial_positions"
+    <xacro:property name="franka_initial_positions"
                     value="${xacro.load_yaml('$(arg initial_positions_file)')}"/>
     <xacro:franka_robot
@@ -36,4 +36,5 @@
       description_pkg="franka_description"
       gazebo_effort="false"
+      use_default_controller_yaml="false"
     />
     <xacro:unless value="$(arg use_gz)">
@@ -47,5 +48,6 @@
           gazebo_effort="false"
           use_fake_hardware="$(arg use_mock_hardware)"
-          fake_sensor_commands="$(arg mock_sensor_commands)"/>
+          fake_sensor_commands="$(arg mock_sensor_commands)"
+          />
       </xacro:if>
     </xacro:unless>

Commit message: Removed ac controller for franka

File: rox_description/urdf/rox.urdf.xacro (robot description, xacro)
@@ -18,5 +18,4 @@
   <xacro:arg name="gripper_type" default=""/>
   <xacro:arg name="use_ur_dc" default="false"/>
-  <xacro:arg name="use_dc_control_box" default="false"/>
   <xacro:arg name="force_abs_paths" default="false"/>
   <xacro:arg name="simulation_controllers" default=""/>
@@ -34,5 +33,4 @@
   <xacro:property name="arm" value="$(arg arm_type)"/>
   <xacro:property name="ur_dc" value="$(arg use_ur_dc)"/>
-  <xacro:property name="dc_control_box" value="$(arg use_dc_control_box)"/>
   <xacro:property name="gripper" value="$(arg gripper_type)"/>
   <xacro:property name="use_mock" value="$(arg use_mock_hardware)"/>
@@ -149,11 +147,5 @@
     <!-- Franka Robotics Arms-->
     <xacro:if value="${arm == 'fr3'}">
-      <!-- Different height for AC arm-->
-      <xacro:if value="${dc_control_box == False}">
-        <xacro:property name="arm_height" value="0.376" />
-      </xacro:if>
-      <xacro:if value="${dc_control_box == True}">
-        <xacro:property name="arm_height" value="0.276" />
-      </xacro:if>
+      <xacro:property name="arm_height" value="0.276" />
       <!-- Include the franka arm -->
       <xacro:include filename="$(find rox_description)/urdf/xacros/franka_arm.urdf.xacro"/>

File: rox_description/urdf/xacros/franka_arm.urdf.xacro (robot description, xacro)
@@ -21,5 +21,5 @@
         value="${xacro.load_yaml('$(find franka_description)/robots/fr3/dynamics.yaml')}" />
   <xacro:if value="${arm == 'fr3'}">
-    <xacro:property name="arm_height" value="0.376"/>
+    <xacro:property name="arm_height" value="0.276"/>
     <xacro:arg name="arm_parent" default="world"/>
     <xacro:arg name="initial_positions_file"
