Commit message: linear-axis Argo variant support for urdf and sim
Signed-off-by: Adarsh Karan Kesavadas Prasanth <adarshkaran01@gmail.com>

File: rox_description/urdf/rox.urdf.xacro (robot description, xacro)
@@ -13,4 +13,5 @@
   <xacro:arg name="rox_type" default="argo"/>
   <xacro:arg name="joint_type" default="fixed"/>
+  <xacro:arg name="enable_linear_axis" default="false"/>
   <!-- Manipulator Arguments-->
   <xacro:arg name="arm_type" default=""/>
@@ -35,4 +36,5 @@
   <xacro:property name="gripper" value="$(arg gripper_type)"/>
   <xacro:property name="use_mock" value="$(arg use_mock_hardware)"/>
+  <xacro:property name="linear_axis" value="$(arg enable_linear_axis)"/>
   <!-- Include xacro files -->
   <xacro:include filename="$(find rox_description)/urdf/xacros/frame.xacro" />
@@ -71,12 +73,31 @@
     <xacro:trike_drive parent="base_link" wheel_separation="${wheel_separation}"/>
   </xacro:if>
+  <!-- Linear axis (EMROX-Argo variant) -->
+  <xacro:if value="${linear_axis == True}">
+    <xacro:include filename="$(find rox_description)/urdf/xacros/linear_axis.xacro"/>
+    <xacro:linear_axis parent="base_link"/>
+  </xacro:if>
+  <!-- Scanner placement -->
+  <!-- Linear-axis variant is wider in X (wheel centers +0.05m per side), Y unchanged. -->
+  <xacro:if value="${linear_axis == True}">
+    <xacro:property name="nanoscan_x" value="0.3495"/>
+    <xacro:property name="nanoscan_y" value="0.2690"/>
+    <xacro:property name="psenscan_x" value="0.3516"/>
+    <xacro:property name="psenscan_y" value="0.2719"/>
+  </xacro:if>
+  <xacro:unless value="${linear_axis == True}">
+    <xacro:property name="nanoscan_x" value="0.2995"/>
+    <xacro:property name="nanoscan_y" value="0.2690"/>
+    <xacro:property name="psenscan_x" value="0.3016"/>
+    <xacro:property name="psenscan_y" value="0.2719"/>
+  </xacro:unless>
   <!-- Laser scanners -->
   <!-- Nanoscans -->
   <xacro:if value="${scanner == 'nanoscan'}">
     <xacro:sick_nanoscan name="lidar_1" parent="base_link">
-      <origin rpy="${pi} 0 ${pi/4}" xyz="${0.2995} 0.269 0.189"/>
+      <origin rpy="${pi} 0 ${pi/4}" xyz="${nanoscan_x} ${nanoscan_y} 0.189"/>
     </xacro:sick_nanoscan>
     <xacro:sick_nanoscan name="lidar_2" parent="base_link">
-      <origin rpy="${pi} 0 -${pi - pi/4}" xyz="-${0.2995} -0.269 0.189"/>
+      <origin rpy="${pi} 0 -${pi - pi/4}" xyz="-${nanoscan_x} -${nanoscan_y} 0.189"/>
     </xacro:sick_nanoscan>
   </xacro:if>
@@ -84,8 +105,8 @@
   <xacro:if value="${scanner == 'psenscan'}">
     <xacro:pilz_psenscan name="lidar_1" parent="base_link">
-      <origin rpy="0 0 ${pi/4}" xyz="${0.3016} 0.2719 0.191"/>
+      <origin rpy="0 0 ${pi/4}" xyz="${psenscan_x} ${psenscan_y} 0.191"/>
     </xacro:pilz_psenscan>
     <xacro:pilz_psenscan name="lidar_2" parent="base_link">
-      <origin rpy="0 0 -${pi - pi/4}" xyz="-${0.3016} -0.2719 0.191"/>
+      <origin rpy="0 0 -${pi - pi/4}" xyz="-${psenscan_x} -${psenscan_y} 0.191"/>
     </xacro:pilz_psenscan>
   </xacro:if>
@@ -121,6 +142,6 @@
     </xacro:sensor_d435>
   </xacro:if>
-  <!-- arm -->
-  <xacro:unless value="${arm == ''}">
+  <!-- arm (excluded when linear axis is enabled — arms are a separate unit) -->
+  <xacro:unless value="${arm == '' or linear_axis == True}">
     <!-- Include cabinet -->
     <xacro:include filename="$(find rox_description)/urdf/xacros/cabinet.xacro" />

File: rox_description/urdf/xacros/argo_caster.xacro (robot description, xacro)
@@ -17,16 +17,32 @@
       <inertia ixx="0.00499743171" ixy="0.00000004464" ixz="-0.00000002245" iyy="0.00499741733" iyz="-0.00000000164" izz="0.00839239692"/>
     </inertial>
-    <visual>
-     <origin xyz="${vis_pos}" rpy="${vis_rot}" />
-     <geometry>
-        <mesh filename="package://rox_description/meshes/argo_caster.dae" scale="0.001 0.001 0.001"/>
-     </geometry>
-    </visual>
-    <collision>
-     <origin xyz="${vis_pos}" rpy="${vis_rot}" />
-     <geometry>
-        <mesh filename="package://rox_description/meshes/argo_caster.dae" scale="0.001 0.001 0.001"/>
-     </geometry>
-    </collision>
+    <xacro:if value="${linear_axis == True}">
+      <visual>
+        <origin xyz="${vis_pos}" rpy="${vis_rot}" />
+        <geometry>
+          <mesh filename="package://rox_description/meshes/linear_axis_argo_caster.dae" scale="0.001 0.001 0.001"/>
+        </geometry>
+      </visual>
+      <collision>
+        <origin xyz="${vis_pos}" rpy="${vis_rot}" />
+        <geometry>
+          <mesh filename="package://rox_description/meshes/linear_axis_argo_caster.dae" scale="0.001 0.001 0.001"/>
+        </geometry>
+      </collision>
+    </xacro:if>
+    <xacro:unless value="${linear_axis == True}">
+      <visual>
+        <origin xyz="${vis_pos}" rpy="${vis_rot}" />
+        <geometry>
+          <mesh filename="package://rox_description/meshes/argo_caster.dae" scale="0.001 0.001 0.001"/>
+        </geometry>
+      </visual>
+      <collision>
+        <origin xyz="${vis_pos}" rpy="${vis_rot}" />
+        <geometry>
+          <mesh filename="package://rox_description/meshes/argo_caster.dae" scale="0.001 0.001 0.001"/>
+        </geometry>
+      </collision>
+    </xacro:unless>
    </link>
   </xacro:macro>

File: rox_description/urdf/xacros/argo_drive.xacro (robot description, xacro)
@@ -4,40 +4,80 @@
   <xacro:include filename="$(find rox_description)/urdf/xacros/argo_wheel.xacro" />
   <xacro:macro name="argo_drive" params="parent">
-    <xacro:argo_caster name="caster_front_left" parent="${parent}"
-        vis_rot="0 0 0" vis_pos="0 0 0"
-        joint_type="${joint_typ}">
-        <origin rpy="0 0 ${pi}" xyz="0.239 0.229 0.123"/>
-    </xacro:argo_caster>
-    <xacro:argo_caster name="caster_front_right" parent="${parent}"
-        vis_rot="0 0 ${pi}" vis_pos="0 0 0"
-        joint_type="${joint_typ}">
-        <origin rpy="0 0 0" xyz="0.239 -0.229 0.123"/>
-    </xacro:argo_caster>
-    <xacro:argo_caster name="caster_back_left" parent="${parent}"
-        vis_rot="0 0 0" vis_pos="0 0 0"
-        joint_type="${joint_typ}">
-        <origin rpy="0 0 ${pi}" xyz="-0.239 0.229 0.123"/>
-    </xacro:argo_caster>
-    <xacro:argo_caster name="caster_back_right" parent="${parent}"
-        vis_rot="0 0 ${pi}" vis_pos="0 0 0"
-        joint_type="${joint_typ}">
-        <origin rpy="0 0 0" xyz="-0.239 -0.229 0.123"/>
-    </xacro:argo_caster>
-    <xacro:argo_wheel name="wheel_front_left" parent="caster_front_left_link"
-        joint_type="${joint_typ}">
-        <origin xyz="0.0 0.0 -0.07225" rpy="0 0 0" />
-    </xacro:argo_wheel>
-    <xacro:argo_wheel name="wheel_front_right" parent="caster_front_right_link"
-        joint_type="${joint_typ}">
-        <origin xyz="0.0 0.0 -0.07225" rpy="0 0 ${pi}" />
-    </xacro:argo_wheel>
-    <xacro:argo_wheel name="wheel_back_left" parent="caster_back_left_link"
-        joint_type="${joint_typ}">
-        <origin xyz="0.0 0.0 -0.07225" rpy="0 0 0" />
-    </xacro:argo_wheel>
-    <xacro:argo_wheel name="wheel_back_right" parent="caster_back_right_link"
-        joint_type="${joint_typ}">
-        <origin xyz="0.0 0.0 -0.07225" rpy="0 0 ${pi}" />
-    </xacro:argo_wheel>
+    <xacro:if value="${linear_axis == True}">
+      <xacro:argo_caster name="caster_front_left" parent="${parent}"
+          vis_rot="0 0 0" vis_pos="-0.289 -0.194 -0.122774"
+          joint_type="${joint_typ}">
+          <origin rpy="0 0 0" xyz="0.289 0.194 0.123"/>
+      </xacro:argo_caster>
+      <xacro:argo_caster name="caster_front_right" parent="${parent}"
+          vis_rot="0 0 ${pi}" vis_pos="0.289 0.194 -0.122774"
+          joint_type="${joint_typ}">
+          <origin rpy="0 0 0" xyz="0.289 -0.194 0.123"/>
+      </xacro:argo_caster>
+      <xacro:argo_caster name="caster_back_left" parent="${parent}"
+          vis_rot="0 0 0" vis_pos="-0.289 -0.194 -0.122774"
+          joint_type="${joint_typ}">
+          <origin rpy="0 0 0" xyz="-0.289 0.194 0.123"/>
+      </xacro:argo_caster>
+      <xacro:argo_caster name="caster_back_right" parent="${parent}"
+          vis_rot="0 0 ${pi}" vis_pos="0.289 0.194 -0.122774"
+          joint_type="${joint_typ}">
+          <origin rpy="0 0 0" xyz="-0.289 -0.194 0.123"/>
+      </xacro:argo_caster>
+      <xacro:argo_wheel name="wheel_front_left" parent="caster_front_left_link"
+          joint_type="${joint_typ}">
+          <origin xyz="0.0 0.035 -0.07225" rpy="0 0 0" />
+      </xacro:argo_wheel>
+      <xacro:argo_wheel name="wheel_front_right" parent="caster_front_right_link"
+          joint_type="${joint_typ}">
+          <origin xyz="0.0 -0.035 -0.07225" rpy="0 0 ${pi}" />
+      </xacro:argo_wheel>
+      <xacro:argo_wheel name="wheel_back_left" parent="caster_back_left_link"
+          joint_type="${joint_typ}">
+          <origin xyz="0.0 0.035 -0.07225" rpy="0 0 0" />
+      </xacro:argo_wheel>
+      <xacro:argo_wheel name="wheel_back_right" parent="caster_back_right_link"
+          joint_type="${joint_typ}">
+          <origin xyz="0.0 -0.035 -0.07225" rpy="0 0 ${pi}" />
+      </xacro:argo_wheel>
+    </xacro:if>
+    <xacro:unless value="${linear_axis == True}">
+      <xacro:argo_caster name="caster_front_left" parent="${parent}"
+          vis_rot="0 0 0" vis_pos="0 0 0"
+          joint_type="${joint_typ}">
+          <origin rpy="0 0 ${pi}" xyz="0.239 0.229 0.123"/>
+      </xacro:argo_caster>
+      <xacro:argo_caster name="caster_front_right" parent="${parent}"
+          vis_rot="0 0 ${pi}" vis_pos="0 0 0"
+          joint_type="${joint_typ}">
+          <origin rpy="0 0 0" xyz="0.239 -0.229 0.123"/>
+      </xacro:argo_caster>
+      <xacro:argo_caster name="caster_back_left" parent="${parent}"
+          vis_rot="0 0 0" vis_pos="0 0 0"
+          joint_type="${joint_typ}">
+          <origin rpy="0 0 ${pi}" xyz="-0.239 0.229 0.123"/>
+      </xacro:argo_caster>
+      <xacro:argo_caster name="caster_back_right" parent="${parent}"
+          vis_rot="0 0 ${pi}" vis_pos="0 0 0"
+          joint_type="${joint_typ}">
+          <origin rpy="0 0 0" xyz="-0.239 -0.229 0.123"/>
+      </xacro:argo_caster>
+      <xacro:argo_wheel name="wheel_front_left" parent="caster_front_left_link"
+          joint_type="${joint_typ}">
+          <origin xyz="0.0 0.0 -0.07225" rpy="0 0 0" />
+      </xacro:argo_wheel>
+      <xacro:argo_wheel name="wheel_front_right" parent="caster_front_right_link"
+          joint_type="${joint_typ}">
+          <origin xyz="0.0 0.0 -0.07225" rpy="0 0 ${pi}" />
+      </xacro:argo_wheel>
+      <xacro:argo_wheel name="wheel_back_left" parent="caster_back_left_link"
+          joint_type="${joint_typ}">
+          <origin xyz="0.0 0.0 -0.07225" rpy="0 0 0" />
+      </xacro:argo_wheel>
+      <xacro:argo_wheel name="wheel_back_right" parent="caster_back_right_link"
+          joint_type="${joint_typ}">
+          <origin xyz="0.0 0.0 -0.07225" rpy="0 0 ${pi}" />
+      </xacro:argo_wheel>
+    </xacro:unless>
   </xacro:macro>
 </robot>

File: rox_description/urdf/xacros/argo_wheel.xacro (robot description, xacro)
@@ -17,10 +17,20 @@
     <inertia ixx="0.11042056" ixy="0.0" ixz="0.0" iyy="0.11042056" iyz="0.0" izz="0.11042056"/>
     </inertial>
-    <visual>
-      <origin rpy="0 0 3.14" xyz="0 0.0 0" />
-      <geometry>
-        <mesh filename="package://rox_description/meshes/argo_wheel.dae" scale="0.1 0.1 0.1"/>
-      </geometry>
-    </visual>
+    <xacro:if value="${linear_axis == True}">
+      <visual>
+        <origin rpy="0 0 ${pi}" xyz="0.289 0.229 -0.050" />
+        <geometry>
+          <mesh filename="package://rox_description/meshes/linear_axis_argo_wheel.dae" scale="0.001 0.001 0.001"/>
+        </geometry>
+      </visual>
+    </xacro:if>
+    <xacro:unless value="${linear_axis == True}">
+      <visual>
+        <origin rpy="0 0 ${pi}" xyz="0 0.0 0" />
+        <geometry>
+          <mesh filename="package://rox_description/meshes/argo_wheel.dae" scale="0.1 0.1 0.1"/>
+        </geometry>
+      </visual>
+    </xacro:unless>
     <collision>
      <origin rpy="0 0 0" xyz="0 0.0 0" />

File: rox_description/urdf/xacros/frame.xacro (robot description, xacro)
@@ -18,5 +18,10 @@
         <origin xyz="0.0 0.0 0.0" rpy="0 0 0" />
         <geometry>
-          <mesh filename="package://rox_description/meshes/short_frame.dae" scale="0.1 0.1 0.1"/>
+          <xacro:if value="${linear_axis == True}">
+            <mesh filename="package://rox_description/meshes/linear_axis_frame.dae" scale="0.001 0.001 0.001"/>
+          </xacro:if>
+          <xacro:unless value="${linear_axis == True}">
+            <mesh filename="package://rox_description/meshes/short_frame.dae" scale="0.1 0.1 0.1"/>
+          </xacro:unless>
         </geometry>
       </visual>
@@ -24,5 +29,10 @@
         <origin xyz="0.0 0.0 0.0" rpy="0 0 0"/>
         <geometry>
-          <mesh filename="package://rox_description/meshes/short_frame.dae" scale="0.1 0.1 0.1"/>
+          <xacro:if value="${linear_axis == True}">
+            <mesh filename="package://rox_description/meshes/linear_axis_frame.dae" scale="0.001 0.001 0.001"/>
+          </xacro:if>
+          <xacro:unless value="${linear_axis == True}">
+            <mesh filename="package://rox_description/meshes/short_frame.dae" scale="0.1 0.1 0.1"/>
+          </xacro:unless>
         </geometry>
       </collision>

Commit message: separated linear axis sim controllers
Signed-off-by: Adarsh Karan Kesavadas Prasanth <adarshkaran01@gmail.com>

File: rox_description/urdf/rox.urdf.xacro (robot description, xacro)
@@ -21,4 +21,5 @@
   <xacro:arg name="force_abs_paths" default="false"/>
   <xacro:arg name="simulation_controllers" default=""/>
+  <xacro:arg name="linear_axis_simulation_controllers" default=""/>
   <xacro:arg name="use_mock_hardware" default="false" />
   <xacro:arg name="mock_sensor_commands" default="false" />

File: rox_description/urdf/xacros/linear_axis.xacro (robot description, xacro)
@@ -7,4 +7,10 @@
 <robot xmlns:xacro="http://www.ros.org/wiki/xacro" name="rox">
   <xacro:macro name="linear_axis" params="parent">
+    <xacro:if value="${gz == True}">
+      <xacro:property name="linear_axis_effort_limit" value="500.0"/>
+    </xacro:if>
+    <xacro:unless value="${gz == True}">
+      <xacro:property name="linear_axis_effort_limit" value="54.0"/>
+    </xacro:unless>
     <!-- Linear-axis cabinet/dummy body -->
     <!-- All EMROX meshes share one CAD frame, so identity aligns naturally. -->
@@ -89,5 +95,5 @@
       <origin xyz="0 0 0" rpy="0 0 0"/>
       <!-- Travel: 888mm derived from spec (1417mm column top - 529mm base top) -->
-      <limit lower="0.0" upper="0.888" effort="54.0" velocity="0.15"/>
+      <limit lower="0.0" upper="0.888" effort="${linear_axis_effort_limit}" velocity="0.15"/>
       <parent link="linear_axis_fixed_link"/>
       <child link="linear_axis_slide_link"/>
@@ -126,5 +132,4 @@
         <joint name="linear_axis_slide_joint">
           <command_interface name="position"/>
-          <command_interface name="velocity"/>
           <state_interface name="position">
             <param name="initial_value">0.0</param>
@@ -135,5 +140,5 @@
       <gazebo>
         <plugin name="gz_ros2_control::GazeboSimROS2ControlPlugin" filename="libgz_ros2_control-system">
-          <parameters>$(arg simulation_controllers)</parameters>
+          <parameters>$(arg linear_axis_simulation_controllers)</parameters>
         </plugin>
       </gazebo>
