Commit message: fixes to the URDF

File: rox_description/urdf/xacros/ur_arm.urdf.xacro (robot description, xacro)
@@ -9,17 +9,9 @@
   <xacro:include filename="$(find ur_robot_driver)/urdf/ur.ros2_control.xacro"/>
   <xacro:include filename="$(find ur_description)/urdf/inc/ur_transmissions.xacro"/>
-  <!-- Set use_gz = true for simulation -->
-  <xacro:arg name="use_gz" default="false"/>
-  <xacro:arg name="include_arm_ros2_control" default="false"/>
-  <!-- arm parameters -->
-  <xacro:arg name="arm_type" default="ur10"/>
-  <xacro:property name="arm_height" default="0.376" />
-  <xacro:arg name="arm_parent" default="world"/>
   <!-- UR arm parameters -->
-  <xacro:arg name="tf_prefix" default="$(arg arm_type)" />
-  <xacro:arg name="joint_limit_params" default="$(find ur_description)/config/$(arg arm_type)/joint_limits.yaml"/>
-  <xacro:arg name="kinematics_params" default="$(find ur_description)/config/$(arg arm_type)/default_kinematics.yaml"/>
-  <xacro:arg name="physical_params" default="$(find ur_description)/config/$(arg arm_type)/physical_parameters.yaml"/>
-  <xacro:arg name="visual_params" default="$(find ur_description)/config/$(arg arm_type)/visual_parameters.yaml"/>
+  <xacro:arg name="joint_limit_params" default="$(find ur_description)/config/ur10/joint_limits.yaml"/>
+  <xacro:arg name="kinematics_params" default="$(find ur_description)/config/ur10/default_kinematics.yaml"/>
+  <xacro:arg name="physical_params" default="$(find ur_description)/config/ur10/physical_parameters.yaml"/>
+  <xacro:arg name="visual_params" default="$(find ur_description)/config/ur10/visual_parameters.yaml"/>
   <xacro:arg name="transmission_hw_interface" default="hardware_interface/PositionJointInterface"/>
   <xacro:arg name="safety_limits" default="false"/>
@@ -30,102 +22,83 @@
   <!-- When using gazebo simulations absolute paths are necessary -->
   <xacro:arg name="force_abs_paths" default="false" />
-  <!-- parse initial positions as a dictionary -->
-  <xacro:property
-    name="ur_initial_positions"
-    value="${xacro.load_yaml('$(arg initial_positions_file)')}"
-    />
-  <!-- create arm from macro-->
-  <xacro:ur_robot
-    name="$(arg arm_type)"
-    parent="$(arg arm_parent)"
-    tf_prefix="$(arg tf_prefix)"
-    joint_limits_parameters_file="$(arg joint_limit_params)"
-    kinematics_parameters_file="$(arg kinematics_params)"
-    physical_parameters_file="$(arg physical_params)"
-    visual_parameters_file="$(arg visual_params)"
-    safety_limits="$(arg safety_limits)"
-    safety_pos_margin="$(arg safety_pos_margin)"
-    safety_k_position="$(arg safety_k_position)"
-    force_abs_paths="$(arg force_abs_paths)"
-    >
-    <!-- position of arm in the world -->
-    <origin xyz="0.218 0.0 ${arm_height}" rpy="0.0 0.0 3.1415926535897931" />
-  </xacro:ur_robot>
-  <!-- this condition is to ensure that ros2_control doesn't interfere with gz_ros2_control during simulation  -->
-  <xacro:unless value="$(arg use_gz)">
-    <xacro:if value="$(arg include_arm_ros2_control)">
-      <!-- ros2_control related parameters -->
-      <xacro:arg name="headless_mode" default="false" />
-      <xacro:arg name="robot_ip" default="192.168.1.102" />
-      <xacro:arg name="script_filename" default="$(find ur_client_library)/resources/external_control.urscript"/>
-      <xacro:arg name="output_recipe_filename" default="$(find ur_robot_driver)/resources/rtde_output_recipe.txt"/>
-      <xacro:arg name="input_recipe_filename" default="$(find ur_robot_driver)/resources/rtde_input_recipe.txt"/>
-      <xacro:arg name="reverse_ip" default="0.0.0.0"/>
-      <xacro:arg name="script_command_port" default="50004"/>
-      <xacro:arg name="reverse_port" default="50001"/>
-      <xacro:arg name="script_sender_port" default="50002"/>
-      <xacro:arg name="trajectory_port" default="50003"/>
-      <!-- tool communication related parameters-->
-      <xacro:arg name="use_tool_communication" default="false" />
-      <xacro:arg name="tool_voltage" default="0" />
-      <xacro:arg name="tool_parity" default="0" />
-      <xacro:arg name="tool_baud_rate" default="115200" />
-      <xacro:arg name="tool_stop_bits" default="1" />
-      <xacro:arg name="tool_rx_idle_chars" default="1.5" />
-      <xacro:arg name="tool_tx_idle_chars" default="3.5" />
-      <xacro:arg name="tool_device_name" default="/tmp/ttyUR" />
-      <xacro:arg name="tool_tcp_port" default="54321" />
-      <xacro:arg name="use_mock_hardware" default="false" />
-      <xacro:arg name="mock_sensor_commands" default="false" />
-      <xacro:ur_ros2_control
-        name="$(arg arm_type)"
-        tf_prefix="$(arg tf_prefix)"
-        kinematics_parameters_file="$(arg kinematics_params)"
-        transmission_hw_interface="$(arg transmission_hw_interface)"
-        headless_mode="$(arg headless_mode)"
-        initial_positions="${ur_initial_positions}"
-        use_tool_communication="$(arg use_tool_communication)"
-        tool_voltage="$(arg tool_voltage)"
-        tool_parity="$(arg tool_parity)"
-        tool_baud_rate="$(arg tool_baud_rate)"
-        tool_stop_bits="$(arg tool_stop_bits)"
-        tool_rx_idle_chars="$(arg tool_rx_idle_chars)"
-        tool_tx_idle_chars="$(arg tool_tx_idle_chars)"
-        tool_device_name="$(arg tool_device_name)"
-        tool_tcp_port="$(arg tool_tcp_port)"
-        robot_ip="$(arg robot_ip)"
-        script_filename="$(arg script_filename)"
-        output_recipe_filename="$(arg output_recipe_filename)"
-        input_recipe_filename="$(arg input_recipe_filename)"
-        reverse_ip="$(arg reverse_ip)"
-        script_command_port="$(arg script_command_port)"
-        reverse_port="$(arg reverse_port)"
-        script_sender_port="$(arg script_sender_port)"
-        trajectory_port="$(arg trajectory_port)"
-        use_mock_hardware="$(arg use_mock_hardware)"
-        mock_sensor_commands="$(arg mock_sensor_commands)"
-        />
-    </xacro:if>
-  </xacro:unless>
-  <!-- If gz simulation is used -->
-  <xacro:if value="$(arg use_gz)">
-    <!-- simulation controllers will be passed from launch file after substitutions -->
-    <xacro:arg name="simulation_controllers" default=""/>
-    <gazebo reference="$(arg arm_parent)">
-    </gazebo>
-    <gazebo>
-      <plugin name="gz_ros2_control::GazeboSimROS2ControlPlugin" filename="libgz_ros2_control-system">
-        <parameters>$(arg simulation_controllers)</parameters>
-        <!-- <controller_manager_node_name>$(arg tf_prefix)controller_manager</controller_manager_node_name> -->
-      </plugin>
-    </gazebo>
-    <!-- ros2 control instance -->
-    <xacro:include filename="$(find ur_simulation_gz)/urdf/ur_gz.ros2_control.xacro" />
-    <xacro:ur_ros2_control
-      name="$(arg arm_type)"
-      tf_prefix="$(arg tf_prefix)"
-      transmission_hw_interface="$(arg transmission_hw_interface)"
-      initial_positions="${ur_initial_positions}"
+  <!-- ros2_control related parameters -->
+  <xacro:arg name="headless_mode" default="false" />
+  <xacro:arg name="script_filename" default="$(find ur_client_library)/resources/external_control.urscript"/>
+  <xacro:arg name="output_recipe_filename" default="$(find ur_robot_driver)/resources/rtde_output_recipe.txt"/>
+  <xacro:arg name="input_recipe_filename" default="$(find ur_robot_driver)/resources/rtde_input_recipe.txt"/>
+  <xacro:arg name="reverse_ip" default="0.0.0.0"/>
+  <xacro:arg name="script_command_port" default="50004"/>
+  <xacro:arg name="reverse_port" default="50001"/>
+  <xacro:arg name="script_sender_port" default="50002"/>
+  <xacro:arg name="trajectory_port" default="50003"/>
+  <!-- tool communication related parameters-->
+  <xacro:arg name="use_tool_communication" default="false" />
+  <xacro:arg name="tool_voltage" default="0" />
+  <xacro:arg name="tool_parity" default="0" />
+  <xacro:arg name="tool_baud_rate" default="115200" />
+  <xacro:arg name="tool_stop_bits" default="1" />
+  <xacro:arg name="tool_rx_idle_chars" default="1.5" />
+  <xacro:arg name="tool_tx_idle_chars" default="3.5" />
+  <xacro:arg name="tool_device_name" default="/tmp/ttyUR" />
+  <xacro:arg name="tool_tcp_port" default="54321" />
+  <xacro:arg name="use_mock_hardware" default="false" />
+  <xacro:arg name="mock_sensor_commands" default="false" />
+  <!-- simulation controllers will be passed from launch file after substitutions -->
+  <xacro:arg name="simulation_controllers" default=""/>
+  <xacro:macro name="ur_robot" params="name parent use_gz include_arm_ros2_control arm_type tf_prefix robot_ip *origin">
+    <!-- parse initial positions as a dictionary -->
+    <xacro:property
+      name="ur_initial_positions"
+      value="${xacro.load_yaml('$(arg initial_positions_file)')}"
       />
-  </xacro:if>
+    <!-- create arm from macro-->
+    <xacro:ur_robot
+      name="${name}"
+      parent="${parent}"
+      tf_prefix="${tf_prefix}"
+      joint_limits_parameters_file="$(arg joint_limit_params)"
+      kinematics_parameters_file="$(arg kinematics_params)"
+      physical_parameters_file="$(arg physical_params)"
+      visual_parameters_file="$(arg visual_params)"
+      safety_limits="$(arg safety_limits)"
+      safety_pos_margin="$(arg safety_pos_margin)"
+      safety_k_position="$(arg safety_k_position)"
+      force_abs_paths="$(arg force_abs_paths)"
+      >
+      <xacro:insert_block name="origin" />
+    </xacro:ur_robot>
+    <!-- this condition is to ensure that ros2_control doesn't interfere with gz_ros2_control during simulation  -->
+    <xacro:unless value="${use_gz}">
+      <xacro:if value="${include_arm_ros2_control}">
+        <xacro:ur_ros2_control
+          name="${name}"
+          tf_prefix="${tf_prefix}"
+          kinematics_parameters_file="$(arg kinematics_params)"
+          transmission_hw_interface="$(arg transmission_hw_interface)"
+          headless_mode="$(arg headless_mode)"
+          initial_positions="${ur_initial_positions}"
+          use_tool_communication="$(arg use_tool_communication)"
+          tool_voltage="$(arg tool_voltage)"
+          tool_parity="$(arg tool_parity)"
+          tool_baud_rate="$(arg tool_baud_rate)"
+          tool_stop_bits="$(arg tool_stop_bits)"
+          tool_rx_idle_chars="$(arg tool_rx_idle_chars)"
+          tool_tx_idle_chars="$(arg tool_tx_idle_chars)"
+          tool_device_name="$(arg tool_device_name)"
+          tool_tcp_port="$(arg tool_tcp_port)"
+          robot_ip="${robot_ip}"
+          script_filename="$(arg script_filename)"
+          output_recipe_filename="$(arg output_recipe_filename)"
+          input_recipe_filename="$(arg input_recipe_filename)"
+          reverse_ip="$(arg reverse_ip)"
+          script_command_port="$(arg script_command_port)"
+          reverse_port="$(arg reverse_port)"
+          script_sender_port="$(arg script_sender_port)"
+          trajectory_port="$(arg trajectory_port)"
+          use_mock_hardware="$(arg use_mock_hardware)"
+          mock_sensor_commands="$(arg mock_sensor_commands)"
+          />
+      </xacro:if>
+    </xacro:unless>
+  </xacro:macro>
 </robot>

Commit message: fixed prefix usage and macro usage

File: rox_description/urdf/rox.urdf.xacro (robot description, xacro)
@@ -35,5 +35,6 @@
   <xacro:arg name="safety_pos_margin" default="0.15"/>
   <xacro:arg name="safety_k_position" default="20"/>
-  <xacro:arg name="initial_positions_file" default="$(find rox_bringup)/configs/ur/initial_joint_positions.yaml"/>
+  <xacro:arg name="arm1_initial_positions" default="$(find rox_bringup)/configs/ur/initial_joint_positions.yaml"/>
+  <xacro:arg name="arm2_initial_positions" default="$(find rox_bringup)/configs/ur/initial_joint_positions-2.yaml"/>
   <!-- Xacro Properties -->
   <xacro:property name="gz" value="$(arg use_gz)"/>
@@ -247,6 +248,4 @@
       <xacro:if value="${arm2 == 'ur5' or arm2 == 'ur10' or arm2 == 'ur5e' or arm2 == 'ur10e'}">
         <!-- Include UR macros -->
-        <!-- <xacro:include filename="$(find ur_description)/urdf/ur_macro.xacro"/>
-        <xacro:include filename="$(find ur_robot_driver)/urdf/ur.ros2_control.xacro"/> -->
         <xacro:include filename="$(find rox_description)/urdf/xacros/ur_arm.urdf.xacro"/>
         <!-- Arm 2 -->
@@ -267,5 +266,5 @@
             robot_ip="$(arg robot_ip)"
             >
-            <origin xyz="0.0 0.0 0.0" rpy="0 0 -2.355" />
+            <origin xyz="0.0 0.0 0.0" rpy="0 0 -0.7854" />
           </xacro:ur>
         </xacro:if>
@@ -337,5 +336,5 @@
           <xacro:property
             name="arm1_initial_positions"
-            value="${xacro.load_yaml('$(arg initial_positions_file)')}"
+            value="${xacro.load_yaml('$(arg arm1_initial_positions)')}"
             />
           <xacro:ur_ros2_control
@@ -346,4 +345,18 @@
         </xacro:if>
       </xacro:unless>
+      <!-- Arm 2 ros2_control -->
+      <xacro:unless value="${arm2 == ''}">
+        <xacro:if value="${arm2 == 'ur5' or arm2 == 'ur10' or arm2 == 'ur5e' or arm2 == 'ur10e'}">
+          <xacro:property
+            name="arm2_initial_positions"
+            value="${xacro.load_yaml('$(arg arm2_initial_positions)')}"
+            />
+          <xacro:ur_ros2_control
+            name="$(arg arm2_prefix)$(arg arm2_type)"
+            tf_prefix="$(arg arm2_prefix)"
+            initial_positions="${arm2_initial_positions}"
+            />
+        </xacro:if>
+      </xacro:unless>
     </xacro:unless>
   </xacro:if>

File: rox_description/urdf/xacros/ur_arm.urdf.xacro (robot description, xacro)
@@ -46,6 +46,7 @@
   <!-- simulation controllers will be passed from launch file after substitutions -->
   <xacro:arg name="simulation_controllers" default=""/>
-  <xacro:macro name="ur_robot" params="name parent use_gz include_arm_ros2_control arm_type tf_prefix robot_ip *origin">
+  <xacro:macro name="ur" params="name parent use_gz include_arm_ros2_control arm_type tf_prefix robot_ip *origin">
     <!-- parse initial positions as a dictionary -->
+    <!-- This is mainly for using with Mock Controller -->
     <xacro:property
       name="ur_initial_positions"

Commit message: handling ip address for multiple arms

File: rox_description/urdf/rox.urdf.xacro (robot description, xacro)
@@ -29,6 +29,7 @@
   <xacro:arg name="include_arm_ros2_control" default="false"/>
   <xacro:arg name="include_gripper_ros2_control" default="false"/>
-  <!-- UR ros2_control parameters (used when include_arm_ros2_control is true) -->
-  <xacro:arg name="robot_ip" default="192.168.1.102" />
+  <!-- ip addresses of the arms -->
+  <xacro:arg name="robot_ip_arm1" default="192.168.1.102" />
+  <xacro:arg name="robot_ip_arm2" default="192.168.1.103" />
   <!-- UR arm parameters (shared) -->
   <xacro:arg name="safety_limits" default="false"/>
@@ -51,4 +52,6 @@
   <xacro:property name="use_mock" value="$(arg use_mock_hardware)"/>
   <xacro:property name="linear_axis" value="$(arg enable_linear_axis)"/>
+  <xacro:property name="arm1_ip" value="$(arg robot_ip_arm1)"/>
+  <xacro:property name="arm2_ip" value="$(arg robot_ip_arm2)"/>
   <!-- Include xacro files -->
   <xacro:include filename="$(find rox_description)/urdf/xacros/frame.xacro" />
@@ -190,5 +193,5 @@
             arm_type="${arm}"
             tf_prefix="$(arg arm1_prefix)"
-            robot_ip="$(arg robot_ip)"
+            robot_ip="$(arg arm1_ip)"
             >
             <origin xyz="0.0 0.0 0.0" rpy="0 0 -2.355" />
@@ -203,5 +206,5 @@
             arm_type="${arm}"
             tf_prefix="$(arg arm1_prefix)"
-            robot_ip="$(arg robot_ip)"
+            robot_ip="$(arg arm1_ip)"
             >
             <origin xyz="0.218 0.0 0.0" rpy="0.0 0.0 0.0" />
@@ -264,5 +267,5 @@
             arm_type="${arm2}"
             tf_prefix="$(arg arm2_prefix)"
-            robot_ip="$(arg robot_ip)"
+            robot_ip="$(arg arm2_ip)"
             >
             <origin xyz="0.0 0.0 0.0" rpy="0 0 -0.7854" />
@@ -277,5 +280,5 @@
             arm_type="${arm2}"
             tf_prefix="$(arg arm2_prefix)"
-            robot_ip="$(arg robot_ip)"
+            robot_ip="$(arg arm2_ip)"
             >
             <origin xyz="0.218 0.0 0.0" rpy="0.0 0.0 0.0" />
