Commit message: Merge pull request #116 from neobotix/ipa-urdf-update
URDF update plus some minors

File: rox_description/urdf/xacros/ur_arm.urdf.xacro (robot description, xacro)
@@ -9,17 +9,5 @@
   <xacro:include filename="$(find ur_robot_driver)/urdf/ur.ros2_control.xacro"/>
   <xacro:include filename="$(find ur_description)/urdf/inc/ur_transmissions.xacro"/>
-  <!-- Set use_gz = true for simulation -->
-  <xacro:arg name="use_gz" default="false"/>
-  <xacro:arg name="include_arm_ros2_control" default="false"/>
-  <!-- arm parameters -->
-  <xacro:arg name="arm_type" default="ur10"/>
-  <xacro:property name="arm_height" default="0.376" />
-  <xacro:arg name="arm_parent" default="world"/>
   <!-- UR arm parameters -->
-  <xacro:arg name="tf_prefix" default="$(arg arm_type)" />
-  <xacro:arg name="joint_limit_params" default="$(find ur_description)/config/$(arg arm_type)/joint_limits.yaml"/>
-  <xacro:arg name="kinematics_params" default="$(find ur_description)/config/$(arg arm_type)/default_kinematics.yaml"/>
-  <xacro:arg name="physical_params" default="$(find ur_description)/config/$(arg arm_type)/physical_parameters.yaml"/>
-  <xacro:arg name="visual_params" default="$(find ur_description)/config/$(arg arm_type)/visual_parameters.yaml"/>
   <xacro:arg name="transmission_hw_interface" default="hardware_interface/PositionJointInterface"/>
   <xacro:arg name="safety_limits" default="false"/>
@@ -30,102 +18,89 @@
   <!-- When using gazebo simulations absolute paths are necessary -->
   <xacro:arg name="force_abs_paths" default="false" />
-  <!-- parse initial positions as a dictionary -->
-  <xacro:property
-    name="ur_initial_positions"
-    value="${xacro.load_yaml('$(arg initial_positions_file)')}"
-    />
-  <!-- create arm from macro-->
-  <xacro:ur_robot
-    name="$(arg arm_type)"
-    parent="$(arg arm_parent)"
-    tf_prefix="$(arg tf_prefix)"
-    joint_limits_parameters_file="$(arg joint_limit_params)"
-    kinematics_parameters_file="$(arg kinematics_params)"
-    physical_parameters_file="$(arg physical_params)"
-    visual_parameters_file="$(arg visual_params)"
-    safety_limits="$(arg safety_limits)"
-    safety_pos_margin="$(arg safety_pos_margin)"
-    safety_k_position="$(arg safety_k_position)"
-    force_abs_paths="$(arg force_abs_paths)"
-    >
-    <!-- position of arm in the world -->
-    <origin xyz="0.218 0.0 ${arm_height}" rpy="0.0 0.0 3.1415926535897931" />
-  </xacro:ur_robot>
-  <!-- this condition is to ensure that ros2_control doesn't interfere with gz_ros2_control during simulation  -->
-  <xacro:unless value="$(arg use_gz)">
-    <xacro:if value="$(arg include_arm_ros2_control)">
-      <!-- ros2_control related parameters -->
-      <xacro:arg name="headless_mode" default="false" />
-      <xacro:arg name="robot_ip" default="192.168.1.102" />
-      <xacro:arg name="script_filename" default="$(find ur_client_library)/resources/external_control.urscript"/>
-      <xacro:arg name="output_recipe_filename" default="$(find ur_robot_driver)/resources/rtde_output_recipe.txt"/>
-      <xacro:arg name="input_recipe_filename" default="$(find ur_robot_driver)/resources/rtde_input_recipe.txt"/>
-      <xacro:arg name="reverse_ip" default="0.0.0.0"/>
-      <xacro:arg name="script_command_port" default="50004"/>
-      <xacro:arg name="reverse_port" default="50001"/>
-      <xacro:arg name="script_sender_port" default="50002"/>
-      <xacro:arg name="trajectory_port" default="50003"/>
-      <!-- tool communication related parameters-->
-      <xacro:arg name="use_tool_communication" default="false" />
-      <xacro:arg name="tool_voltage" default="0" />
-      <xacro:arg name="tool_parity" default="0" />
-      <xacro:arg name="tool_baud_rate" default="115200" />
-      <xacro:arg name="tool_stop_bits" default="1" />
-      <xacro:arg name="tool_rx_idle_chars" default="1.5" />
-      <xacro:arg name="tool_tx_idle_chars" default="3.5" />
-      <xacro:arg name="tool_device_name" default="/tmp/ttyUR" />
-      <xacro:arg name="tool_tcp_port" default="54321" />
-      <xacro:arg name="use_mock_hardware" default="false" />
-      <xacro:arg name="mock_sensor_commands" default="false" />
-      <xacro:ur_ros2_control
-        name="$(arg arm_type)"
-        tf_prefix="$(arg tf_prefix)"
-        kinematics_parameters_file="$(arg kinematics_params)"
-        transmission_hw_interface="$(arg transmission_hw_interface)"
-        headless_mode="$(arg headless_mode)"
-        initial_positions="${ur_initial_positions}"
-        use_tool_communication="$(arg use_tool_communication)"
-        tool_voltage="$(arg tool_voltage)"
-        tool_parity="$(arg tool_parity)"
-        tool_baud_rate="$(arg tool_baud_rate)"
-        tool_stop_bits="$(arg tool_stop_bits)"
-        tool_rx_idle_chars="$(arg tool_rx_idle_chars)"
-        tool_tx_idle_chars="$(arg tool_tx_idle_chars)"
-        tool_device_name="$(arg tool_device_name)"
-        tool_tcp_port="$(arg tool_tcp_port)"
-        robot_ip="$(arg robot_ip)"
-        script_filename="$(arg script_filename)"
-        output_recipe_filename="$(arg output_recipe_filename)"
-        input_recipe_filename="$(arg input_recipe_filename)"
-        reverse_ip="$(arg reverse_ip)"
-        script_command_port="$(arg script_command_port)"
-        reverse_port="$(arg reverse_port)"
-        script_sender_port="$(arg script_sender_port)"
-        trajectory_port="$(arg trajectory_port)"
-        use_mock_hardware="$(arg use_mock_hardware)"
-        mock_sensor_commands="$(arg mock_sensor_commands)"
-        />
-    </xacro:if>
-  </xacro:unless>
-  <!-- If gz simulation is used -->
-  <xacro:if value="$(arg use_gz)">
-    <!-- simulation controllers will be passed from launch file after substitutions -->
-    <xacro:arg name="simulation_controllers" default=""/>
-    <gazebo reference="$(arg arm_parent)">
-    </gazebo>
-    <gazebo>
-      <plugin name="gz_ros2_control::GazeboSimROS2ControlPlugin" filename="libgz_ros2_control-system">
-        <parameters>$(arg simulation_controllers)</parameters>
-        <!-- <controller_manager_node_name>$(arg tf_prefix)controller_manager</controller_manager_node_name> -->
-      </plugin>
-    </gazebo>
-    <!-- ros2 control instance -->
-    <xacro:include filename="$(find ur_simulation_gz)/urdf/ur_gz.ros2_control.xacro" />
-    <xacro:ur_ros2_control
-      name="$(arg arm_type)"
-      tf_prefix="$(arg tf_prefix)"
-      transmission_hw_interface="$(arg transmission_hw_interface)"
-      initial_positions="${ur_initial_positions}"
+  <!-- ros2_control related parameters -->
+  <xacro:arg name="headless_mode" default="false" />
+  <xacro:arg name="script_filename" default="$(find ur_client_library)/resources/external_control.urscript"/>
+  <xacro:arg name="output_recipe_filename" default="$(find ur_robot_driver)/resources/rtde_output_recipe.txt"/>
+  <xacro:arg name="input_recipe_filename" default="$(find ur_robot_driver)/resources/rtde_input_recipe.txt"/>
+  <xacro:arg name="reverse_ip" default="0.0.0.0"/>
+  <xacro:arg name="script_command_port" default="50004"/>
+  <xacro:arg name="reverse_port" default="50001"/>
+  <xacro:arg name="script_sender_port" default="50002"/>
+  <xacro:arg name="trajectory_port" default="50003"/>
+  <!-- tool communication related parameters-->
+  <xacro:arg name="use_tool_communication" default="false" />
+  <xacro:arg name="tool_voltage" default="0" />
+  <xacro:arg name="tool_parity" default="0" />
+  <xacro:arg name="tool_baud_rate" default="115200" />
+  <xacro:arg name="tool_stop_bits" default="1" />
+  <xacro:arg name="tool_rx_idle_chars" default="1.5" />
+  <xacro:arg name="tool_tx_idle_chars" default="3.5" />
+  <xacro:arg name="tool_device_name" default="/tmp/ttyUR" />
+  <xacro:arg name="tool_tcp_port" default="54321" />
+  <xacro:arg name="use_mock_hardware" default="false" />
+  <xacro:arg name="mock_sensor_commands" default="false" />
+  <!-- simulation controllers will be passed from launch file after substitutions -->
+  <xacro:arg name="simulation_controllers" default=""/>
+  <xacro:macro name="ur" params="name parent use_gz include_arm_ros2_control arm_type tf_prefix robot_ip *origin">
+    <!-- default config path for ur arm -->
+    <xacro:arg name="joint_limit_params" default="$(find ur_description)/config/$(arg arm_type)/joint_limits.yaml"/>
+    <xacro:arg name="kinematics_params" default="$(find ur_description)/config/$(arg arm_type)/default_kinematics.yaml"/>
+    <xacro:arg name="physical_params" default="$(find ur_description)/config/$(arg arm_type)/physical_parameters.yaml"/>
+    <xacro:arg name="visual_params" default="$(find ur_description)/config/$(arg arm_type)/visual_parameters.yaml"/>
+    <!-- parse initial positions as a dictionary -->
+    <!-- This is mainly for using with Mock Controller -->
+    <xacro:property
+      name="ur_initial_positions"
+      value="${xacro.load_yaml('$(arg initial_positions_file)')}"
       />
-  </xacro:if>
+    <!-- create arm from macro-->
+    <xacro:ur_robot
+      name="${name}"
+      parent="${parent}"
+      tf_prefix="${tf_prefix}"
+      joint_limits_parameters_file="$(arg joint_limit_params)"
+      kinematics_parameters_file="$(arg kinematics_params)"
+      physical_parameters_file="$(arg physical_params)"
+      visual_parameters_file="$(arg visual_params)"
+      safety_limits="$(arg safety_limits)"
+      safety_pos_margin="$(arg safety_pos_margin)"
+      safety_k_position="$(arg safety_k_position)"
+      force_abs_paths="$(arg force_abs_paths)"
+      >
+      <xacro:insert_block name="origin" />
+    </xacro:ur_robot>
+    <!-- this condition is to ensure that ros2_control doesn't interfere with gz_ros2_control during simulation  -->
+    <xacro:unless value="${use_gz}">
+      <xacro:if value="${include_arm_ros2_control}">
+        <xacro:ur_ros2_control
+          name="${name}"
+          tf_prefix="${tf_prefix}"
+          kinematics_parameters_file="$(arg kinematics_params)"
+          transmission_hw_interface="$(arg transmission_hw_interface)"
+          headless_mode="$(arg headless_mode)"
+          initial_positions="${ur_initial_positions}"
+          use_tool_communication="$(arg use_tool_communication)"
+          tool_voltage="$(arg tool_voltage)"
+          tool_parity="$(arg tool_parity)"
+          tool_baud_rate="$(arg tool_baud_rate)"
+          tool_stop_bits="$(arg tool_stop_bits)"
+          tool_rx_idle_chars="$(arg tool_rx_idle_chars)"
+          tool_tx_idle_chars="$(arg tool_tx_idle_chars)"
+          tool_device_name="$(arg tool_device_name)"
+          tool_tcp_port="$(arg tool_tcp_port)"
+          robot_ip="${robot_ip}"
+          script_filename="$(arg script_filename)"
+          output_recipe_filename="$(arg output_recipe_filename)"
+          input_recipe_filename="$(arg input_recipe_filename)"
+          reverse_ip="$(arg reverse_ip)"
+          script_command_port="$(arg script_command_port)"
+          reverse_port="$(arg reverse_port)"
+          script_sender_port="$(arg script_sender_port)"
+          trajectory_port="$(arg trajectory_port)"
+          use_mock_hardware="$(arg use_mock_hardware)"
+          mock_sensor_commands="$(arg mock_sensor_commands)"
+          />
+      </xacro:if>
+    </xacro:unless>
+  </xacro:macro>
 </robot>

Commit message: updating the position of the realsense camera

File: rox_description/urdf/rox.urdf.xacro (robot description, xacro)
@@ -117,6 +117,6 @@
     <xacro:include filename="$(find realsense2_description)/urdf/_d435.urdf.xacro"/>
     <!-- use_nominal_extrinsics is True for simulation-->
-    <xacro:sensor_d435 parent="base_link" name="d435_camera" use_nominal_extrinsics="true">
-      <origin xyz="0.375 0.0 0.220" rpy="0 0 0"/>
+    <xacro:sensor_d435 parent="base_link" name="d435_camera" use_nominal_extrinsics=${gz}>
+      <origin xyz="0.3591 -0.0175 0.2475" rpy="0 0 0"/>
     </xacro:sensor_d435>
   </xacro:if>

Commit message: updating the position of the realsense camera

File: rox_description/urdf/rox.urdf.xacro (robot description, xacro)
@@ -117,6 +117,6 @@
     <xacro:include filename="$(find realsense2_description)/urdf/_d435.urdf.xacro"/>
     <!-- use_nominal_extrinsics is True for simulation-->
-    <xacro:sensor_d435 parent="base_link" name="d435_camera" use_nominal_extrinsics="true">
-      <origin xyz="0.375 0.0 0.220" rpy="0 0 0"/>
+    <xacro:sensor_d435 parent="base_link" name="d435_camera" use_nominal_extrinsics="${gz}">
+      <origin xyz="0.3591 -0.0175 0.2475" rpy="0 0 0"/>
     </xacro:sensor_d435>
   </xacro:if>

Commit message: updating the position of the imu

File: rox_description/urdf/rox.urdf.xacro (robot description, xacro)
@@ -108,5 +108,5 @@
     <joint name="imu_joint" type="fixed">
       <axis xyz="0 1 0"/>
-      <origin rpy="0 0 0" xyz="-0.052 0.208 0.266"/>
+      <origin rpy="0 0 0" xyz="-0.206 0.0 0.179"/>
       <parent link="base_link"/>
       <child link="imu_link"/>

Commit message: adding ewellix_lift axis

File: rox_description/urdf/rox.urdf.xacro (robot description, xacro)
@@ -13,4 +13,5 @@
   <xacro:arg name="rox_type" default="argo"/>
   <xacro:arg name="joint_type" default="fixed"/>
+  <xacro:arg name="enable_lift_axis" default="true"/>
   <!-- Manipulator Arguments-->
   <xacro:arg name="arm_type" default=""/>
@@ -35,4 +36,5 @@
   <xacro:property name="gripper" value="$(arg gripper_type)"/>
   <xacro:property name="use_mock" value="$(arg use_mock_hardware)"/>
+  <xacro:property name="lift" value="$(arg enable_lift_axis)"/>
   <!-- Include xacro files -->
   <xacro:include filename="$(find rox_description)/urdf/xacros/frame.xacro" />
@@ -71,12 +73,31 @@
     <xacro:trike_drive parent="base_link" wheel_separation="${wheel_separation}"/>
   </xacro:if>
+  <!-- Lift axis -->
+  <xacro:if value="${lift == True}">
+    <xacro:include filename="$(find ewellix_description)/urdf/ewellix_macro.xacro"/>
+    <xacro:ewellix_linear_actuator sim_gazebo="${gz}" type="tlt_x25" />
+  </xacro:if>
   <!-- Laser scanners -->
+  <!-- Lift-axis variant is wider in X and Y -->
+  <!-- ToDo: waiting for the lift axis dimensions and ROX base frame dimension -->
   <!-- Nanoscans -->
+  <xacro:if value="${lift == True}">
+    <xacro:property name="nanoscan_x" value="0.3495"/>
+    <xacro:property name="nanoscan_y" value="0.2690"/>
+    <xacro:property name="psenscan_x" value="0.3516"/>
+    <xacro:property name="psenscan_y" value="0.2719"/>
+  </xacro:if>
+  <xacro:unless value="${lift == True}">
+    <xacro:property name="nanoscan_x" value="0.2995"/>
+    <xacro:property name="nanoscan_y" value="0.2690"/>
+    <xacro:property name="psenscan_x" value="0.3016"/>
+    <xacro:property name="psenscan_y" value="0.2719"/>
+  </xacro:unless>
   <xacro:if value="${scanner == 'nanoscan'}">
     <xacro:sick_nanoscan name="lidar_1" parent="base_link">
-      <origin rpy="${pi} 0 ${pi/4}" xyz="${0.2995} 0.269 0.189"/>
+      <origin rpy="${pi} 0 ${pi/4}" xyz="${nanoscan_x} ${nanoscan_y} 0.189"/>
     </xacro:sick_nanoscan>
     <xacro:sick_nanoscan name="lidar_2" parent="base_link">
-      <origin rpy="${pi} 0 -${pi - pi/4}" xyz="-${0.2995} -0.269 0.189"/>
+      <origin rpy="${pi} 0 -${pi - pi/4}" xyz="-${nanoscan_x} -${nanoscan_y} 0.189"/>
     </xacro:sick_nanoscan>
   </xacro:if>
@@ -84,8 +105,8 @@
   <xacro:if value="${scanner == 'psenscan'}">
     <xacro:pilz_psenscan name="lidar_1" parent="base_link">
-      <origin rpy="0 0 ${pi/4}" xyz="${0.3016} 0.2719 0.191"/>
+      <origin rpy="0 0 ${pi/4}" xyz="${psenscan_x} ${psenscan_y} 0.191"/>
     </xacro:pilz_psenscan>
     <xacro:pilz_psenscan name="lidar_2" parent="base_link">
-      <origin rpy="0 0 -${pi - pi/4}" xyz="-${0.3016} -0.2719 0.191"/>
+      <origin rpy="0 0 -${pi - pi/4}" xyz="-${psenscan_x} -${psenscan_y} 0.191"/>
     </xacro:pilz_psenscan>
   </xacro:if>
@@ -124,8 +145,10 @@
   <xacro:unless value="${arm == ''}">
     <!-- Include cabinet -->
-    <xacro:include filename="$(find rox_description)/urdf/xacros/cabinet.xacro" />
-    <xacro:cabinet name="cabinet" parent="base_footprint">
-      <origin rpy="0 0 0" xyz="0 0 0.33"/>
-    </xacro:cabinet>
+    <xacro:unless value="${lift == True}">
+      <xacro:include filename="$(find rox_description)/urdf/xacros/cabinet.xacro" />
+      <xacro:cabinet name="cabinet" parent="base_footprint">
+        <origin rpy="0 0 0" xyz="0 0 0.33"/>
+      </xacro:cabinet>
+    </xacro:unless>
     <!-- Universal Robotics (UR) Arms-->
     <xacro:if value="${arm == 'ur5' or arm == 'ur10' or arm == 'ur5e' or arm == 'ur10e' or arm == 'ur8long'}">
@@ -139,4 +162,36 @@
       <!-- Include the UR arm -->
       <xacro:include filename="$(find rox_description)/urdf/xacros/ur_arm.urdf.xacro"/>
+      <xacro:if value="${lift == True}">
+          <link name="ur_lift_axis_connector"/>
+          <joint name="lift_axis_connector_joint" type="fixed">
+            <origin xyz="0.450 0.156 0.529" rpy="-${pi/3} 0 0" />
+            <parent link="linear_axis_slide_link"/>
+            <child link="ur_lift_axis_connector"/>
+          </joint>
+          <xacro:ur
+            name="${arm}"
+            parent="ur_lift_axis_connector"
+            use_gz="${gz}"
+            include_arm_ros2_control="$(arg include_arm_ros2_control)"
+            arm_type="${arm}"
+            tf_prefix="$(arg arm_prefix)"
+            robot_ip="${arm_ip}"
+            >
+            <origin xyz="0.0 0.0 0.0" rpy="0 0 -2.355" />
+          </xacro:ur>
+      </xacro:if>
+      <xacro:unless value="${lift == True}">
+        <xacro:ur
+          name="${arm}"
+          parent="cabinet_link"
+          use_gz="${gz}"
+          include_arm_ros2_control="$(arg include_arm_ros2_control)"
+          arm_type="${arm}"
+          tf_prefix="$(arg arm_prefix)"
+          robot_ip="${arm_ip}"
+          >
+          <origin xyz="0.218 0.0 0.0" rpy="0.0 0.0 0.0" />
+        </xacro:ur>
+      </xacro:unless>
     </xacro:if>
     <!-- Elite Arms-->

Commit message: updates

File: rox_description/urdf/rox.urdf.xacro (robot description, xacro)
@@ -83,6 +83,6 @@
   <!-- Nanoscans -->
   <xacro:if value="${lift == True}">
-    <xacro:property name="nanoscan_x" value="0.3495"/>
-    <xacro:property name="nanoscan_y" value="0.2690"/>
+    <xacro:property name="nanoscan_x" value="0.427"/>
+    <xacro:property name="nanoscan_y" value="0.314"/>
     <xacro:property name="psenscan_x" value="0.3516"/>
     <xacro:property name="psenscan_y" value="0.2719"/>

File: rox_description/urdf/xacros/argo_drive.xacro (robot description, xacro)
@@ -7,20 +7,20 @@
         vis_rot="0 0 0" vis_pos="0 0 0"
         joint_type="${joint_typ}">
-        <origin rpy="0 0 ${pi}" xyz="0.239 0.229 0.123"/>
+        <origin rpy="0 0 ${pi}" xyz="0.367 0.274 0.123"/>
     </xacro:argo_caster>
     <xacro:argo_caster name="caster_front_right" parent="${parent}"
         vis_rot="0 0 ${pi}" vis_pos="0 0 0"
         joint_type="${joint_typ}">
-        <origin rpy="0 0 0" xyz="0.239 -0.229 0.123"/>
+        <origin rpy="0 0 0" xyz="0.367 -0.274 0.123"/>
     </xacro:argo_caster>
     <xacro:argo_caster name="caster_back_left" parent="${parent}"
         vis_rot="0 0 0" vis_pos="0 0 0"
         joint_type="${joint_typ}">
-        <origin rpy="0 0 ${pi}" xyz="-0.239 0.229 0.123"/>
+        <origin rpy="0 0 ${pi}" xyz="-0.367 0.274 0.123"/>
     </xacro:argo_caster>
     <xacro:argo_caster name="caster_back_right" parent="${parent}"
         vis_rot="0 0 ${pi}" vis_pos="0 0 0"
         joint_type="${joint_typ}">
-        <origin rpy="0 0 0" xyz="-0.239 -0.229 0.123"/>
+        <origin rpy="0 0 0" xyz="-0.367 -0.274 0.123"/>
     </xacro:argo_caster>
     <xacro:argo_wheel name="wheel_front_left" parent="caster_front_left_link"
