Commit message: updating the urdf and the charge current

File: rox_description/urdf/rox.urdf.xacro (robot description, xacro)
@@ -155,5 +155,5 @@
     <xacro:include filename="$(find rox_description)/urdf/xacros/cabinet.xacro" />
     <xacro:cabinet name="cabinet" parent="base_footprint">
-      <origin rpy="0 0 0" xyz="0 0 0.334"/>
+      <origin rpy="0 0 3.14" xyz="0 0 0.334"/>
     </xacro:cabinet>
     <!-- Universal Robotics (UR) Arms-->

Commit message: fixing the laserscanner orientation

File: rox_description/urdf/rox.urdf.xacro (robot description, xacro)
@@ -75,8 +75,8 @@
   <xacro:if value="${scanner == 'nanoscan'}">
     <xacro:sick_nanoscan name="lidar_1" parent="base_link">
-      <origin rpy="${pi} 0 ${pi/4}" xyz="${0.2995} 0.269 0.189"/>
+      <origin rpy="0 0 ${pi/4}" xyz="${0.2995} 0.269 0.189"/>
     </xacro:sick_nanoscan>
     <xacro:sick_nanoscan name="lidar_2" parent="base_link">
-      <origin rpy="${pi} 0 -${pi - pi/4}" xyz="-${0.2995} -0.269 0.189"/>
+      <origin rpy="0 0 -${pi - pi/4}" xyz="-${0.2995} -0.269 0.189"/>
     </xacro:sick_nanoscan>
   </xacro:if>

File: rox_description/urdf/xacros/sick_nanoscan.xacro (robot description, xacro)
@@ -11,9 +11,9 @@
       <inertial>
       <mass value="0.001"/>
-      <origin rpy="${pi} 0 ${pi/2}" xyz="0 0 0.0"/>
+      <origin rpy="0 0 -${pi/2}" xyz="0 0 0.0"/>
       <inertia ixx="0.0001" ixy="0" ixz="0" iyy="0.000001" iyz="0" izz="0.0001"/>
     </inertial>
     <visual>
-      <origin rpy="${pi} 0 ${pi/2}" xyz="0 0 -0.02"/>
+      <origin rpy="0 0 -${pi/2}" xyz="0 0 0.02"/>
       <geometry>
         <mesh filename="package://rox_description/meshes/nanoscan_3.dae" scale="0.1 0.1 0.1"/>
@@ -21,5 +21,5 @@
     </visual>
     <collision>
-      <origin rpy="${pi} 0 ${pi/2}" xyz="0 0 -0.02"/>
+      <origin rpy="0 0 -${pi/2}" xyz="0 0 0.02"/>
       <geometry>
         <mesh filename="package://rox_description/meshes/nanoscan_3.dae" scale="0.1 0.1 0.1"/>

Commit message: updating the position of the scanners

File: rox_description/urdf/rox.urdf.xacro (robot description, xacro)
@@ -75,8 +75,8 @@
   <xacro:if value="${scanner == 'nanoscan'}">
     <xacro:sick_nanoscan name="lidar_1" parent="base_link">
-      <origin rpy="${pi} 0 ${pi/4}" xyz="${0.2995} 0.269 0.189"/>
+      <origin rpy="${pi} 0 ${pi/4}" xyz="0.429 0.269 0.189"/>
     </xacro:sick_nanoscan>
     <xacro:sick_nanoscan name="lidar_2" parent="base_link">
-      <origin rpy="${pi} 0 -${pi - pi/4}" xyz="-${0.2995} -0.269 0.189"/>
+      <origin rpy="${pi} 0 -${pi - pi/4}" xyz="-0.429 -0.269 0.189"/>
     </xacro:sick_nanoscan>
   </xacro:if>

Commit message: updates for dual arm support

File: rox_description/urdf/rox.urdf.xacro (robot description, xacro)
@@ -27,4 +27,5 @@
   <xacro:arg name="use_mock_hardware" default="false" />
   <xacro:arg name="mock_sensor_commands" default="false" />
+  <xacro:arg name="use_mock_linear_axis" default="$(arg use_mock_hardware)" />
   <xacro:arg name="include_arm_ros2_control" default="false"/>
   <xacro:arg name="include_gripper_ros2_control" default="false"/>
@@ -38,4 +39,16 @@
   <xacro:arg name="arm1_initial_positions" default="$(find rox_bringup)/configs/ur/initial_joint_positions.yaml"/>
   <xacro:arg name="arm2_initial_positions" default="$(find rox_bringup)/configs/ur/initial_joint_positions-2.yaml"/>
+  <xacro:arg name="arm1_kinematics_parameters_file" default="$(find ur_description)/config/$(arg arm_type)/default_kinematics.yaml"/>
+  <xacro:arg name="arm2_kinematics_parameters_file" default="$(find ur_description)/config/$(arg arm2_type)/default_kinematics.yaml"/>
+  <xacro:arg name="headless_mode" default="false"/>
+  <!-- Unique local ports are required when both UR drivers run on this host. -->
+  <xacro:arg name="arm1_reverse_port" default="50001"/>
+  <xacro:arg name="arm1_script_sender_port" default="50002"/>
+  <xacro:arg name="arm1_script_command_port" default="50004"/>
+  <xacro:arg name="arm1_trajectory_port" default="50003"/>
+  <xacro:arg name="arm2_reverse_port" default="50006"/>
+  <xacro:arg name="arm2_script_sender_port" default="50007"/>
+  <xacro:arg name="arm2_script_command_port" default="50010"/>
+  <xacro:arg name="arm2_trajectory_port" default="50009"/>
   <!-- Xacro Properties -->
   <xacro:property name="gz" value="$(arg use_gz)"/>
@@ -51,4 +64,5 @@
   <xacro:property name="gripper2" value="$(arg gripper2_type)"/>
   <xacro:property name="use_mock" value="$(arg use_mock_hardware)"/>
+  <xacro:property name="mock_linear_axis" value="$(arg use_mock_linear_axis)"/>
   <xacro:property name="linear_axis" value="$(arg enable_linear_axis)"/>
   <xacro:property name="arm1_ip" value="$(arg robot_ip_arm1)"/>
@@ -93,5 +107,5 @@
   <xacro:if value="${linear_axis == True}">
     <xacro:include filename="$(find rox_description)/urdf/xacros/linear_axis.xacro"/>
-    <xacro:linear_axis parent="base_link"/>
+    <xacro:linear_axis parent="base_link" use_mock_hardware="${mock_linear_axis}"/>
   </xacro:if>
   <!-- Scanner placement -->
@@ -194,4 +208,15 @@
             tf_prefix="$(arg arm1_prefix)"
             robot_ip="${arm1_ip}"
+            initial_positions_file="$(arg arm1_initial_positions)"
+            joint_limits_parameters_file="$(find ur_description)/config/$(arg arm_type)/joint_limits.yaml"
+            kinematics_parameters_file="$(arg arm1_kinematics_parameters_file)"
+            physical_parameters_file="$(find ur_description)/config/$(arg arm_type)/physical_parameters.yaml"
+            visual_parameters_file="$(find ur_description)/config/$(arg arm_type)/visual_parameters.yaml"
+            headless_mode="$(arg headless_mode)"
+            reverse_port="$(arg arm1_reverse_port)"
+            script_sender_port="$(arg arm1_script_sender_port)"
+            script_command_port="$(arg arm1_script_command_port)"
+            trajectory_port="$(arg arm1_trajectory_port)"
+            tool_device_name="/tmp/ttyUR_arm1"
             >
             <origin xyz="0.0 0.0 0.0" rpy="0 0 -2.355" />
@@ -207,4 +232,15 @@
             tf_prefix="$(arg arm1_prefix)"
             robot_ip="${arm1_ip}"
+            initial_positions_file="$(arg arm1_initial_positions)"
+            joint_limits_parameters_file="$(find ur_description)/config/$(arg arm_type)/joint_limits.yaml"
+            kinematics_parameters_file="$(arg arm1_kinematics_parameters_file)"
+            physical_parameters_file="$(find ur_description)/config/$(arg arm_type)/physical_parameters.yaml"
+            visual_parameters_file="$(find ur_description)/config/$(arg arm_type)/visual_parameters.yaml"
+            headless_mode="$(arg headless_mode)"
+            reverse_port="$(arg arm1_reverse_port)"
+            script_sender_port="$(arg arm1_script_sender_port)"
+            script_command_port="$(arg arm1_script_command_port)"
+            trajectory_port="$(arg arm1_trajectory_port)"
+            tool_device_name="/tmp/ttyUR_arm1"
             >
             <origin xyz="0.218 0.0 0.0" rpy="0.0 0.0 0.0" />
@@ -268,4 +304,15 @@
             tf_prefix="$(arg arm2_prefix)"
             robot_ip="${arm2_ip}"
+            initial_positions_file="$(arg arm2_initial_positions)"
+            joint_limits_parameters_file="$(find ur_description)/config/$(arg arm2_type)/joint_limits.yaml"
+            kinematics_parameters_file="$(arg arm2_kinematics_parameters_file)"
+            physical_parameters_file="$(find ur_description)/config/$(arg arm2_type)/physical_parameters.yaml"
+            visual_parameters_file="$(find ur_description)/config/$(arg arm2_type)/visual_parameters.yaml"
+            headless_mode="$(arg headless_mode)"
+            reverse_port="$(arg arm2_reverse_port)"
+            script_sender_port="$(arg arm2_script_sender_port)"
+            script_command_port="$(arg arm2_script_command_port)"
+            trajectory_port="$(arg arm2_trajectory_port)"
+            tool_device_name="/tmp/ttyUR_arm2"
             >
             <origin xyz="0.0 0.0 0.0" rpy="0 0 -0.7854" />
@@ -281,4 +328,15 @@
             tf_prefix="$(arg arm2_prefix)"
             robot_ip="${arm2_ip}"
+            initial_positions_file="$(arg arm2_initial_positions)"
+            joint_limits_parameters_file="$(find ur_description)/config/$(arg arm2_type)/joint_limits.yaml"
+            kinematics_parameters_file="$(arg arm2_kinematics_parameters_file)"
+            physical_parameters_file="$(find ur_description)/config/$(arg arm2_type)/physical_parameters.yaml"
+            visual_parameters_file="$(find ur_description)/config/$(arg arm2_type)/visual_parameters.yaml"
+            headless_mode="$(arg headless_mode)"
+            reverse_port="$(arg arm2_reverse_port)"
+            script_sender_port="$(arg arm2_script_sender_port)"
+            script_command_port="$(arg arm2_script_command_port)"
+            trajectory_port="$(arg arm2_trajectory_port)"
+            tool_device_name="/tmp/ttyUR_arm2"
             >
             <origin xyz="0.218 0.0 0.0" rpy="0.0 0.0 0.0" />

File: rox_description/urdf/xacros/linear_axis.xacro (robot description, xacro)
@@ -6,5 +6,5 @@
 -->
 <robot xmlns:xacro="http://www.ros.org/wiki/xacro" name="rox">
-  <xacro:macro name="linear_axis" params="parent">
+  <xacro:macro name="linear_axis" params="parent use_mock_hardware:=false">
     <xacro:if value="${gz == True}">
       <xacro:property name="linear_axis_effort_limit" value="5000.0"/>
@@ -93,9 +93,15 @@
       <ros2_control name="linear_axis_control" type="system" rw_rate="100">
         <hardware>
-          <plugin>nla/NlaHardwareInterface</plugin>
-          <param name="can_iface">can0</param>
-          <param name="timeout">0.2</param>
-          <param name="control_rate">100.0</param>
-          <param name="initial_pose">0.02</param>
+          <xacro:if value="${use_mock_hardware}">
+            <plugin>mock_components/GenericSystem</plugin>
+            <param name="calculate_dynamics">true</param>
+          </xacro:if>
+          <xacro:unless value="${use_mock_hardware}">
+            <plugin>nla/NlaHardwareInterface</plugin>
+            <param name="can_iface">can0</param>
+            <param name="timeout">0.2</param>
+            <param name="control_rate">100.0</param>
+            <param name="initial_pose">0.02</param>
+          </xacro:unless>
         </hardware>
         <joint name="linear_axis_slide_joint">

File: rox_description/urdf/xacros/ur_arm.urdf.xacro (robot description, xacro)
@@ -14,6 +14,4 @@
   <xacro:arg name="safety_pos_margin" default="0.15"/>
   <xacro:arg name="safety_k_position" default="20"/>
-  <!-- initial positions file for ur arm on rox-->
-  <xacro:arg name="initial_positions_file" default="$(find rox_bringup)/configs/ur/initial_joint_positions.yaml"/>
   <!-- When using gazebo simulations absolute paths are necessary -->
   <xacro:arg name="force_abs_paths" default="false" />
@@ -42,15 +40,31 @@
   <!-- simulation controllers will be passed from launch file after substitutions -->
   <xacro:arg name="simulation_controllers" default=""/>
-  <xacro:macro name="ur" params="name parent use_gz include_arm_ros2_control arm_type tf_prefix robot_ip *origin">
-    <!-- default config path for ur arm -->
-    <xacro:arg name="joint_limit_params" default="$(find ur_description)/config/$(arg arm_type)/joint_limits.yaml"/>
-    <xacro:arg name="kinematics_params" default="$(find ur_description)/config/$(arg arm_type)/default_kinematics.yaml"/>
-    <xacro:arg name="physical_params" default="$(find ur_description)/config/$(arg arm_type)/physical_parameters.yaml"/>
-    <xacro:arg name="visual_params" default="$(find ur_description)/config/$(arg arm_type)/visual_parameters.yaml"/>
+  <!--
+    All robot-specific driver settings are macro parameters.  This is important
+    for a multi-robot description: xacro arguments are global and would make
+    both hardware components use the same calibration, ports and tool device.
+  -->
+  <xacro:macro name="ur" params="
+      name parent use_gz include_arm_ros2_control arm_type tf_prefix robot_ip
+      initial_positions_file
+      joint_limits_parameters_file
+      kinematics_parameters_file
+      physical_parameters_file
+      visual_parameters_file
+      headless_mode:=false
+      reverse_ip:=0.0.0.0
+      script_command_port:=50004
+      reverse_port:=50001
+      script_sender_port:=50002
+      trajectory_port:=50003
+      use_tool_communication:=false
+      tool_device_name:=/tmp/ttyUR
+      tool_tcp_port:=54321
+      *origin">
     <!-- parse initial positions as a dictionary -->
     <!-- This is mainly for using with Mock Controller -->
     <xacro:property
       name="ur_initial_positions"
-      value="${xacro.load_yaml('$(arg initial_positions_file)')}"
+      value="${xacro.load_yaml(initial_positions_file)}"
       />
     <!-- create arm from macro-->
@@ -59,8 +73,8 @@
       parent="${parent}"
       tf_prefix="${tf_prefix}"
-      joint_limits_parameters_file="$(arg joint_limit_params)"
-      kinematics_parameters_file="$(arg kinematics_params)"
-      physical_parameters_file="$(arg physical_params)"
-      visual_parameters_file="$(arg visual_params)"
+      joint_limits_parameters_file="${joint_limits_parameters_file}"
+      kinematics_parameters_file="${kinematics_parameters_file}"
+      physical_parameters_file="${physical_parameters_file}"
+      visual_parameters_file="${visual_parameters_file}"
       safety_limits="$(arg safety_limits)"
       safety_pos_margin="$(arg safety_pos_margin)"
@@ -76,9 +90,9 @@
           name="${name}"
           tf_prefix="${tf_prefix}"
-          kinematics_parameters_file="$(arg kinematics_params)"
+          kinematics_parameters_file="${kinematics_parameters_file}"
           transmission_hw_interface="$(arg transmission_hw_interface)"
-          headless_mode="$(arg headless_mode)"
+          headless_mode="${headless_mode}"
           initial_positions="${ur_initial_positions}"
-          use_tool_communication="$(arg use_tool_communication)"
+          use_tool_communication="${use_tool_communication}"
           tool_voltage="$(arg tool_voltage)"
           tool_parity="$(arg tool_parity)"
@@ -87,15 +101,15 @@
           tool_rx_idle_chars="$(arg tool_rx_idle_chars)"
           tool_tx_idle_chars="$(arg tool_tx_idle_chars)"
-          tool_device_name="$(arg tool_device_name)"
-          tool_tcp_port="$(arg tool_tcp_port)"
+          tool_device_name="${tool_device_name}"
+          tool_tcp_port="${tool_tcp_port}"
           robot_ip="${robot_ip}"
           script_filename="$(arg script_filename)"
           output_recipe_filename="$(arg output_recipe_filename)"
           input_recipe_filename="$(arg input_recipe_filename)"
-          reverse_ip="$(arg reverse_ip)"
-          script_command_port="$(arg script_command_port)"
-          reverse_port="$(arg reverse_port)"
-          script_sender_port="$(arg script_sender_port)"
-          trajectory_port="$(arg trajectory_port)"
+          reverse_ip="${reverse_ip}"
+          script_command_port="${script_command_port}"
+          reverse_port="${reverse_port}"
+          script_sender_port="${script_sender_port}"
+          trajectory_port="${trajectory_port}"
           use_mock_hardware="$(arg use_mock_hardware)"
           mock_sensor_commands="$(arg mock_sensor_commands)"

Commit message: fixes URDF

File: rox_description/urdf/rox.urdf.xacro (robot description, xacro)
@@ -126,5 +126,5 @@
     <xacro:include filename="$(find rox_description)/urdf/xacros/cabinet.xacro" />
     <xacro:cabinet name="cabinet" parent="base_footprint">
-      <origin rpy="0 0 0" xyz="0 0 0.33"/>
+      <origin rpy="0 0 0" xyz="0 0 0.328"/>
     </xacro:cabinet>
     <!-- Universal Robotics (UR) Arms-->

Commit message: update xacro

File: rox_description/urdf/rox.urdf.xacro (robot description, xacro)
@@ -75,8 +75,8 @@
   <xacro:if value="${scanner == 'nanoscan'}">
     <xacro:sick_nanoscan name="lidar_1" parent="base_link">
-      <origin rpy="${pi} 0 ${pi/4}" xyz="0.429 0.269 0.189"/>
+      <origin rpy="${pi} 0 ${pi/4}" xyz="0.2995 0.269 0.189"/>
     </xacro:sick_nanoscan>
     <xacro:sick_nanoscan name="lidar_2" parent="base_link">
-      <origin rpy="${pi} 0 -${pi - pi/4}" xyz="-0.429 -0.269 0.189"/>
+      <origin rpy="${pi} 0 -${pi - pi/4}" xyz="-0.2995 -0.269 0.189"/>
     </xacro:sick_nanoscan>
   </xacro:if>

Commit message: restoring normal

File: rox_description/urdf/rox.urdf.xacro (robot description, xacro)
@@ -75,8 +75,8 @@
   <xacro:if value="${scanner == 'nanoscan'}">
     <xacro:sick_nanoscan name="lidar_1" parent="base_link">
-      <origin rpy="${pi} 0 ${pi/4}" xyz="0.2995 0.269 0.189"/>
+      <origin rpy="${pi} 0 ${pi/4}" xyz="${0.2995} 0.269 0.189"/>
     </xacro:sick_nanoscan>
     <xacro:sick_nanoscan name="lidar_2" parent="base_link">
-      <origin rpy="${pi} 0 -${pi - pi/4}" xyz="-0.2995 -0.269 0.189"/>
+      <origin rpy="${pi} 0 -${pi - pi/4}" xyz="-${0.2995} -0.269 0.189"/>
     </xacro:sick_nanoscan>
   </xacro:if>

File: rox_description/urdf/xacros/argo_drive.xacro (robot description, xacro)
@@ -7,20 +7,20 @@
         vis_rot="0 0 0" vis_pos="0 0 0"
         joint_type="${joint_typ}">
-        <origin rpy="0 0 ${pi}" xyz="0.369 0.229 0.123"/>
+        <origin rpy="0 0 ${pi}" xyz="0.239 0.229 0.123"/>
     </xacro:argo_caster>
     <xacro:argo_caster name="caster_front_right" parent="${parent}"
         vis_rot="0 0 ${pi}" vis_pos="0 0 0"
         joint_type="${joint_typ}">
-        <origin rpy="0 0 0" xyz="0.369 -0.229 0.123"/>
+        <origin rpy="0 0 0" xyz="0.239 -0.229 0.123"/>
     </xacro:argo_caster>
     <xacro:argo_caster name="caster_back_left" parent="${parent}"
         vis_rot="0 0 0" vis_pos="0 0 0"
         joint_type="${joint_typ}">
-        <origin rpy="0 0 ${pi}" xyz="-0.369 0.229 0.123"/>
+        <origin rpy="0 0 ${pi}" xyz="-0.239 0.229 0.123"/>
     </xacro:argo_caster>
     <xacro:argo_caster name="caster_back_right" parent="${parent}"
         vis_rot="0 0 ${pi}" vis_pos="0 0 0"
         joint_type="${joint_typ}">
-        <origin rpy="0 0 0" xyz="-0.369 -0.229 0.123"/>
+        <origin rpy="0 0 0" xyz="-0.239 -0.229 0.123"/>
     </xacro:argo_caster>
     <xacro:argo_wheel name="wheel_front_left" parent="caster_front_left_link"
