Commit message: fixing physics for short frame

File: rox_description/urdf/xacros/argo_wheel.xacro (robot description, xacro)
@@ -11,7 +11,7 @@
     <inertial>
     <!-- These are not accurate value -->
-      <mass value="0.03" />
-      <origin rpy="0 0 0" xyz="0 0.0 0" />
-      <inertia ixx="0.02" ixy="0" ixz="0" iyy="0.0000005" iyz="0" izz="0.02" />
+      <mass value="5" />
+      <origin xyz="0 0 0" rpy="0 0 0"/>
+      <inertia ixx="0.02" ixy="0" ixz="0" iyy="0.02" iyz="0" izz="0.02" />
     </inertial>
     <visual>
@@ -22,8 +22,8 @@
     </visual>
     <collision>
-     <origin rpy="0 0 3.14" xyz="0 0.0 0" />
-     <geometry>
-        <mesh filename="package://rox_description/meshes/argo_wheel.dae" scale="0.1 0.1 0.1"/>
-     </geometry>
+     <origin rpy="0 0 0" xyz="0 0.0 0" />
+      <geometry>
+        <sphere radius="0.05" />
+      </geometry>
     </collision>
    </link>

File: rox_description/urdf/xacros/frame.xacro (robot description, xacro)
@@ -11,30 +11,23 @@
       <inertial>
       <!-- These are not accurate value -->
-        <mass value="0.1" />
-        <origin xyz="0 0 0.0" rpy="0.00 0.00 0.0"/>
-        <inertia ixx="0.05" ixy="0.000" ixz="0.000"
-                 iyy="0.0" iyz="0.000"
-                 izz="0.05" />
+        <mass value="80.1" />
+        <origin xyz="0 0 0.18" rpy="0.00 0.00 0.0"/>
+        <inertia ixx="3.947" ixy="0.000" ixz="0.000"
+                 iyy="6.249" iyz="0.000"
+                 izz="8.467" />
       </inertial>
       <visual>
         <origin xyz="0 0 0" rpy="0 0 0" />
         <geometry>
-            <mesh filename="package://rox_description/meshes/${type}_frame.dae" scale="0.1 0.1 0.1"/>
+          <mesh filename="package://rox_description/meshes/${type}_frame.dae" scale="0.1 0.1 0.1"/>
         </geometry>
       </visual>
       <collision>
-        <origin xyz="0 0 0" rpy="0 0 0"/>
+        <origin xyz="0.0 0.0 0.18" rpy="0 0 0"/>
         <geometry>
-            <mesh filename="package://rox_description/meshes/${type}_frame.dae" scale="0.1 0.1 0.1"/>
+          <box size="0.811 0.680 0.360"/>
         </geometry>
       </collision>
     </link>
-    <gazebo reference="${name}">
-    <!-- <kp> 10000 </kp> -->
-    <!-- <fdir1>0 1 0</fdir1> -->
-    <!-- <slip1> 0.1 </slip1> -->
-    <mu1>0.0001</mu1>
-    <mu2>0.0001</mu2>
-  </gazebo>
   </xacro:macro>
 </robot>
