Commit message: updating Trike description

File: rox_description/urdf/xacros/diff_wheel.xacro (robot description, xacro)
@@ -18,5 +18,5 @@
         <origin rpy="0 0 ${pi/2}" xyz="0 0.0 0" />
         <geometry>
-        <mesh filename="package://rox_description/meshes/diff_wheel.dae" scale="0.1 0.1 0.1"/>
+        <mesh filename="package://rox_description/meshes/diff_wheel.dae" scale="0.001 0.001 0.001"/>
         </geometry>
       </visual>
@@ -24,5 +24,5 @@
         <origin rpy="0 0 0" xyz="0 0.0 0" />
         <geometry>
-        <mesh filename="package://rox_description/meshes/diff_wheel.dae" scale="0.1 0.1 0.1"/>
+        <mesh filename="package://rox_description/meshes/diff_wheel.dae" scale="0.001 0.001 0.001"/>
         </geometry>
       </collision>

File: rox_description/urdf/xacros/trike_drive.xacro (robot description, xacro)
@@ -7,6 +7,6 @@
         vis_rot="-${pi/2} 0 -${pi/2}" vis_pos="0 0 0"
         joint_type="${joint_typ}">
-        <origin rpy="0 0 0" xyz="-${0.2785 - 0.04 + frame_len} 0.0 0.123"/>
-        <!-- For the caster position 0.2785 is   -->
+        <origin rpy="0 0 0" xyz="-${0.2785 - 0.045 + frame_len} 0.0 0.124"/>
+        <!-- For the caster position 0.2785 is L3.2 and 0.045 is the Swivel lead -->
     </xacro:diff_caster>
     <xacro:diff_wheel name="wheel_left" parent="${parent}"
