Commit message: updating mass and inertia for better simulation

File: rox_description/urdf/xacros/frame.xacro (robot description, xacro)
@@ -12,9 +12,9 @@
       <inertial>
       <!-- These are not accurate value -->
-        <mass value="30" />
-        <origin xyz="0 0 0" rpy="0 0 0"/>
-        <inertia ixx="1.71402" ixy="0.0" ixz="0.0"
-                 iyy="0.8856" iyz="0.0"
-                 izz="2.5725" />
+        <mass value="0.5" />
+        <origin xyz="0 0 0.0" rpy="0 0 0"/>
+        <inertia ixx="0.005" ixy="0.0" ixz="0.0"
+                 iyy="0.005" iyz="0.0"
+                 izz="0.005" />
       </inertial>
       <visual>

Commit message: setting the frame back for the collision

File: rox_description/urdf/xacros/frame.xacro (robot description, xacro)
@@ -24,7 +24,7 @@
       </visual>
       <collision>
-        <origin xyz="0.0 0.0 0.18" rpy="0 0 0"/>
+        <origin xyz="0.0 0.0 0.0" rpy="0 0 0"/>
         <geometry>
-          <box size="0.811 0.680 0.360"/>
+          <mesh filename="package://rox_description/meshes/${type}_frame.dae" scale="0.1 0.1 0.1"/>
         </geometry>
       </collision>

Commit message: Supporting Jazzy (#26)
* updating gz

* fixing physics for short frame

* updating the params

* updating the behavior trees to v4.0

* setting the frame back for the collision

* updating the navigation params

* using relative path for setting the behavior tree

* updating the dependencies

* Trike support (#28)

* added trike support to rox-desc

* updating Trike description

* param tuning, model updates and more

* comment fixes

File: rox_description/urdf/xacros/frame.xacro (robot description, xacro)
@@ -11,30 +11,23 @@
       <inertial>
       <!-- These are not accurate value -->
-        <mass value="0.1" />
-        <origin xyz="0 0 0.0" rpy="0.00 0.00 0.0"/>
-        <inertia ixx="0.05" ixy="0.000" ixz="0.000"
-                 iyy="0.0" iyz="0.000"
-                 izz="0.05" />
+        <mass value="8.0" />
+        <origin xyz="-0.243 0 0.18" rpy="0.0 0.0 0.0"/>
+        <inertia ixx="0.299" ixy="0.0" ixz="0.0"
+                 iyy="0.351" iyz="0.0"
+                 izz="0.360" />
       </inertial>
       <visual>
-        <origin xyz="0 0 0" rpy="0 0 0" />
+        <origin xyz="-0.243 0.0 0.0" rpy="0 0 0" />
         <geometry>
-            <mesh filename="package://rox_description/meshes/${type}_frame.dae" scale="0.1 0.1 0.1"/>
+          <mesh filename="package://rox_description/meshes/${type}_frame.dae" scale="0.1 0.1 0.1"/>
         </geometry>
       </visual>
       <collision>
-        <origin xyz="0 0 0" rpy="0 0 0"/>
+        <origin xyz="-0.243 0.0 0.0" rpy="0 0 0"/>
         <geometry>
-            <mesh filename="package://rox_description/meshes/${type}_frame.dae" scale="0.1 0.1 0.1"/>
+          <mesh filename="package://rox_description/meshes/${type}_frame.dae" scale="0.1 0.1 0.1"/>
         </geometry>
       </collision>
     </link>
-    <gazebo reference="${name}">
-    <!-- <kp> 10000 </kp> -->
-    <!-- <fdir1>0 1 0</fdir1> -->
-    <!-- <slip1> 0.1 </slip1> -->
-    <mu1>0.0001</mu1>
-    <mu2>0.0001</mu2>
-  </gazebo>
   </xacro:macro>
 </robot>

File: rox_description/urdf/xacros/gazebo.xacro (robot description, xacro)
@@ -35,5 +35,5 @@
         <!-- Set output to sensor_msgs/LaserScan to get same output type as gazebo_ros_laser -->
         <output_type>sensor_msgs/LaserScan</output_type>
-        <ignition_frame_id>lidar_1_link</ignition_frame_id>
+        <gz_frame_id>lidar_1_link</gz_frame_id>
       </sensor>
     </gazebo>
@@ -71,10 +71,10 @@
         <!-- Set output to sensor_msgs/LaserScan to get same output type as gazebo_ros_laser -->
         <output_type>sensor_msgs/LaserScan</output_type>
-        <ignition_frame_id>lidar_2_link</ignition_frame_id>
+        <gz_frame_id>lidar_2_link</gz_frame_id>
       </sensor>
     </gazebo>
     <gazebo reference="imu_link">
         <sensor name="imu_sensor" type="imu">
-            <ignition_frame_id>imu_link</ignition_frame_id>
+            <gz_frame_id>imu_link</gz_frame_id>
             <update_rate>50</update_rate>
             <visualize>false</visualize>
@@ -84,6 +84,6 @@
     </gazebo>
     <gazebo>
-      <plugin filename="ignition-gazebo-odometry-publisher-system"
-          name="ignition::gazebo::systems::OdometryPublisher">
+      <plugin filename="gz-sim-odometry-publisher-system"
+          name="gz::sim::systems::OdometryPublisher">
           <odom_frame>odom</odom_frame>
           <odom_covariance_topic>odom</odom_covariance_topic>
@@ -92,13 +92,46 @@
           <odom_publish_frequency>100</odom_publish_frequency>
       </plugin>
-      <plugin filename="ignition-gazebo-imu-system"
-          name="ignition::gazebo::systems::Imu">
+      <plugin filename="gz-sim-imu-system"
+          name="gz::sim::systems::Imu">
       </plugin>
-      <plugin filename="ignition-gazebo-velocity-control-system"
-          name="ignition::gazebo::systems::VelocityControl">
-          <topic>cmd_vel</topic>
-      </plugin>
-      <plugin filename="ignition-gazebo-sensors-system"
-          name="ignition::gazebo::systems::Sensors">
+      <!-- For ArgoDrive platforms -->
+      <xacro:if value="${rox_typ == 'argo'}">
+        <plugin filename="gz-sim-velocity-control-system"
+            name="gz::sim::systems::VelocityControl">
+            <topic>cmd_vel</topic>
+        </plugin>
+      </xacro:if>
+      <!-- DiffDrive control for trike and diff -->
+      <xacro:if value="${rox_typ == 'diff' or rox_typ == 'trike'}">
+        <plugin filename="gz-sim-diff-drive-system"
+          name="gz::sim::systems::DiffDrive">
+          <left_joint>wheel_left_joint</left_joint>
+          <right_joint>wheel_right_joint</right_joint>
+          <wheel_separation>0.555</wheel_separation>
+          <wheel_radius>0.075</wheel_radius>
+          <max_linear_acceleration>1</max_linear_acceleration>
+          <min_linear_acceleration>-1</min_linear_acceleration>
+          <max_angular_acceleration>10.0</max_angular_acceleration>
+          <min_angular_acceleration>-10.0</min_angular_acceleration>
+          <max_linear_velocity>2.0</max_linear_velocity>
+          <min_linear_velocity>-2.0</min_linear_velocity>
+          <max_angular_velocity>10.0</max_angular_velocity>
+          <min_angular_velocity>-10.0</min_angular_velocity>
+          <topic>/cmd_vel</topic>
+          <odom_topic>/odom</odom_topic>
+          <tf_topic>/tf</tf_topic>
+          <odom_publish_frequency>50</odom_publish_frequency>
+        </plugin>
+        <plugin
+          filename="gz-sim-joint-state-publisher-system"
+          name="gz::sim::systems::JointStatePublisher">
+          <joint_name>wheel_left_joint</joint_name>
+          <joint_name>wheel_right_joint</joint_name>
+          <topic>joint_states</topic>
+          <update_rate>30</update_rate>
+        </plugin>
+      </xacro:if>
+      <plugin filename="gz-sim-sensors-system"
+        name="gz::sim::systems::Sensors">
       </plugin>
     </gazebo>
