Commit message: fixing the wheel dimensions

File: rox_description/urdf/xacros/argo_drive.xacro (robot description, xacro)
@@ -7,20 +7,20 @@
         vis_rot="0 0 0" vis_pos="0 0 0"
         joint_type="${joint_typ}">
-        <origin rpy="0 0 ${pi}" xyz="0.519 0.359 0.112"/>
+        <origin rpy="0 0 ${pi}" xyz="0.519 0.359 0.1095"/>
     </xacro:argo_caster>
     <xacro:argo_caster name="caster_front_right" parent="${parent}"
         vis_rot="0 0 ${pi}" vis_pos="0 0 0"
         joint_type="${joint_typ}">
-        <origin rpy="0 0 0" xyz="0.519 -0.359 0.112"/>
+        <origin rpy="0 0 0" xyz="0.519 -0.359 0.1095"/>
     </xacro:argo_caster>
     <xacro:argo_caster name="caster_back_left" parent="${parent}"
         vis_rot="0 0 0" vis_pos="0 0 0"
         joint_type="${joint_typ}">
-        <origin rpy="0 0 ${pi}" xyz="-0.519 0.359 0.112"/>
+        <origin rpy="0 0 ${pi}" xyz="-0.519 0.359 0.1095"/>
     </xacro:argo_caster>
     <xacro:argo_caster name="caster_back_right" parent="${parent}"
         vis_rot="0 0 ${pi}" vis_pos="0 0 0"
         joint_type="${joint_typ}">
-        <origin rpy="0 0 0" xyz="-0.519 -0.359 0.112"/>
+        <origin rpy="0 0 0" xyz="-0.519 -0.359 0.1095"/>
     </xacro:argo_caster>
     <xacro:argo_wheel name="wheel_front_left" parent="caster_front_left_link"
