Commit message: fixed issue with linear axis not moving in gz when dual arm was spawned
Signed-off-by: Adarsh Karan Kesavadas Prasanth <adarshkaran01@gmail.com>

File: rox_description/urdf/xacros/linear_axis.xacro (robot description, xacro)
@@ -85,5 +85,5 @@
       <origin xyz="0 0 0" rpy="0 0 0"/>
       <!-- Travel: 888mm derived from spec (1417mm column top - 529mm base top) -->
-      <limit lower="0.0" upper="0.888" effort="50000" velocity="0.15"/>
+      <limit lower="0.0" upper="0.888" effort="${linear_axis_effort_limit}" velocity="0.15"/>
       <parent link="linear_axis_fixed_link"/>
       <child link="linear_axis_slide_link"/>
@@ -124,5 +124,5 @@
           </command_interface>
           <state_interface name="position">
-            <param name="initial_value">0.0</param>
+            <param name="initial_value">0.05</param>
           </state_interface>
           <state_interface name="velocity"/>

Commit message: fixing the height

File: rox_description/urdf/xacros/linear_axis.xacro (robot description, xacro)
@@ -63,10 +63,10 @@
     <!--
       Slide mesh sits at Z=861-1161mm in CAD frame (mid-stroke position).
-      At joint=0 (lowest), slide should be at Z≈335mm (just above rail base).
-      Visual offset: -(861 - 335) = -526mm = -0.526m shifts mesh to bottom of travel.
+      At joint=0 (lowest), slide should be at Z≈394mm (just above rail base).
+      Visual offset: -(861 - 394) = -467mm = -0.467m shifts mesh to bottom of travel.
     -->
     <link name="linear_axis_slide_link">
       <visual>
-        <origin rpy="0 0 0" xyz="0 0 -0.527"/>
+        <origin rpy="0 0 0" xyz="0 0 -0.467"/>
         <geometry>
           <mesh filename="package://rox_description/meshes/linear_axis_slide.dae" scale="0.001 0.001 0.001"/>
@@ -74,5 +74,5 @@
       </visual>
       <collision>
-        <origin rpy="0 0 0" xyz="0 0 -0.527"/>
+        <origin rpy="0 0 0" xyz="0 0 -0.467"/>
         <geometry>
           <mesh filename="package://rox_description/meshes/linear_axis_slide.dae" scale="0.001 0.001 0.001"/>
