Commit message: better physics

File: rox_description/urdf/xacros/argo_caster.xacro (robot description, xacro)
@@ -4,7 +4,5 @@
    <joint name="${name}_joint" type="${joint_type}">
     <xacro:insert_block name="origin" />
-    <limit effort="1000.0" lower="-1e+16" upper="1e+16" velocity="3.5"/>
     <axis xyz="1 0 0" />
-    <joint_properties damping="1" friction="1" />
     <parent link="${parent}" />
     <child link="${name}_link" />
@@ -13,7 +11,7 @@
     <inertial>
     <!-- These are not accurate value -->
-      <mass value="2" />
-      <origin xyz="0 0 0" rpy="0 0 0" />
-      <inertia ixx="0.00044332" ixy="0" ixz="0" iyy="0.00044332" iyz="0" izz="0.00072" />
+      <mass value="0.025" />
+      <origin xyz="${vis_pos}" rpy="${vis_rot}" />
+      <inertia ixx="0.02" ixy="0" ixz="0" iyy="0.0" iyz="0" izz="0.02" />
     </inertial>
     <visual>

File: rox_description/urdf/xacros/argo_wheel.xacro (robot description, xacro)
@@ -4,7 +4,5 @@
    <joint name="${name}_joint" type="${joint_type}">
     <xacro:insert_block name="origin" />
-    <limit effort="1000.0" lower="-1e+16" upper="1e+16" velocity="3.5"/>
     <axis xyz="1 0 0" />
-    <joint_properties damping="1" friction="1" />
     <parent link="${parent}" />
     <child link="${name}_link" />
@@ -13,10 +11,10 @@
     <inertial>
     <!-- These are not accurate value -->
-      <mass value="2" />
-      <origin rpy="0 0 3.14" xyz="0 0.020 0" />
-      <inertia ixx="0.00044332" ixy="0" ixz="0" iyy="0.00044332" iyz="0" izz="0.00072" />
+      <mass value="0.03" />
+      <origin rpy="0 0 0" xyz="0 0.0 0" />
+      <inertia ixx="0.02" ixy="0" ixz="0" iyy="0.0000005" iyz="0" izz="0.02" />
     </inertial>
     <visual>
-      <origin rpy="0 0 3.14" xyz="0 0.020 0" />
+      <origin rpy="0 0 3.14" xyz="0 0.0 0" />
       <geometry>
         <mesh filename="package://rox_description/meshes/argo_wheel.dae" scale="0.1 0.1 0.1"/>
@@ -24,5 +22,5 @@
     </visual>
     <collision>
-     <origin rpy="0 0 3.14" xyz="0 0.020 0" />
+     <origin rpy="0 0 3.14" xyz="0 0.0 0" />
      <geometry>
         <mesh filename="package://rox_description/meshes/argo_wheel.dae" scale="0.1 0.1 0.1"/>

File: rox_description/urdf/xacros/frame.xacro (robot description, xacro)
@@ -5,5 +5,4 @@
     <xacro:insert_block name="origin" />
     <axis xyz="0 0 -1" />
-    <joint_properties damping="1" friction="1" />
     <parent link="${parent}" />
     <child link="${name}" />
@@ -12,9 +11,9 @@
       <inertial>
       <!-- These are not accurate value -->
-        <mass value="0.5" />
-        <origin xyz="0 0 0.0" rpy="0 0 0"/>
-        <inertia ixx="0.005" ixy="0.0" ixz="0.0"
-                 iyy="0.005" iyz="0.0"
-                 izz="0.005" />
+        <mass value="0.1" />
+        <origin xyz="0 0 0.0" rpy="0.00 0.00 0.0"/>
+        <inertia ixx="0.05" ixy="0.000" ixz="0.000"
+                 iyy="0.0" iyz="0.000"
+                 izz="0.05" />
       </inertial>
       <visual>
@@ -31,4 +30,11 @@
       </collision>
     </link>
+    <gazebo reference="${name}">
+    <!-- <kp> 10000 </kp> -->
+    <!-- <fdir1>0 1 0</fdir1> -->
+    <!-- <slip1> 0.1 </slip1> -->
+    <mu1>0.0001</mu1>
+    <mu2>0.0001</mu2>
+  </gazebo>
   </xacro:macro>
 </robot>

Commit message: updating the rotation axis of the argo drives

File: rox_description/urdf/xacros/argo_caster.xacro (robot description, xacro)
@@ -4,5 +4,5 @@
    <joint name="${name}_joint" type="${joint_type}">
     <xacro:insert_block name="origin" />
-    <axis xyz="1 0 0" />
+    <axis xyz="0 0 1" />
     <dynamics damping="1." friction="1.0"/>
     <limit effort="1000.0" lower="-1e+16" upper="1e+16" velocity="100"/>
