Commit message: updating arm orientation

File: rox_description/urdf/xacros/ur_arm.urdf.xacro (robot description, xacro)
@@ -49,5 +49,5 @@
     >
     <!-- position of arm in the world -->
-    <origin xyz="0.0 0.0 ${arm_height}" rpy="0.0 0.0 0.0" />
+    <origin xyz="0.0 0.0 ${arm_height}" rpy="0.0 0.0 -1.57" />
   </xacro:ur_robot>
   <!-- this condition is to ensure that ros2_control doesn't interfere with gz_ros2_control during simulation  -->
